File: kicad_files/bcrl_power_supply/_autosave-bcrl_power_supply.kicad_sch (KiCad schematic)
At the start: 7 parts, among them J1 OSTVN02A150, J2 OSTVN02A150, J3 OSTVN02A150, J4 OSTVN02A150, J5 OSTVN02A150, J6 OSTVN02A150, J7 OSTVN02A150

Commit message: ...
Changed lines of the file:
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@@
     )
   )
-  (symbol (lib_id "power:GND") (at 60.96 24.13 0) (unit 1)
+  (symbol (lib_id "power:GND") (at 68.58 27.94 0) (unit 1)
     (in_bom yes) (on_board yes) (dnp no) (fields_autoplaced)
-    (property "Reference" "#PWR02" (at 60.96 30.48 0)
+    (property "Reference" "#PWR02" (at 68.58 34.29 0)
       (effects (font (size 1.27 1.27)) hide)
     )
-    (property "Value" "GND" (at 60.96 29.21 0)
+    (property "Value" "GND" (at 68.58 33.02 0)
       (effects (font (size 1.27 1.27)))
     )
-    (property "Footprint" "" (at 60.96 24.13 0)
+    (property "Footprint" "" (at 68.58 27.94 0)
       (effects (font (size 1.27 1.27)) hide)
     )
-    (property "Datasheet" "" (at 60.96 24.13 0)
+    (property "Datasheet" "" (at 68.58 27.94 0)
       (effects (font (size 1.27 1.27)) hide)
     )
