File: kicad_files/bcrl_power_supply/PYBE20-Q48-S5_EMC.kicad_sch (KiCad schematic)
At the start: 8 parts

Commit message: cleanup PCB
Parts:
- renumbered C15 to C41, C16 to C42, C17 to C43, C18 to C44, C19 to C45, C20 to C46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
