File: kicad_files/bcrl_power_supply/TxRFswMUXv1_board.kicad_sch (KiCad schematic)
At the start: 27 parts, among them J1 OSTVN02A150, J11 5034801600, J2 OSTVN02A150, J3 OSTVN02A150, J4 OSTVN02A150, J5 OSTVN02A150, J6 OSTVN02A150, J7 OSTVN02A150, J8 OSTVN02A150, J9 5034801600, P1 5104338-1, P2 5104338-1, P3 Conn_01x10, P4 Conn_01x10, U1 PDQ10-Q48-S3-D

Commit message: fixed path
Parts:
- removed CJ1, CJ2, CJ3, CJ4: Conn_01x10, Connector_PinSocket_2.54mm:PinSocket_1x10_P2.54mm_Vertical, symbol Connector_Generic:Conn_01x10
- removed P3, P4: Conn_01x10, Connector_PinSocket_1.27mm:PinSocket_1x10_P1.27mm_Vertical, symbol Connector_Generic:Conn_01x10
- added P3, P4: 5104338-1, symbol BCRL_power_supply:5104338-1
- added PS9: EHHD010A0B41-HZ, symbol BCRL_power_supply:EHHD010A0B41-HZ
- PS1, PS2, PS3, PS4: footprint (none) -> BCRL_power_supply:CONV_PYBE20-Q48-S9
- PS5, PS6, PS7, PS8: footprint PYBE20-Q48-S5:CONV_PYBE20-Q48-S5 -> BCRL_power_supply:CONV_PYBE20-Q48-S5
Connections:
- net 48V: now also PS1.2 (VIN), PS2.2 (VIN), PS3.2 (VIN), PS4.2 (VIN), PS6.2 (VIN), PS7.2 (VIN), PS8.2 (VIN)
- net GND: now also J11.1, J11.16, J11.7, J11.8, J9.1, J9.16, J9.8, J9.9, P1.4, P1.6, P2.4, P2.6, PS1.1 (GND), PS1.5 (0V), PS2.1 (GND), PS2.5 (0V), PS3.1 (GND), PS3.5 (0V), PS4.1 (GND), PS4.5 (0V), PS5.1 (GND), PS6.1 (GND), PS7.1 (GND), PS8.1 (GND), P3.4, P3.6, P4.4, P4.6
- net P3.1_VCTL2_SW1: now reaches J9.10
- net P3.1_VCTL2_SW1: now also J9.11, P3.1, P3.2
- net P3.3_VCTL1: now reaches J9.12
- net P3.3_VCTL1: now also P3.3
- net P4.1_VCTL2_SW1: now reaches J9.13
- net P4.1_VCTL2_SW1: now also J9.14, P4.1, P4.2
- net P4.3_VCTL1: now reaches J9.15
- net P4.3_VCTL1: now also P4.3
- net P1.1_VCTL2_SW1: now reaches J9.2
- net P1.1_VCTL2_SW1: now also P1.1
- net P1.2_VCTL2_SW2: now reaches J9.3
- net P1.2_VCTL2_SW2: now also P1.2
- net P1.3_VCTL1: now reaches J9.4
- net P1.3_VCTL1: now also P1.3
- net P2.1_VCTL2_SW1: now reaches J9.5
- net P2.1_VCTL2_SW1: now also J9.6, P2.1, P2.2
- net P2.3_VCTL1: now reaches J9.7
- net P2.3_VCTL1: now also P2.3
- net +5V: now reaches PS6.3 (+VO)
- net +5V: now also PS5.3 (+VO), PS7.3 (+VO), PS8.3 (+VO)
- net TxPA2_5V_CTL: now reaches PS6.6 (CTRL)
- net TxPA2_5V_CTL: now also J11.3
- net +3.3V: now reaches U1.3 (+VOUT)
- net +3.3V: now also P1.5, P2.5, P3.5, P4.5
- net TxPA4_5V_CTL: now reaches PS8.6 (CTRL)
- net TxPA4_5V_CTL: now also J11.5
- net +9V: now reaches PS2.3 (+VO)
- net +9V: now also PS1.3 (+VO), PS3.3 (+VO), PS4.3 (+VO)
- net TxPA2_9V_CTL: now reaches PS2.6 (CTRL)
- net TxPA1_5V_CTL: now reaches J11.2
- net TxPA1_5V_CTL: now also PS5.6 (CTRL)
- net TxPA3_5V_CTL: now reaches J11.4
- net TxPA3_5V_CTL: now also PS7.6 (CTRL)
- net TxPA3_9V_CTL: now reaches PS3.6 (CTRL)
- net TxPA4_9V_CTL: now reaches PS4.6 (CTRL)
- net TxPA1_9V_CTL: now reaches PS1.6 (CTRL)
Other:
- moved on the sheet: J11, J9, PS1, PS2, PS3, PS4, PS5, PS6, PS7, PS8, U1

Commit message: added 8V dcdc
Parts:
- added PS10: PQC50-48-S12-O, symbol BCRL_power_supply:PQC50-48-S12-O
- added PS11: PQC50-48-S5-O, symbol BCRL_power_supply:PQC50-48-S5-O
Connections:
- net +5V: now also J1.1, J2.1, J3.1, J4.1, PS11.8 (+VO)
- net 48V: now also PS9.1 (VI+), U1.1 (+VIN), PS10.1 (VIN)
- net GND: now also J1.2, J2.2, J3.2, J4.2, J5.2, J6.2, J7.2, J8.2, PS5.5 (0V), PS6.5 (0V), PS7.5 (0V), PS8.5 (0V), PS9.3 (VI-), PS9.4 (VO-), U1.2 (-VIN), U1.5 (-VOUT), PS10.3 (GND), PS10.4 (0V)
- net +8V: now reaches J5.1
- net +8V: now also J6.1, J7.1, J8.1
- net +12V: now reaches PS9.8 (VO+)
- net +12V: now also PS10.8 (+VO)
Other:
- moved on the sheet: J1, PS9, U1

Commit message: TxMUX done
Parts:
- removed PS10: PQC50-48-S12-O, symbol BCRL_power_supply:PQC50-48-S12-O
- J11, J9: footprint (none) -> BCRL_power_supply:MOLEX_5034801600
- P1, P2, P3, P4: footprint (none) -> BCRL_power_supply:TE_5104338-1
- PS11: footprint (none) -> BCRL_power_supply:CONV_PQC50-48-S5-O
- PS9: footprint (none) -> BCRL_power_supply:CONV_EHHD010A0B41-HZ
- U1: footprint PDQ10-Q48-S3-D:CONV_PDQ10-Q48-S3-D -> BCRL_power_supply:CONV_PDQ10-Q48-S3-D
Connections:
- net +12V: now also PS11.2 (CTRL)
- net +5V: now also PS11.7 (SENSE+)
- net 48V: now also PS11.1 (VIN)
- net GND: now also J11.S1 (SHIELD), J11.S2 (SHIELD__1), J9.S1 (SHIELD), J9.S2 (SHIELD__1), PS11.3 (GND), PS11.4 (0V), PS11.5 (SENSE-)
- no-connect marks 0 -> 35
Other:
- moved on the sheet: PS11

Commit message: added decoupling
Parts:
- added C1, C2, C3, C4: C, symbol Device:C
- added PS10, PS12, PS13: PQC50-48-S5-O, BCRL_power_supply:CONV_PQC50-48-S5-O, symbol BCRL_power_supply:PQC50-48-S5-O
- added R1, R2, R3: R, symbol Device:R
- added RV1: R_Potentiometer_Trim, symbol Device:R_Potentiometer_Trim
Connections:
- net +12V: now also PS10.2 (CTRL), PS12.2 (CTRL), PS13.2 (CTRL)
- net +5V: now also J1.2, J11.1, J11.16, J11.8, J11.9, J11.S1 (SHIELD), J11.S2 (SHIELD__1), J2.2, J3.2, J4.2, J5.2, J6.2, J7.2, J8.2, J9.1, J9.16, J9.8, J9.9, J9.S1 (SHIELD), J9.S2 (SHIELD__1), P1.4, P1.6, P2.4, P2.6, P3.4, P3.6, P4.4, P4.6, PS1.1 (GND), PS1.5 (0V), PS11.3 (GND), PS11.4 (0V), PS11.5 (SENSE-), PS2.1 (GND), PS2.5 (0V), PS3.1 (GND), PS3.5 (0V), PS4.1 (GND), PS4.5 (0V), PS5.1 (GND), PS5.5 (0V), PS6.1 (GND), PS6.5 (0V), PS7.1 (GND), PS7.5 (0V), PS8.1 (GND), PS8.5 (0V), PS9.3 (VI-), PS9.4 (VO-), U1.2 (-VIN), U1.5 (-VOUT), C1.2, C2.1, C2.2, C3.2, C4.1, C4.2, PS10.3 (GND), PS10.4 (0V), PS10.5 (SENSE-), PS10.7 (SENSE+), PS10.8 (+VO), PS12.3 (GND), PS12.4 (0V), PS12.5 (SENSE-), PS12.7 (SENSE+), PS12.8 (+VO), PS13.3 (GND), PS13.4 (0V), PS13.5 (SENSE-), PS13.7 (SENSE+), PS13.8 (+VO), R1.2, R2.1, RV1.1
- net 48V: now also C1.1, C3.1, PS10.1 (VIN), PS12.1 (VIN), PS13.1 (VIN)
- net TxPAx4_8V_CTL: now reaches J11.6
- net at PS11.6 (TRIM): now also RV1.2
- removed net GND: J1.2, J11.1, J11.16, J11.7, J11.8, J11.S1 (SHIELD), J11.S2 (SHIELD__1), J2.2, J3.2, J4.2, J5.2, J6.2, J7.2, J8.2, J9.1, J9.16, J9.8, J9.9, J9.S1 (SHIELD), J9.S2 (SHIELD__1), P1.4, P1.6, P2.4, P2.6, P3.4, P3.6, P4.4, P4.6, PS1.1 (GND), PS1.5 (0V), PS11.3 (GND), PS11.4 (0V), PS11.5 (SENSE-), PS2.1 (GND), PS2.5 (0V), PS3.1 (GND), PS3.5 (0V), PS4.1 (GND), PS4.5 (0V), PS5.1 (GND), PS5.5 (0V), PS6.1 (GND), PS6.5 (0V), PS7.1 (GND), PS7.5 (0V), PS8.1 (GND), PS8.5 (0V), PS9.3 (VI-), PS9.4 (VO-), U1.2 (-VIN), U1.5 (-VOUT)
- new net: R1.1, R2.2, R3.2
- new net: R3.1, RV1.3
- no-connect marks 35 -> 34
Other:
- moved on the sheet: PS11

Commit message: added EMC
Parts:
- removed C1, C2, C3, C4: C, symbol Device:C
- removed PS1, PS2, PS3, PS4: PYBE20-Q48-S9, BCRL_power_supply:CONV_PYBE20-Q48-S9, symbol BCRL_power_supply:PYBE20-Q48-S9
- removed PS10, PS11, PS12, PS13: PQC50-48-S5-O, BCRL_power_supply:CONV_PQC50-48-S5-O, symbol BCRL_power_supply:PQC50-48-S5-O
- removed PS5, PS6, PS7, PS8: PYBE20-Q48-S5, BCRL_power_supply:CONV_PYBE20-Q48-S5, symbol BCRL_power_supply:PYBE20-Q48-S5
- removed PS9: EHHD010A0B41-HZ, BCRL_power_supply:CONV_EHHD010A0B41-HZ, symbol BCRL_power_supply:EHHD010A0B41-HZ
- removed R1, R2, R3: R, symbol Device:R
- removed RV1: R_Potentiometer_Trim, symbol Device:R_Potentiometer_Trim
- removed U1: PDQ10-Q48-S3-D, BCRL_power_supply:CONV_PDQ10-Q48-S3-D, symbol BCRL_power_supply:PDQ10-Q48-S3-D
- added J13, J14: OSTVN02A150, BCRL_power_supply:CONN_OSTVN02A150_OST, symbol 2024-02-14_22-22-09:OSTVN02A150
- renumbered J8 to J10, J9 to J11, J11 to J12, J1 to J3, J2 to J4, J3 to J5, J4 to J6, J5 to J7, J6 to J8, J7 to J9
Connections:
- net +5V: no longer J10.2, J11.1, J11.16, J11.8, J11.9, J11.S1 (SHIELD), J11.S2 (SHIELD__1), J12.1, J12.16, J12.8, J12.9, J12.S1 (SHIELD), J12.S2 (SHIELD__1), J3.2, J4.2, J5.2, J6.2, J7.2, J8.2, J9.2, P1.4, P1.6, P2.4, P2.6, P3.4, P3.6, P4.4, P4.6
- new net EN_12V_FROM_5V: J13.1
- new net EN_3.3V_FROM_5V: J14.1
- new net GND: J10.2, J11.1, J11.16, J11.8, J11.9, J11.S1 (SHIELD), J11.S2 (SHIELD__1), J12.1, J12.16, J12.8, J12.9, J12.S1 (SHIELD), J12.S2 (SHIELD__1), J13.2, J14.2, J3.2, J4.2, J5.2, J6.2, J7.2, J8.2, J9.2, P1.4, P1.6, P2.4, P2.6, P3.4, P3.6, P4.4, P4.6
- no-connect marks 34 -> 23
Other:
- added sheet EHHD010A0B41-HZ_EMC (EHHD010A0B41-HZ.kicad_sch)
- added sheet PDQ10-Q48-S3-D_EMC_1 (PDQ10-Q48-S3-D_EMC.kicad_sch)
- added sheet PQC50-48-S5-O_EMC_trimmed_1 (PQC50-48-S5-O_EMC_trimmed.kicad_sch)
- added sheet PQC50-48-S5-O_EMC_trimmed_2 (PQC50-48-S5-O_EMC_trimmed.kicad_sch)
- added sheet PQC50-48-S5-O_EMC_trimmed_3 (PQC50-48-S5-O_EMC_trimmed.kicad_sch)
- added sheet PQC50-48-S5-O_EMC_trimmed_4 (PQC50-48-S5-O_EMC_trimmed.kicad_sch)
- added sheet PYBE20-Q48-S5_EMC_1 (PYBE20-Q48-S5_EMC.kicad_sch)
- added sheet PYBE20-Q48-S5_EMC_2 (PYBE20-Q48-S5_EMC.kicad_sch)
- added sheet PYBE20-Q48-S5_EMC_3 (PYBE20-Q48-S5_EMC.kicad_sch)
- added sheet PYBE20-Q48-S5_EMC_4 (PYBE20-Q48-S5_EMC.kicad_sch)
- moved on the sheet: J10, J11, J12, J3, J4, J5, J6, J7, J8, J9, P1, P2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

Commit message: added more circuits
Parts:
- renumbered J13 to J11, J14 to J12, J11 to J13, J12 to J14

Commit message: WIP
Parts:
- removed J12: OSTVN02A150, BCRL_power_supply:CONN_OSTVN02A150_OST, symbol 2024-02-14_22-22-09:OSTVN02A150
- added D1: LED, symbol Device:LED
- added J46, J47, J48, J49, J50: Conn_01x02, symbol Connector_Generic:Conn_01x02
- added J55: 5034801600, BCRL_power_supply:MOLEX_5034801600, symbol BCRL_power_supply:5034801600
- added R13: R, symbol Device:R
Connections:
- net GND: now also J46.2 (Pin_2), J47.2 (Pin_2), J48.2 (Pin_2), J49.2 (Pin_2), J50.2 (Pin_2), R13.1
- net TxPA1_5V_CTL: now also J46.1 (Pin_1)
- net TxPA2_5V_CTL: now also J47.1 (Pin_1)
- net TxPA3_5V_CTL: now also J48.1 (Pin_1)
- net TxPA4_5V_CTL: now also J49.1 (Pin_1)
- net TxPAx4_8V_CTL: now also J50.1 (Pin_1)
- new net: D1.1 (K), R13.2
Other:
- removed sheet PDQ10-Q48-S3-D_EMC_1

Commit message: cleanup PCB
Parts:
- removed J50: Conn_01x02, symbol Connector_Generic:Conn_01x02
- added D2, D3, D4, D5, D6, D7, D8: LED, LED_SMD:LED_0603_1608Metric, symbol Device:LED
- added J17, J18, J19, J20: Conn_01x02, Connector_PinHeader_2.54mm:PinHeader_1x02_P2.54mm_Vertical, symbol Connector_Generic:Conn_01x02
- added R2, R3, R4, R5, R6, R7, R8: 1k, Resistor_SMD:R_0603_1608Metric, symbol Device:R
- D1: footprint (none) -> LED_SMD:LED_0603_1608Metric
- J13: renamed from J46; footprint (none) -> Connector_PinHeader_2.54mm:PinHeader_1x02_P2.54mm_Vertical
- J14: renamed from J47; footprint (none) -> Connector_PinHeader_2.54mm:PinHeader_1x02_P2.54mm_Vertical
- J15: renamed from J48; footprint (none) -> Connector_PinHeader_2.54mm:PinHeader_1x02_P2.54mm_Vertical
- J16: renamed from J49; footprint (none) -> Connector_PinHeader_2.54mm:PinHeader_1x02_P2.54mm_Vertical
- R1: renamed from R13; value R -> 1k; footprint (none) -> Resistor_SMD:R_0603_1608Metric
- renumbered J9 to J10, J10 to J11, J11 to J12, J13 to J21, J14 to J22, J55 to J23, J3 to J4, J4 to J5, J5 to J6, J6 to J7, J7 to J8, J8 to J9
Connections:
- net +5V_1: now also D1.2 (A), J4.1
- net GND: now also J23.S1 (SHIELD), J23.S2 (SHIELD__1), J17.2 (Pin_2), J18.2 (Pin_2), J19.2 (Pin_2), J20.2 (Pin_2), R2.1, R3.1, R4.1, R5.1, R6.1, R7.1, R8.1
- net TxPA1_8V_CTL: now reaches J22.10
- net TxPA1_8V_CTL: now also J17.1 (Pin_1)
- net TxPA2_8V_CTL: now reaches J22.11
- net TxPA2_8V_CTL: now also J18.1 (Pin_1)
- net TxPA3_8V_CTL: now reaches J22.12
- net TxPA3_8V_CTL: now also J19.1 (Pin_1)
- net TxPA4_8V_CTL: now reaches J22.13
- net TxPA4_8V_CTL: now also J20.1 (Pin_1)
- removed net +5V: J4.1, J5.1, J6.1, J7.1
- removed net +8V: J10.1, J11.1, J8.1, J9.1
- net TxPAx4_8V_CTL: no longer names the net of J22.6
- new net: D8.1 (K), R8.2
- new net: D4.1 (K), R4.2
- new net: D7.1 (K), R7.2
- new net: D6.1 (K), R6.2
- new net: D3.1 (K), R3.2
- new net: D5.1 (K), R5.2
- new net: D2.1 (K), R2.2
- new net +5V_2: D2.2 (A), J5.1
- new net +5V_3: D3.2 (A), J6.1
- new net +5V_4: D4.2 (A), J7.1
- new net +8V_1: D5.2 (A), J8.1
- new net +8V_2: D7.2 (A), J9.1
- new net +8V_3: D6.2 (A), J10.1
- new net +8V_4: D8.2 (A), J11.1
- no-connect marks 23 -> 20
Other:
- removed sheet PYBE20-Q48-S5_EMC_1
- removed sheet PYBE20-Q48-S5_EMC_2
- removed sheet PYBE20-Q48-S5_EMC_3
- removed sheet PYBE20-Q48-S5_EMC_4
- added sheet PDQ10-Q48-S5-D_EMC_1 (PDQ10-Q48-S5-D_EMC.kicad_sch)
- added sheet PDQ10-Q48-S5-D_EMC_2 (PDQ10-Q48-S5-D_EMC.kicad_sch)
- added sheet PDQ10-Q48-S5-D_EMC_3 (PDQ10-Q48-S5-D_EMC.kicad_sch)
- added sheet PDQ10-Q48-S5-D_EMC_4 (PDQ10-Q48-S5-D_EMC.kicad_sch)
- moved on the sheet: D1, J13, J14, J15, J16, R1
