File: kicad_files/bcrl_power_supply/TxRFswMUXv1_board.kicad_sch (KiCad schematic)
At the start: 40 parts, among them J10 OSTVN02A150, J11 OSTVN02A150, J12 OSTVN02A150, J13 Conn_01x02, J14 Conn_01x02, J15 Conn_01x02, J16 Conn_01x02, J17 Conn_01x02, J18 Conn_01x02, J19 Conn_01x02, J20 Conn_01x02, J21 5034801600, J22 5034801600, J23 5034801600, J4 OSTVN02A150, J5 OSTVN02A150, J6 OSTVN02A150, J7 OSTVN02A150, J8 OSTVN02A150, J9 OSTVN02A150, P1 5104338-1, P2 5104338-1, P3 5104338-1, P4 5104338-1

Commit message: ...
Parts:
- removed J12: OSTVN02A150, BCRL_power_supply:CONN_OSTVN02A150_OST, symbol 2024-02-14_22-22-09:OSTVN02A150
- removed J23: 5034801600, BCRL_power_supply:MOLEX_5034801600, symbol BCRL_power_supply:5034801600
Other:
- removed sheet EHHD010A0B41-HZ_EMC

Commit message: started LCSC, fixing DCDC
Other:
- added sheet PYBE20-Q48-S9_8V_trim_1 (PYBE20-Q48-S9_8V_trim.kicad_sch)

Commit message: big reorg
Parts:
- removed J10, J11, J4, J5, J6, J7, J8, J9: OSTVN02A150, BCRL_power_supply:CONN_OSTVN02A150_OST, symbol 2024-02-14_22-22-09:OSTVN02A150
- removed J13, J14, J15, J16, J17, J18, J19, J20: Conn_01x02, Connector_PinHeader_2.54mm:PinHeader_1x02_P2.54mm_Vertical, symbol Connector_Generic:Conn_01x02
- removed J21, J22: 5034801600, BCRL_power_supply:MOLEX_5034801600, symbol BCRL_power_supply:5034801600
- added J30, J31, J32, J33, J34, J35, J36, J37: OSTVN02A150, BCRL_power_supply:CONN_OSTVN02A150_OST, symbol 2024-02-14_22-22-09:OSTVN02A150
- added J38, J39, J40, J41, J42, J43, J44, J45: Conn_01x02, Connector_PinHeader_2.54mm:PinHeader_1x02_P2.54mm_Vertical, symbol Connector_Generic:Conn_01x02
- added J46, J47: 5034801600, BCRL_power_supply:MOLEX_5034801600, symbol BCRL_power_supply:5034801600
Connections:
- net +5V_1: now also J30.1
- net +5V_2: now also J31.1
- net +5V_3: now also J32.1
- net +5V_4: now also J33.1
- net +8V_1: now also J34.1
- net +8V_2: now also J35.1
- net +8V_3: now also J36.1
- net +8V_4: now also J37.1
- net GND: now also J30.2, J31.2, J32.2, J33.2, J34.2, J35.2, J36.2, J37.2, J38.2 (Pin_2), J39.2 (Pin_2), J40.2 (Pin_2), J41.2 (Pin_2), J42.2 (Pin_2), J43.2 (Pin_2), J44.2 (Pin_2), J45.2 (Pin_2), J46.1, J46.16, J46.8, J46.9, J46.S1 (SHIELD), J46.S2 (SHIELD__1), J47.1, J47.16, J47.8, J47.9, J47.S1 (SHIELD), J47.S2 (SHIELD__1)
- net P1.1_VCTL2_SW1 renamed P1.1_VCTRL2_SW1
- net P1.1_VCTRL2_SW1: now also J46.2
- net P1.2_VCTL2_SW2 renamed P1.2_VCTRL2_SW2
- net P1.2_VCTRL2_SW2: now also J46.3
- net P1.3_VCTL1 renamed P1.3_VCTRL1
- net P1.3_VCTRL1: now also J46.4
- net P2.1_VCTL2_SW1 renamed P2.1_VCTRL2_SW1
- net P2.1_VCTRL2_SW1: now also J46.5, J46.6
- net P2.3_VCTL1 renamed P2.3_VCTRL1
- net P2.3_VCTRL1: now also J46.7
- net P3.1_VCTL2_SW1 renamed P3.1_VCTRL2_SW1
- net P3.1_VCTRL2_SW1: now also J46.10, J46.11
- net P3.3_VCTL1 renamed P3.3_VCTRL1
- net P3.3_VCTRL1: now also J46.12
- net P4.1_VCTL2_SW1 renamed P4.1_VCTRL2_SW1
- net P4.1_VCTRL2_SW1: now also J46.13, J46.14
- net P4.3_VCTL1 renamed P4.3_VCTRL1
- net P4.3_VCTRL1: now also J46.15
- new net TxPA1_5V_CTRL: J38.1 (Pin_1), J47.2
- new net TxPA1_8V_CTRL: J42.1 (Pin_1), J47.10
- new net TxPA2_5V_CTRL: J39.1 (Pin_1), J47.3
- new net TxPA2_8V_CTRL: J43.1 (Pin_1), J47.11
- new net TxPA3_5V_CTRL: J40.1 (Pin_1), J47.4
- new net TxPA3_8V_CTRL: J44.1 (Pin_1), J47.12
- new net TxPA4_5V_CTRL: J41.1 (Pin_1), J47.5
- new net TxPA4_8V_CTRL: J45.1 (Pin_1), J47.13
Other:
- removed sheet PYBE20-Q48-S9_8V_trim_1

Commit message: big changes
Parts:
- added D18: LED, LED_SMD:LED_0603_1608Metric, symbol Device:LED
- added J38: Conn_01x02, Connector_PinHeader_2.54mm:PinHeader_1x02_P2.54mm_Vertical, symbol Connector_Generic:Conn_01x02
- added R25: 1k, Resistor_SMD:R_0603_1608Metric, symbol Device:R
- renumbered J36 to J10, J37 to J11, J38 to J12, J39 to J13, J40 to J14, J41 to J15, J42 to J16, J43 to J17, J44 to J18, J45 to J19, J46 to J20, J47 to J21, J30 to J4, J31 to J5, J32 to J6, J33 to J7, J34 to J8, J35 to J9
Connections:
- net GND: now also J38.2 (Pin_2), R25.1
- new net: D18.1 (K), R25.2
- new net +12V: D18.2 (A)
- new net +12V_CTRL: J38.1 (Pin_1)
Other:
- removed sheet PQC50-48-S5-O_EMC_trimmed_1
- removed sheet PQC50-48-S5-O_EMC_trimmed_2
- removed sheet PQC50-48-S5-O_EMC_trimmed_3
- removed sheet PQC50-48-S5-O_EMC_trimmed_4
- added sheet EHHD010A0B41-HZ3 (EHHD010A0B41-HZ.kicad_sch)
- added sheet IND108W_EMC_8V_5 (IND108W_EMC_8V.kicad_sch)
- added sheet IND108W_EMC_8V_6 (IND108W_EMC_8V.kicad_sch)
- added sheet IND108W_EMC_8V_7 (IND108W_EMC_8V.kicad_sch)
- added sheet IND108W_EMC_8V_8 (IND108W_EMC_8V.kicad_sch)
- moved on the sheet: D1, D2, D3, D4, D5, D6, D7, D8, J10, J11, J20, J21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
