File: kicad_files/bcrl_power_supply/TxRFswMUXv1_board.kicad_sch (KiCad schematic)
At the start: 41 parts, among them J10 OSTVN02A150, J11 OSTVN02A150, J12 Conn_01x02, J13 Conn_01x02, J14 Conn_01x02, J15 Conn_01x02, J16 Conn_01x02, J17 Conn_01x02, J18 Conn_01x02, J19 Conn_01x02, J20 5034801600, J21 5034801600, J38 Conn_01x02, J4 OSTVN02A150, J5 OSTVN02A150, J6 OSTVN02A150, J7 OSTVN02A150, J8 OSTVN02A150, J9 OSTVN02A150, P1 5104338-1, P2 5104338-1, P3 5104338-1, P4 5104338-1

Commit message: almost done schematic
Parts:
- renumbered D18 to D1, D1 to D2, D2 to D3, D3 to D4, D4 to D5, D5 to D6, D6 to D7, D7 to D8, D8 to D9, J38 to J20, J20 to J21, J21 to J22, R25 to R1, R1 to R2, R2 to R3, R3 to R4, R4 to R5, R5 to R6, R6 to R7, R7 to R8, R8 to R9

Commit message: board review
Parts:
- D1, D2, D3, D4, D5, D6, D7, D8, D9: value LED -> LED 0603
Changed lines of the file:
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@@
 			)
 		)
-		(property "Value" "LED"
+		(property "Value" "LED 0603"
 			(at 265.7475 60.96 0)
 			(effects
@@
 			)
 		)
-		(property "Value" "LED"
+		(property "Value" "LED 0603"
 			(at 265.7475 41.91 0)
 			(effects
@@
 			)
 		)
-		(property "Value" "LED"
+		(property "Value" "LED 0603"
 			(at 265.7475 142.24 0)
 			(effects
@@
 			)
 		)
-		(property "Value" "LED"
+		(property "Value" "LED 0603"
 			(at 264.4775 20.32 0)
 			(effects
@@
 			)
 		)
-		(property "Value" "LED"
+		(property "Value" "LED 0603"
 			(at 265.7475 99.06 0)
 			(effects
@@
 			)
 		)
-		(property "Value" "LED"
+		(property "Value" "LED 0603"
 			(at 267.0175 120.65 0)
 			(effects
@@
 			)
 		)
-		(property "Value" "LED"
+		(property "Value" "LED 0603"
 			(at 265.7475 80.01 0)
 			(effects
@@
 			)
 		)
-		(property "Value" "LED"
+		(property "Value" "LED 0603"
 			(at 267.0175 162.56 0)
 			(effects
@@
 			)
 		)
-		(property "Value" "LED"
+		(property "Value" "LED 0603"
 			(at 181.9275 149.86 0)
 			(effects

Commit message: digikey BOM
Parts:
- D1, D2, D3, D4, D5, D6, D7, D8, D9: DigiKey_Part_Number (none) -> 150060GS75000
- J10, J11, J4, J5, J6, J7, J8, J9: DigiKey_Part_Number (none) -> OSTVN02A150
- J21, J22: DigiKey_Part_Number (none) -> 5034801600
- P1, P2, P3, P4: DigiKey_Part_Number (none) -> 5104338-1
- R1, R2, R3, R4, R5, R6, R7, R8, R9: DigiKey_Part_Number (none) -> ESR03EZPF1001
