File: kicad_files/bcrl_power_supply/bcrl_power_supply.kicad_pcb (KiCad board)
At the start: 2 copper layers, 0 parts

Commit message: cleanup PCB
Parts:
- added C1: 4.7uf/100v, Capacitor_SMD:C_0603_1608Metric, F.Cu at (283.7, 162.8)
- added C10: 4.7uf/100v, Capacitor_SMD:C_0603_1608Metric, F.Cu at (116.3, 228.7)
- added C100: 330uf/63v, Capacitor_SMD:C_0603_1608Metric, F.Cu at (83.1, 192.2)
- added C101: 680uf/100v, Capacitor_SMD:C_0603_1608Metric, F.Cu at (116.3, 109.3)
- added C102: 4.7uf/100v, Capacitor_SMD:C_0603_1608Metric, F.Cu at (116.3, 111.8)
- added C103: 4.7uf/100v, Capacitor_SMD:C_0603_1608Metric, F.Cu at (116.3, 114.3)
- added C104: 4.7uf/100v, Capacitor_SMD:C_0603_1608Metric, F.Cu at (116.3, 116.8)
- added C105: 4.7uf/100v, Capacitor_SMD:C_0603_1608Metric, F.Cu at (116.3, 119.3)
- added C106: 2.2nf/400vac, Capacitor_SMD:C_0603_1608Metric, F.Cu at (120.3, 109.3)
- added C107: 2.2nf/400vac, Capacitor_SMD:C_0603_1608Metric, F.Cu at (120.3, 111.8)
- added C108: 330uf/63v, Capacitor_SMD:C_0603_1608Metric, F.Cu at (120.3, 114.3)
- added C109: 4.7uf/100v, Capacitor_SMD:C_0603_1608Metric, F.Cu at (217.7, 223.5)
- added C11: 4.7uf/100v, Capacitor_SMD:C_0603_1608Metric, F.Cu at (116.3, 231.2)
- added C110: 4.7uf/100v, Capacitor_SMD:C_0603_1608Metric, F.Cu at (217.7, 226.0)
- added C111: 4.7uf/100v, Capacitor_SMD:C_0603_1608Metric, F.Cu at (250.7, 193.1)
- added C112: 4.7uf/100v, Capacitor_SMD:C_0603_1608Metric, F.Cu at (250.7, 195.6)
- added C113: 680uf/100v, Capacitor_SMD:C_0603_1608Metric, F.Cu at (190.8, 148.2)
- added C114: 4.7uf/100v, Capacitor_SMD:C_0603_1608Metric, F.Cu at (190.8, 150.8)
- added C115: 4.7uf/100v, Capacitor_SMD:C_0603_1608Metric, F.Cu at (190.8, 153.3)
- added C116: 4.7uf/100v, Capacitor_SMD:C_0603_1608Metric, F.Cu at (190.8, 155.8)
- added C117: 4.7uf/100v, Capacitor_SMD:C_0603_1608Metric, F.Cu at (190.8, 158.3)
- added C118: 2.2nf/400vac, Capacitor_SMD:C_0603_1608Metric, F.Cu at (194.8, 148.2)
- added C119: 2.2nf/400vac, Capacitor_SMD:C_0603_1608Metric, F.Cu at (194.8, 150.8)
- added C12: 4.7uf/100v, Capacitor_SMD:C_0603_1608Metric, F.Cu at (116.3, 233.7)
- added C120: 330uf/63v, Capacitor_SMD:C_0603_1608Metric, F.Cu at (194.8, 153.3)
- added C121: 680uf/100v, Capacitor_SMD:C_0603_1608Metric, F.Cu at (153.6, 187.2)
- added C122: 4.7uf/100v, Capacitor_SMD:C_0603_1608Metric, F.Cu at (153.6, 189.7)
- added C123: 4.7uf/100v, Capacitor_SMD:C_0603_1608Metric, F.Cu at (153.6, 192.2)
- added C124: 4.7uf/100v, Capacitor_SMD:C_0603_1608Metric, F.Cu at (153.6, 194.7)
- added C125: 4.7uf/100v, Capacitor_SMD:C_0603_1608Metric, F.Cu at (153.6, 197.2)
- added C126: 2.2nf/400vac, Capacitor_SMD:C_0603_1608Metric, F.Cu at (157.6, 187.2)
- added C127: 2.2nf/400vac, Capacitor_SMD:C_0603_1608Metric, F.Cu at (157.6, 189.7)
- added C128: 330uf/63v, Capacitor_SMD:C_0603_1608Metric, F.Cu at (157.6, 192.2)
- added C129: 680uf/100v, Capacitor_SMD:C_0603_1608Metric, F.Cu at (228.0, 109.3)
- added C13: 4.7uf/100v, Capacitor_SMD:C_0603_1608Metric, F.Cu at (116.3, 236.2)
- added C130: 4.7uf/100v, Capacitor_SMD:C_0603_1608Metric, F.Cu at (228.0, 111.8)
- added C131: 4.7uf/100v, Capacitor_SMD:C_0603_1608Metric, F.Cu at (228.0, 114.3)
- added C132: 4.7uf/100v, Capacitor_SMD:C_0603_1608Metric, F.Cu at (228.0, 116.8)
- added C133: 4.7uf/100v, Capacitor_SMD:C_0603_1608Metric, F.Cu at (228.0, 119.3)
- added C134: 2.2nf/400vac, Capacitor_SMD:C_0603_1608Metric, F.Cu at (232.0, 109.3)
- added C135: 2.2nf/400vac, Capacitor_SMD:C_0603_1608Metric, F.Cu at (232.0, 111.8)
- added C136: 330uf/63v, Capacitor_SMD:C_0603_1608Metric, F.Cu at (232.0, 114.3)
- added C137: 680uf/100v, Capacitor_SMD:C_0603_1608Metric, F.Cu at (153.6, 109.3)
- added C138: 4.7uf/100v, Capacitor_SMD:C_0603_1608Metric, F.Cu at (153.6, 111.8)
- added C139: 4.7uf/100v, Capacitor_SMD:C_0603_1608Metric, F.Cu at (153.6, 114.3)
- added C14: 2.2nf/400vac, Capacitor_SMD:C_0603_1608Metric, F.Cu at (120.3, 226.2)
- added C140: 4.7uf/100v, Capacitor_SMD:C_0603_1608Metric, F.Cu at (153.6, 116.8)
- added C141: 4.7uf/100v, Capacitor_SMD:C_0603_1608Metric, F.Cu at (153.6, 119.3)
- added C142: 2.2nf/400vac, Capacitor_SMD:C_0603_1608Metric, F.Cu at (157.6, 109.3)
- added C143: 2.2nf/400vac, Capacitor_SMD:C_0603_1608Metric, F.Cu at (157.6, 111.8)
- added C144: 330uf/63v, Capacitor_SMD:C_0603_1608Metric, F.Cu at (157.6, 114.3)
- added C145: 4.7uf/100v, Capacitor_SMD:C_0603_1608Metric, F.Cu at (217.7, 162.8)
- added C146: 4.7uf/100v, Capacitor_SMD:C_0603_1608Metric, F.Cu at (217.7, 165.3)
- added C15: 2.2nf/400vac, Capacitor_SMD:C_0603_1608Metric, F.Cu at (120.3, 228.7)
- added C16: 330uf/63v, Capacitor_SMD:C_0603_1608Metric, F.Cu at (120.3, 231.2)
- added C17: 680uf/100v, Capacitor_SMD:C_0603_1608Metric, F.Cu at (116.3, 187.2)
- added C18: 4.7uf/100v, Capacitor_SMD:C_0603_1608Metric, F.Cu at (116.3, 189.7)
- added C19: 4.7uf/100v, Capacitor_SMD:C_0603_1608Metric, F.Cu at (116.3, 192.2)
- added C2: 4.7uf/100v, Capacitor_SMD:C_0603_1608Metric, F.Cu at (283.7, 165.3)
- added C20: 4.7uf/100v, Capacitor_SMD:C_0603_1608Metric, F.Cu at (116.3, 194.7)
- added C21: 4.7uf/100v, Capacitor_SMD:C_0603_1608Metric, F.Cu at (116.3, 197.2)
- added C22: 2.2nf/400vac, Capacitor_SMD:C_0603_1608Metric, F.Cu at (120.3, 187.2)
- added C23: 2.2nf/400vac, Capacitor_SMD:C_0603_1608Metric, F.Cu at (120.3, 189.7)
- added C24: 330uf/63v, Capacitor_SMD:C_0603_1608Metric, F.Cu at (120.3, 192.2)
- added C25: 680uf/100v, Capacitor_SMD:C_0603_1608Metric, F.Cu at (79.1, 226.2)
- added C26: 4.7uf/100v, Capacitor_SMD:C_0603_1608Metric, F.Cu at (79.1, 228.7)
- added C27: 4.7uf/100v, Capacitor_SMD:C_0603_1608Metric, F.Cu at (79.1, 231.2)
- added C28: 4.7uf/100v, Capacitor_SMD:C_0603_1608Metric, F.Cu at (79.1, 233.7)
- added C29: 4.7uf/100v, Capacitor_SMD:C_0603_1608Metric, F.Cu at (79.1, 236.2)
- added C3: 4.7uf/100v, Capacitor_SMD:C_0603_1608Metric, F.Cu at (250.7, 223.5)
- added C30: 2.2nf/400vac, Capacitor_SMD:C_0603_1608Metric, F.Cu at (83.1, 226.2)
- added C31: 2.2nf/400vac, Capacitor_SMD:C_0603_1608Metric, F.Cu at (83.1, 228.7)
- added C32: 330uf/63v, Capacitor_SMD:C_0603_1608Metric, F.Cu at (83.1, 231.2)
- added C33: 680uf/100v, Capacitor_SMD:C_0603_1608Metric, F.Cu at (79.1, 148.2)
- added C34: 4.7uf/100v, Capacitor_SMD:C_0603_1608Metric, F.Cu at (79.1, 150.8)
- added C35: 4.7uf/100v, Capacitor_SMD:C_0603_1608Metric, F.Cu at (79.1, 153.3)
- added C36: 4.7uf/100v, Capacitor_SMD:C_0603_1608Metric, F.Cu at (79.1, 155.8)
- added C37: 4.7uf/100v, Capacitor_SMD:C_0603_1608Metric, F.Cu at (79.1, 158.3)
- added C38: 2.2nf/400vac, Capacitor_SMD:C_0603_1608Metric, F.Cu at (83.1, 148.2)
- added C39: 2.2nf/400vac, Capacitor_SMD:C_0603_1608Metric, F.Cu at (83.1, 150.8)
- added C4: 4.7uf/100v, Capacitor_SMD:C_0603_1608Metric, F.Cu at (250.7, 226.0)
- added C40: 330uf/63v, Capacitor_SMD:C_0603_1608Metric, F.Cu at (83.1, 153.3)
- added C41: 4.7uf/100v, Capacitor_SMD:C_0603_1608Metric, F.Cu at (250.7, 162.8)
- added C42: 4.7uf/100v, Capacitor_SMD:C_0603_1608Metric, F.Cu at (250.7, 165.3)
- added C43: 680uf/100v, Capacitor_SMD:C_0603_1608Metric, F.Cu at (248.2, 54.3)
- added C44: 4.7uf/100v, Capacitor_SMD:C_0603_1608Metric, F.Cu at (248.2, 56.8)
- added C45: 4.7uf/100v, Capacitor_SMD:C_0603_1608Metric, F.Cu at (248.2, 59.3)
- added C46: 4.7uf/100v, Capacitor_SMD:C_0603_1608Metric, F.Cu at (248.2, 61.8)
- added C47: 4.7uf/100v, Capacitor_SMD:C_0603_1608Metric, F.Cu at (248.2, 64.3)
- added C48: 2.2nf/400vac, Capacitor_SMD:C_0603_1608Metric, F.Cu at (252.2, 54.3)
- added C49: 2.2nf/400vac, Capacitor_SMD:C_0603_1608Metric, F.Cu at (252.2, 56.8)
- added C5: 4.7uf/100v, Capacitor_SMD:C_0603_1608Metric, F.Cu at (255.0, 123.8)
- added C50: 330uf/63v, Capacitor_SMD:C_0603_1608Metric, F.Cu at (252.2, 59.3)
- added C51: 680uf/100v, Capacitor_SMD:C_0603_1608Metric, F.Cu at (153.6, 226.2)
- added C52: 4.7uf/100v, Capacitor_SMD:C_0603_1608Metric, F.Cu at (153.6, 228.7)
- added C53: 4.7uf/100v, Capacitor_SMD:C_0603_1608Metric, F.Cu at (153.6, 231.2)
- added C54: 4.7uf/100v, Capacitor_SMD:C_0603_1608Metric, F.Cu at (153.6, 233.7)
- added C55: 4.7uf/100v, Capacitor_SMD:C_0603_1608Metric, F.Cu at (153.6, 236.2)
- added C56: 2.2nf/400vac, Capacitor_SMD:C_0603_1608Metric, F.Cu at (157.6, 226.2)
- added C57: 2.2nf/400vac, Capacitor_SMD:C_0603_1608Metric, F.Cu at (157.6, 228.7)
- added C58: 330uf/63v, Capacitor_SMD:C_0603_1608Metric, F.Cu at (157.6, 231.2)
- added C59: 680uf/100v, Capacitor_SMD:C_0603_1608Metric, F.Cu at (153.6, 148.2)
- added C6: 4.7uf/100uf, Capacitor_SMD:C_0603_1608Metric, F.Cu at (255.0, 126.3)
- added C60: 4.7uf/100v, Capacitor_SMD:C_0603_1608Metric, F.Cu at (153.6, 150.8)
- added C61: 4.7uf/100v, Capacitor_SMD:C_0603_1608Metric, F.Cu at (153.6, 153.3)
- added C62: 4.7uf/100v, Capacitor_SMD:C_0603_1608Metric, F.Cu at (153.6, 155.8)
- added C63: 4.7uf/100v, Capacitor_SMD:C_0603_1608Metric, F.Cu at (153.6, 158.3)
- added C64: 2.2nf/400vac, Capacitor_SMD:C_0603_1608Metric, F.Cu at (157.6, 148.2)
- added C65: 2.2nf/400vac, Capacitor_SMD:C_0603_1608Metric, F.Cu at (157.6, 150.8)
- added C66: 330uf/63v, Capacitor_SMD:C_0603_1608Metric, F.Cu at (157.6, 153.3)
- added C67: 680uf/100v, Capacitor_SMD:C_0603_1608Metric, F.Cu at (190.8, 109.3)
- added C68: 4.7uf/100v, Capacitor_SMD:C_0603_1608Metric, F.Cu at (190.8, 111.8)
- added C69: 4.7uf/100v, Capacitor_SMD:C_0603_1608Metric, F.Cu at (190.8, 114.3)
- added C7: 4.7uf/100v, Capacitor_SMD:C_0603_1608Metric, F.Cu at (283.7, 193.1)
- added C70: 4.7uf/100v, Capacitor_SMD:C_0603_1608Metric, F.Cu at (190.8, 116.8)
- added C71: 4.7uf/100v, Capacitor_SMD:C_0603_1608Metric, F.Cu at (190.8, 119.3)
- added C72: 2.2nf/400vac, Capacitor_SMD:C_0603_1608Metric, F.Cu at (194.8, 109.3)
- added C73: 2.2nf/400vac, Capacitor_SMD:C_0603_1608Metric, F.Cu at (194.8, 111.8)
- added C74: 330uf/63v, Capacitor_SMD:C_0603_1608Metric, F.Cu at (194.8, 114.3)
- added C75: 680uf/100v, Capacitor_SMD:C_0603_1608Metric, F.Cu at (79.1, 109.3)
- added C76: 4.7uf/100v, Capacitor_SMD:C_0603_1608Metric, F.Cu at (79.1, 111.8)
- added C77: 4.7uf/100v, Capacitor_SMD:C_0603_1608Metric, F.Cu at (79.1, 114.3)
- added C78: 4.7uf/100v, Capacitor_SMD:C_0603_1608Metric, F.Cu at (79.1, 116.8)
- added C79: 4.7uf/100v, Capacitor_SMD:C_0603_1608Metric, F.Cu at (79.1, 119.3)
- added C8: 4.7uf/100v, Capacitor_SMD:C_0603_1608Metric, F.Cu at (283.7, 195.6)
- added C80: 2.2nf/400vac, Capacitor_SMD:C_0603_1608Metric, F.Cu at (83.1, 109.3)
- added C81: 2.2nf/400vac, Capacitor_SMD:C_0603_1608Metric, F.Cu at (83.1, 111.8)
- added C82: 330uf/63v, Capacitor_SMD:C_0603_1608Metric, F.Cu at (83.1, 114.3)
- added C83: 680uf/100v, Capacitor_SMD:C_0603_1608Metric, F.Cu at (116.3, 148.2)
- added C84: 4.7uf/100v, Capacitor_SMD:C_0603_1608Metric, F.Cu at (116.3, 150.8)
- added C85: 4.7uf/100v, Capacitor_SMD:C_0603_1608Metric, F.Cu at (116.3, 153.3)
- added C86: 4.7uf/100v, Capacitor_SMD:C_0603_1608Metric, F.Cu at (116.3, 155.8)
- added C87: 4.7uf/100v, Capacitor_SMD:C_0603_1608Metric, F.Cu at (116.3, 158.3)
- added C88: 2.2nf/400vac, Capacitor_SMD:C_0603_1608Metric, F.Cu at (120.3, 148.2)
- added C89: 2.2nf/400vac, Capacitor_SMD:C_0603_1608Metric, F.Cu at (120.3, 150.8)
- added C9: 680uf/100v, Capacitor_SMD:C_0603_1608Metric, F.Cu at (116.3, 226.2)
- added C90: 330uf/63v, Capacitor_SMD:C_0603_1608Metric, F.Cu at (120.3, 153.3)
- added C91: 4.7uf/100v, Capacitor_SMD:C_0603_1608Metric, F.Cu at (217.7, 193.1)
- added C92: 4.7uf/100v, Capacitor_SMD:C_0603_1608Metric, F.Cu at (217.7, 195.6)
- added C93: 680uf/100v, Capacitor_SMD:C_0603_1608Metric, F.Cu at (79.1, 187.2)
- added C94: 4.7uf/100v, Capacitor_SMD:C_0603_1608Metric, F.Cu at (79.1, 189.7)
- added C95: 4.7uf/100v, Capacitor_SMD:C_0603_1608Metric, F.Cu at (79.1, 192.2)
- added C96: 4.7uf/100v, Capacitor_SMD:C_0603_1608Metric, F.Cu at (79.1, 194.7)
- added C97: 4.7uf/100v, Capacitor_SMD:C_0603_1608Metric, F.Cu at (79.1, 197.2)
- added C98: 2.2nf/400vac, Capacitor_SMD:C_0603_1608Metric, F.Cu at (83.1, 187.2)
- added C99: 2.2nf/400vac, Capacitor_SMD:C_0603_1608Metric, F.Cu at (83.1, 189.7)
- added D1: LED, LED_SMD:LED_0603_1608Metric, F.Cu at (143.5, 62.2)
- added D10: LED, LED_SMD:LED_0603_1608Metric, F.Cu at (90.4, 64.8)
- added D11: LED, LED_SMD:LED_0603_1608Metric, F.Cu at (90.4, 67.4)
- added D12: LED, LED_SMD:LED_0603_1608Metric, F.Cu at (90.4, 70.0)
- added D13: LED, LED_SMD:LED_0603_1608Metric, F.Cu at (90.4, 72.5)
- added D14: LED, LED_SMD:LED_0603_1608Metric, F.Cu at (90.4, 75.1)
- added D15: LED, LED_SMD:LED_0603_1608Metric, F.Cu at (90.4, 77.7)
- added D16: LED, LED_SMD:LED_0603_1608Metric, F.Cu at (90.4, 80.3)
- added D2: LED, LED_SMD:LED_0603_1608Metric, F.Cu at (143.5, 64.8)
- added D3: LED, LED_SMD:LED_0603_1608Metric, F.Cu at (143.5, 67.4)
- added D4: LED, LED_SMD:LED_0603_1608Metric, F.Cu at (143.5, 70.0)
- added D5: LED, LED_SMD:LED_0603_1608Metric, F.Cu at (143.5, 72.5)
- added D6: LED, LED_SMD:LED_0603_1608Metric, F.Cu at (143.5, 75.1)
- added D7: LED, LED_SMD:LED_0603_1608Metric, F.Cu at (143.5, 77.7)
- added D8: LED, LED_SMD:LED_0603_1608Metric, F.Cu at (143.5, 80.3)
- added D9: LED, LED_SMD:LED_0603_1608Metric, F.Cu at (90.4, 62.2)
- added J1: OSTVN02A150, BCRL_power_supply:CONN_OSTVN02A150_OST, F.Cu at (263.5, 146.2)
- added J10: OSTVN02A150, BCRL_power_supply:CONN_OSTVN02A150_OST, F.Cu at (153.8, 40.1)
- added J11: OSTVN02A150, BCRL_power_supply:CONN_OSTVN02A150_OST, F.Cu at (153.8, 48.5)
- added J12: OSTVN02A150, BCRL_power_supply:CONN_OSTVN02A150_OST, F.Cu at (153.8, 56.8)
- added J13: Conn_01x02, Connector_PinHeader_2.54mm:PinHeader_1x02_P2.54mm_Vertical, F.Cu at (132.5, 30.9)
- added J14: Conn_01x02, Connector_PinHeader_2.54mm:PinHeader_1x02_P2.54mm_Vertical, F.Cu at (137.2, 30.9)
- added J15: Conn_01x02, Connector_PinHeader_2.54mm:PinHeader_1x02_P2.54mm_Vertical, F.Cu at (141.8, 30.9)
- added J16: Conn_01x02, Connector_PinHeader_2.54mm:PinHeader_1x02_P2.54mm_Vertical, F.Cu at (146.5, 30.9)
- added J17: Conn_01x02, Connector_PinHeader_2.54mm:PinHeader_1x02_P2.54mm_Vertical, F.Cu at (151.1, 30.9)
- added J18: Conn_01x02, Connector_PinHeader_2.54mm:PinHeader_1x02_P2.54mm_Vertical, F.Cu at (155.8, 30.9)
- added J19: Conn_01x02, Connector_PinHeader_2.54mm:PinHeader_1x02_P2.54mm_Vertical, F.Cu at (160.4, 30.9)
- added J2: OSTVN02A150, BCRL_power_supply:CONN_OSTVN02A150_OST, F.Cu at (263.5, 154.6)
- added J20: Conn_01x02, Connector_PinHeader_2.54mm:PinHeader_1x02_P2.54mm_Vertical, F.Cu at (165.1, 30.9)
- added J21: 5034801600, BCRL_power_supply:MOLEX_5034801600, F.Cu at (135.8, 64.0)
- added J22: 5034801600, BCRL_power_supply:MOLEX_5034801600, F.Cu at (135.8, 69.9)
- added J23: 5034801600, BCRL_power_supply:MOLEX_5034801600, F.Cu at (135.8, 75.7)
- added J24: OSTVN02A150, BCRL_power_supply:CONN_OSTVN02A150_OST, F.Cu at (81.6, 40.1)
- added J25: OSTVN02A150, BCRL_power_supply:CONN_OSTVN02A150_OST, F.Cu at (81.6, 48.5)
- added J26: OSTVN02A150, BCRL_power_supply:CONN_OSTVN02A150_OST, F.Cu at (81.6, 56.8)
- added J27: OSTVN02A150, BCRL_power_supply:CONN_OSTVN02A150_OST, F.Cu at (91.2, 40.1)
- added J28: OSTVN02A150, BCRL_power_supply:CONN_OSTVN02A150_OST, F.Cu at (91.2, 48.5)
- added J29: OSTVN02A150, BCRL_power_supply:CONN_OSTVN02A150_OST, F.Cu at (91.2, 56.8)
- added J3: Conn_01x02, Connector_PinHeader_2.54mm:PinHeader_1x02_P2.54mm_Vertical, F.Cu at (270.8, 144.2)
- added J30: OSTVN02A150, BCRL_power_supply:CONN_OSTVN02A150_OST, F.Cu at (100.7, 40.1)
- added J31: OSTVN02A150, BCRL_power_supply:CONN_OSTVN02A150_OST, F.Cu at (100.7, 48.5)
- added J32: OSTVN02A150, BCRL_power_supply:CONN_OSTVN02A150_OST, F.Cu at (100.7, 56.8)
- added J33: Conn_01x02, Connector_PinHeader_2.54mm:PinHeader_1x02_P2.54mm_Vertical, F.Cu at (79.4, 30.9)
- added J34: Conn_01x02, Connector_PinHeader_2.54mm:PinHeader_1x02_P2.54mm_Vertical, F.Cu at (84.1, 30.9)
- added J35: Conn_01x02, Connector_PinHeader_2.54mm:PinHeader_1x02_P2.54mm_Vertical, F.Cu at (88.7, 30.9)
- added J36: Conn_01x02, Connector_PinHeader_2.54mm:PinHeader_1x02_P2.54mm_Vertical, F.Cu at (93.4, 30.9)
- added J37: Conn_01x02, Connector_PinHeader_2.54mm:PinHeader_1x02_P2.54mm_Vertical, F.Cu at (98.0, 30.9)
- added J38: Conn_01x02, Connector_PinHeader_2.54mm:PinHeader_1x02_P2.54mm_Vertical, F.Cu at (102.7, 30.9)
- added J39: Conn_01x02, Connector_PinHeader_2.54mm:PinHeader_1x02_P2.54mm_Vertical, F.Cu at (107.3, 30.9)
- added J4: OSTVN02A150, BCRL_power_supply:CONN_OSTVN02A150_OST, F.Cu at (134.7, 40.1)
- added J40: Conn_01x02, Connector_PinHeader_2.54mm:PinHeader_1x02_P2.54mm_Vertical, F.Cu at (112.0, 30.9)
- added J41: 5034801600, BCRL_power_supply:MOLEX_5034801600, F.Cu at (82.7, 64.0)
- added J42: 5034801600, BCRL_power_supply:MOLEX_5034801600, F.Cu at (82.7, 69.9)
- added J43: Conn_01x04_Pin, Connector_PinHeader_2.54mm:PinHeader_1x04_P2.54mm_Vertical, F.Cu at (269.2, 69.9)
- added J44: Conn_01x04_Pin, Connector_PinHeader_2.54mm:PinHeader_1x04_P2.54mm_Vertical, F.Cu at (273.8, 69.9)
- added J45: Conn_01x04_Pin, Connector_PinHeader_2.54mm:PinHeader_1x04_P2.54mm_Vertical, F.Cu at (278.5, 69.9)
- added J46: Conn_01x04_Pin, Connector_PinHeader_2.54mm:PinHeader_1x04_P2.54mm_Vertical, F.Cu at (283.1, 69.9)
- added J47: Conn_01x04_Pin, Connector_PinHeader_2.54mm:PinHeader_1x04_P2.54mm_Vertical, F.Cu at (248.6, 69.9)
- added J48: Conn_01x04_Pin, Connector_PinHeader_2.54mm:PinHeader_1x04_P2.54mm_Vertical, F.Cu at (253.2, 69.9)
- added J49: Conn_01x04_Pin, Connector_PinHeader_2.54mm:PinHeader_1x04_P2.54mm_Vertical, F.Cu at (257.9, 69.9)
- added J5: OSTVN02A150, BCRL_power_supply:CONN_OSTVN02A150_OST, F.Cu at (134.7, 48.5)
- added J50: Conn_01x04_Pin, Connector_PinHeader_2.54mm:PinHeader_1x04_P2.54mm_Vertical, F.Cu at (262.5, 69.9)
- added J51: Conn_01x04_Pin, Connector_PinHeader_2.54mm:PinHeader_1x04_P2.54mm_Vertical, F.Cu at (265.6, 85.9)
- added J52: Conn_01x04_Pin, Connector_PinHeader_2.54mm:PinHeader_1x04_P2.54mm_Vertical, F.Cu at (270.2, 85.9)
- added J53: Conn_01x04_Pin, Connector_PinHeader_2.54mm:PinHeader_1x04_P2.54mm_Vertical, F.Cu at (274.9, 85.9)
- added J54: Conn_01x04_Pin, Connector_PinHeader_2.54mm:PinHeader_1x04_P2.54mm_Vertical, F.Cu at (279.5, 85.9)
- added J55: Conn_01x04_Pin, Connector_PinHeader_2.54mm:PinHeader_1x04_P2.54mm_Vertical, F.Cu at (265.6, 100.2)
- added J56: Conn_01x04_Pin, Connector_PinHeader_2.54mm:PinHeader_1x04_P2.54mm_Vertical, F.Cu at (270.2, 100.2)
- added J57: Conn_01x04_Pin, Connector_PinHeader_2.54mm:PinHeader_1x04_P2.54mm_Vertical, F.Cu at (274.9, 100.2)
- added J58: Conn_01x04_Pin, Connector_PinHeader_2.54mm:PinHeader_1x04_P2.54mm_Vertical, F.Cu at (279.5, 100.2)
- added J59: Conn_01x06_Pin, Connector_PinHeader_2.54mm:PinHeader_1x06_P2.54mm_Vertical, F.Cu at (261.3, 124.9)
- added J6: OSTVN02A150, BCRL_power_supply:CONN_OSTVN02A150_OST, F.Cu at (134.7, 56.8)
- added J60: Conn_01x06_Pin, Connector_PinHeader_2.54mm:PinHeader_1x06_P2.54mm_Vertical, F.Cu at (265.9, 124.9)
- added J61: Conn_01x06_Pin, Connector_PinHeader_2.54mm:PinHeader_1x06_P2.54mm_Vertical, F.Cu at (270.6, 124.9)
- added J62: Conn_01x06_Pin, Connector_PinHeader_2.54mm:PinHeader_1x06_P2.54mm_Vertical, F.Cu at (275.2, 124.9)
- added J63: Conn_01x04_Pin, Connector_PinHeader_2.54mm:PinHeader_1x04_P2.54mm_Vertical, F.Cu at (277.5, 144.2)
- added J64: Conn_01x04_Pin, Connector_PinHeader_2.54mm:PinHeader_1x04_P2.54mm_Vertical, F.Cu at (281.9, 124.9)
- added J65: Conn_01x06_Pin, Connector_PinHeader_2.54mm:PinHeader_1x06_P2.54mm_Vertical, F.Cu at (257.0, 224.5)
- added J66: Conn_01x06_Pin, Connector_PinHeader_2.54mm:PinHeader_1x06_P2.54mm_Vertical, F.Cu at (261.7, 224.5)
- added J67: Conn_01x06_Pin, Connector_PinHeader_2.54mm:PinHeader_1x06_P2.54mm_Vertical, F.Cu at (266.3, 224.5)
- added J68: Conn_01x06_Pin, Connector_PinHeader_2.54mm:PinHeader_1x06_P2.54mm_Vertical, F.Cu at (271.0, 224.5)
- added J7: OSTVN02A150, BCRL_power_supply:CONN_OSTVN02A150_OST, F.Cu at (144.3, 40.1)
- added J8: OSTVN02A150, BCRL_power_supply:CONN_OSTVN02A150_OST, F.Cu at (144.3, 48.5)
- added J9: OSTVN02A150, BCRL_power_supply:CONN_OSTVN02A150_OST, F.Cu at (144.3, 56.8)
- added L1: 4.7uh/3.1a, Inductor_SMD:L_0603_1608Metric, F.Cu at (283.7, 167.8)
- added L10: 2.2mh, Inductor_SMD:L_0603_1608Metric, F.Cu at (83.1, 155.8)
- added L11: 2.2mh, Inductor_SMD:L_0603_1608Metric, F.Cu at (83.1, 158.3)
- added L12: 4.7uh/3.1a, Inductor_SMD:L_0603_1608Metric, F.Cu at (250.7, 167.8)
- added L13: 2.2mh, Inductor_SMD:L_0603_1608Metric, F.Cu at (252.2, 61.8)
- added L14: 2.2mh, Inductor_SMD:L_0603_1608Metric, F.Cu at (252.2, 64.3)
- added L15: 2.2mh, Inductor_SMD:L_0603_1608Metric, F.Cu at (157.6, 233.7)
- added L16: 2.2mh, Inductor_SMD:L_0603_1608Metric, F.Cu at (157.6, 236.2)
- added L17: 2.2mh, Inductor_SMD:L_0603_1608Metric, F.Cu at (157.6, 155.8)
- added L18: 2.2mh, Inductor_SMD:L_0603_1608Metric, F.Cu at (157.6, 158.3)
- added L19: 2.2mh, Inductor_SMD:L_0603_1608Metric, F.Cu at (194.8, 116.8)
- added L2: 4.7uh/3.1a, Inductor_SMD:L_0603_1608Metric, F.Cu at (250.7, 228.5)
- added L20: 2.2mh, Inductor_SMD:L_0603_1608Metric, F.Cu at (194.8, 119.3)
- added L21: 2.2mh, Inductor_SMD:L_0603_1608Metric, F.Cu at (83.1, 116.8)
- added L22: 2.2mh, Inductor_SMD:L_0603_1608Metric, F.Cu at (83.1, 119.3)
- added L23: 2.2mh, Inductor_SMD:L_0603_1608Metric, F.Cu at (120.3, 155.8)
- added L24: 2.2mh, Inductor_SMD:L_0603_1608Metric, F.Cu at (120.3, 158.3)
- added L25: 4.7uh/3.1a, Inductor_SMD:L_0603_1608Metric, F.Cu at (217.7, 198.2)
- added L26: 2.2mh, Inductor_SMD:L_0603_1608Metric, F.Cu at (83.1, 194.7)
- added L27: 2.2mh, Inductor_SMD:L_0603_1608Metric, F.Cu at (83.1, 197.2)
- added L28: 2.2mh, Inductor_SMD:L_0603_1608Metric, F.Cu at (120.3, 116.8)
- added L29: 2.2mh, Inductor_SMD:L_0603_1608Metric, F.Cu at (120.3, 119.3)
- added L3: 4.7uh/3.1a, Inductor_SMD:L_0603_1608Metric, F.Cu at (283.7, 198.2)
- added L30: 4.7uh/3.1a, Inductor_SMD:L_0603_1608Metric, F.Cu at (217.7, 228.5)
- added L31: 4.7uh/3.1a, Inductor_SMD:L_0603_1608Metric, F.Cu at (250.7, 198.2)
- added L32: 2.2mh, Inductor_SMD:L_0603_1608Metric, F.Cu at (194.8, 155.8)
- added L33: 2.2mh, Inductor_SMD:L_0603_1608Metric, F.Cu at (194.8, 158.3)
- added L34: 2.2mh, Inductor_SMD:L_0603_1608Metric, F.Cu at (157.6, 194.7)
- added L35: 2.2mh, Inductor_SMD:L_0603_1608Metric, F.Cu at (157.6, 197.2)
- added L36: 2.2mh, Inductor_SMD:L_0603_1608Metric, F.Cu at (232.0, 116.8)
- added L37: 2.2mh, Inductor_SMD:L_0603_1608Metric, F.Cu at (232.0, 119.3)
- added L38: 2.2mh, Inductor_SMD:L_0603_1608Metric, F.Cu at (157.6, 116.8)
- added L39: 2.2mh, Inductor_SMD:L_0603_1608Metric, F.Cu at (157.6, 119.3)
- added L4: 2.2mh, Inductor_SMD:L_0603_1608Metric, F.Cu at (120.3, 233.7)
- added L40: 4.7uh/3.1a, Inductor_SMD:L_0603_1608Metric, F.Cu at (217.7, 167.8)
- added L5: 2.2mh, Inductor_SMD:L_0603_1608Metric, F.Cu at (120.3, 236.2)
- added L6: 2.2mh, Inductor_SMD:L_0603_1608Metric, F.Cu at (120.3, 194.7)
- added L7: 2.2mh, Inductor_SMD:L_0603_1608Metric, F.Cu at (120.3, 197.2)
- added L8: 2.2mh, Inductor_SMD:L_0603_1608Metric, F.Cu at (83.1, 233.7)
- added L9: 2.2mh, Inductor_SMD:L_0603_1608Metric, F.Cu at (83.1, 236.2)
- added P1: 5104338-1, BCRL_power_supply:TE_5104338-1, F.Cu at (174.9, 39.9)
- added P2: 5104338-1, BCRL_power_supply:TE_5104338-1, F.Cu at (174.9, 50.6)
- added P3: 5104338-1, BCRL_power_supply:TE_5104338-1, F.Cu at (174.9, 61.3)
- added P4: 5104338-1, BCRL_power_supply:TE_5104338-1, F.Cu at (174.9, 72.0)
- added P5: 5104338-1, BCRL_power_supply:TE_5104338-1, F.Cu at (121.8, 39.9)
- added P6: 5104338-1, BCRL_power_supply:TE_5104338-1, F.Cu at (121.8, 50.6)
- added P7: 5104338-1, BCRL_power_supply:TE_5104338-1, F.Cu at (121.8, 61.3)
- added P8: 5104338-1, BCRL_power_supply:TE_5104338-1, F.Cu at (121.8, 72.0)
- added PS1: EHHD010A0B41-HZ, BCRL_power_supply:CONV_EHHD010A0B41-HZ, F.Cu at (214.3, 40.8)
- added PS10: PQC50-48-S5-O, BCRL_power_supply:CONV_PQC50-48-S5-O, F.Cu at (206.7, 95.8)
- added PS11: PQC50-48-S5-O, BCRL_power_supply:CONV_PQC50-48-S5-O, F.Cu at (95.0, 95.8)
- added PS12: PQC50-48-S5-O, BCRL_power_supply:CONV_PQC50-48-S5-O, F.Cu at (132.3, 134.8)
- added PS13: PQC50-48-S5-O, BCRL_power_supply:CONV_PQC50-48-S5-O, F.Cu at (95.0, 173.7)
- added PS14: PQC50-48-S5-O, BCRL_power_supply:CONV_PQC50-48-S5-O, F.Cu at (132.3, 95.8)
- added PS15: PQC50-48-S5-O, BCRL_power_supply:CONV_PQC50-48-S5-O, F.Cu at (206.7, 134.8)
- added PS16: PQC50-48-S5-O, BCRL_power_supply:CONV_PQC50-48-S5-O, F.Cu at (169.5, 173.7)
- added PS17: PQC50-48-S5-O, BCRL_power_supply:CONV_PQC50-48-S5-O, F.Cu at (244.0, 95.8)
- added PS18: PQC50-48-S5-O, BCRL_power_supply:CONV_PQC50-48-S5-O, F.Cu at (169.5, 95.8)
- added PS2: PQC50-48-S5-O, BCRL_power_supply:CONV_PQC50-48-S5-O, F.Cu at (132.3, 212.7)
- added PS3: PQC50-48-S5-O, BCRL_power_supply:CONV_PQC50-48-S5-O, F.Cu at (132.3, 173.7)
- added PS4: PQC50-48-S5-O, BCRL_power_supply:CONV_PQC50-48-S5-O, F.Cu at (95.0, 212.7)
- added PS5: PQC50-48-S5-O, BCRL_power_supply:CONV_PQC50-48-S5-O, F.Cu at (95.0, 134.8)
- added PS6: EHHD010A0B41-HZ, BCRL_power_supply:CONV_EHHD010A0B41-HZ, F.Cu at (214.3, 67.1)
- added PS7: PQC50-48-S5-O, BCRL_power_supply:CONV_PQC50-48-S5-O, F.Cu at (264.2, 40.8)
- added PS8: PQC50-48-S5-O, BCRL_power_supply:CONV_PQC50-48-S5-O, F.Cu at (169.5, 212.7)
- added PS9: PQC50-48-S5-O, BCRL_power_supply:CONV_PQC50-48-S5-O, F.Cu at (169.5, 134.8)
- added R1: 1k, Resistor_SMD:R_0603_1608Metric, F.Cu at (147.5, 62.1)
- added R10: 3.4k, Resistor_SMD:R_0603_1608Metric, F.Cu at (250.7, 231.0)
- added R11: 3.4k, Resistor_SMD:R_0603_1608Metric, F.Cu at (283.7, 200.7)
- added R12: R, Resistor_SMD:R_0603_1608Metric, F.Cu at (124.3, 226.2)
- added R13: R, Resistor_SMD:R_0603_1608Metric, F.Cu at (124.3, 228.7)
- added R14: R, Resistor_SMD:R_0603_1608Metric, F.Cu at (124.3, 231.2)
- added R15: R, Resistor_SMD:R_0603_1608Metric, F.Cu at (124.3, 187.2)
- added R16: R, Resistor_SMD:R_0603_1608Metric, F.Cu at (124.3, 189.7)
- added R17: R, Resistor_SMD:R_0603_1608Metric, F.Cu at (124.3, 192.2)
- added R18: R, Resistor_SMD:R_0603_1608Metric, F.Cu at (87.1, 226.2)
- added R19: R, Resistor_SMD:R_0603_1608Metric, F.Cu at (87.1, 228.7)
- added R2: 1k, Resistor_SMD:R_0603_1608Metric, F.Cu at (147.5, 64.7)
- added R20: R, Resistor_SMD:R_0603_1608Metric, F.Cu at (87.1, 231.2)
- added R21: R, Resistor_SMD:R_0603_1608Metric, F.Cu at (87.1, 148.2)
- added R22: R, Resistor_SMD:R_0603_1608Metric, F.Cu at (87.1, 150.8)
- added R23: R, Resistor_SMD:R_0603_1608Metric, F.Cu at (87.1, 153.3)
- added R24: 1k, Resistor_SMD:R_0603_1608Metric, F.Cu at (94.4, 62.1)
- added R25: 1k, Resistor_SMD:R_0603_1608Metric, F.Cu at (94.4, 64.7)
- added R26: 1k, Resistor_SMD:R_0603_1608Metric, F.Cu at (94.4, 67.2)
- added R27: 1k, Resistor_SMD:R_0603_1608Metric, F.Cu at (94.4, 69.7)
- added R28: 1k, Resistor_SMD:R_0603_1608Metric, F.Cu at (94.4, 72.2)
- added R29: 1k, Resistor_SMD:R_0603_1608Metric, F.Cu at (94.4, 74.7)
- added R3: 1k, Resistor_SMD:R_0603_1608Metric, F.Cu at (147.5, 67.2)
- added R30: 1k, Resistor_SMD:R_0603_1608Metric, F.Cu at (94.4, 77.2)
- added R31: 1k, Resistor_SMD:R_0603_1608Metric, F.Cu at (94.4, 79.7)
- added R32: 3.4k, Resistor_SMD:R_0603_1608Metric, F.Cu at (250.7, 170.3)
- added R33: R, Resistor_SMD:R_0603_1608Metric, F.Cu at (256.3, 54.3)
- added R34: R, Resistor_SMD:R_0603_1608Metric, F.Cu at (256.3, 56.8)
- added R35: R, Resistor_SMD:R_0603_1608Metric, F.Cu at (256.3, 59.3)
- added R36: R, Resistor_SMD:R_0603_1608Metric, F.Cu at (161.6, 226.2)
- added R37: R, Resistor_SMD:R_0603_1608Metric, F.Cu at (161.6, 228.7)
- added R38: R, Resistor_SMD:R_0603_1608Metric, F.Cu at (161.6, 231.2)
- added R39: R, Resistor_SMD:R_0603_1608Metric, F.Cu at (161.6, 148.2)
- added R4: 1k, Resistor_SMD:R_0603_1608Metric, F.Cu at (147.5, 69.7)
- added R40: R, Resistor_SMD:R_0603_1608Metric, F.Cu at (161.6, 150.8)
- added R41: R, Resistor_SMD:R_0603_1608Metric, F.Cu at (161.6, 153.3)
- added R42: R, Resistor_SMD:R_0603_1608Metric, F.Cu at (198.8, 109.3)
- added R43: R, Resistor_SMD:R_0603_1608Metric, F.Cu at (198.8, 111.8)
- added R44: R, Resistor_SMD:R_0603_1608Metric, F.Cu at (198.8, 114.3)
- added R45: R, Resistor_SMD:R_0603_1608Metric, F.Cu at (87.1, 109.3)
- added R46: R, Resistor_SMD:R_0603_1608Metric, F.Cu at (87.1, 111.8)
- added R47: R, Resistor_SMD:R_0603_1608Metric, F.Cu at (87.1, 114.3)
- added R48: R, Resistor_SMD:R_0603_1608Metric, F.Cu at (124.3, 148.2)
- added R49: R, Resistor_SMD:R_0603_1608Metric, F.Cu at (124.3, 150.8)
- added R5: 1k, Resistor_SMD:R_0603_1608Metric, F.Cu at (147.5, 72.2)
- added R50: R, Resistor_SMD:R_0603_1608Metric, F.Cu at (124.3, 153.3)
- added R51: 3.4k, Resistor_SMD:R_0603_1608Metric, F.Cu at (217.7, 200.7)
- added R52: R, Resistor_SMD:R_0603_1608Metric, F.Cu at (87.1, 187.2)
- added R53: R, Resistor_SMD:R_0603_1608Metric, F.Cu at (87.1, 189.7)
- added R54: R, Resistor_SMD:R_0603_1608Metric, F.Cu at (87.1, 192.2)
- added R55: R, Resistor_SMD:R_0603_1608Metric, F.Cu at (124.3, 109.3)
- added R56: R, Resistor_SMD:R_0603_1608Metric, F.Cu at (124.3, 111.8)
- added R57: R, Resistor_SMD:R_0603_1608Metric, F.Cu at (124.3, 114.3)
- added R58: 3.4k, Resistor_SMD:R_0603_1608Metric, F.Cu at (217.7, 231.0)
- added R59: 3.4k, Resistor_SMD:R_0603_1608Metric, F.Cu at (250.7, 200.7)
- added R6: 1k, Resistor_SMD:R_0603_1608Metric, F.Cu at (147.5, 74.7)
- added R60: R, Resistor_SMD:R_0603_1608Metric, F.Cu at (198.8, 148.2)
- added R61: R, Resistor_SMD:R_0603_1608Metric, F.Cu at (198.8, 150.8)
- added R62: R, Resistor_SMD:R_0603_1608Metric, F.Cu at (198.8, 153.3)
- added R63: R, Resistor_SMD:R_0603_1608Metric, F.Cu at (161.6, 187.2)
- added R64: R, Resistor_SMD:R_0603_1608Metric, F.Cu at (161.6, 189.7)
- added R65: R, Resistor_SMD:R_0603_1608Metric, F.Cu at (161.6, 192.2)
- added R66: R, Resistor_SMD:R_0603_1608Metric, F.Cu at (236.0, 109.3)
- added R67: R, Resistor_SMD:R_0603_1608Metric, F.Cu at (236.0, 111.8)
- added R68: R, Resistor_SMD:R_0603_1608Metric, F.Cu at (236.0, 114.3)
- added R69: R, Resistor_SMD:R_0603_1608Metric, F.Cu at (161.6, 109.3)
- added R7: 1k, Resistor_SMD:R_0603_1608Metric, F.Cu at (147.5, 77.2)
- added R70: R, Resistor_SMD:R_0603_1608Metric, F.Cu at (161.6, 111.8)
- added R71: R, Resistor_SMD:R_0603_1608Metric, F.Cu at (161.6, 114.3)
- added R72: 3.4k, Resistor_SMD:R_0603_1608Metric, F.Cu at (217.7, 170.3)
- added R8: 1k, Resistor_SMD:R_0603_1608Metric, F.Cu at (147.5, 79.7)
- added R9: 3.4k, Resistor_SMD:R_0603_1608Metric, F.Cu at (283.7, 170.3)
- added U1: PDQ10-Q48-S5-D, BCRL_power_supply:CONV_PDQ10-Q48-S5-D, F.Cu at (268.2, 176.4)
- added U2: PDQ10-Q48-S5-D, BCRL_power_supply:CONV_PDQ10-Q48-S5-D, F.Cu at (235.2, 237.1)
- added U3: PDQ10-Q48-S3-D, BCRL_power_supply:CONV_PDQ10-Q48-S3-D, F.Cu at (239.5, 137.4)
- added U4: PDQ10-Q48-S5-D, BCRL_power_supply:CONV_PDQ10-Q48-S5-D, F.Cu at (268.2, 206.7)
- added U5: PDQ10-Q48-S5-D, BCRL_power_supply:CONV_PDQ10-Q48-S5-D, F.Cu at (235.2, 176.4)
- added U6: PDQ10-Q48-S5-D, BCRL_power_supply:CONV_PDQ10-Q48-S5-D, F.Cu at (202.3, 206.7)
- added U7: PDQ10-Q48-S5-D, BCRL_power_supply:CONV_PDQ10-Q48-S5-D, F.Cu at (202.3, 237.1)
- added U8: PDQ10-Q48-S5-D, BCRL_power_supply:CONV_PDQ10-Q48-S5-D, F.Cu at (235.2, 206.7)
- added U9: PDQ10-Q48-S5-D, BCRL_power_supply:CONV_PDQ10-Q48-S5-D, F.Cu at (202.3, 176.4)
