File: kicad_files/bcrl_power_supply/bcrl_power_supply.kicad_pcb (KiCad board)
At the start: 2 copper layers, 377 parts, among them J1 OSTVN02A150, J10 OSTVN02A150, J11 OSTVN02A150, J12 OSTVN02A150, J13 Conn_01x02, J14 Conn_01x02, J15 Conn_01x02, J16 Conn_01x02, J17 Conn_01x02, J18 Conn_01x02, J19 Conn_01x02, J2 OSTVN02A150, J20 Conn_01x02, J21 5034801600, J22 5034801600, J23 5034801600, J24 OSTVN02A150, J25 OSTVN02A150, J26 OSTVN02A150, J27 OSTVN02A150, J28 OSTVN02A150, J29 OSTVN02A150, J3 Conn_01x02, J30 OSTVN02A150, J31 OSTVN02A150, J32 OSTVN02A150, J33 Conn_01x02, J34 Conn_01x02, J35 Conn_01x02, J36 Conn_01x02, J37 Conn_01x02, J38 Conn_01x02, J39 Conn_01x02, J4 OSTVN02A150, J40 Conn_01x02, J41 5034801600, J42 5034801600, J43 Conn_01x04_Pin, J44 Conn_01x04_Pin, J45 Conn_01x04_Pin, J46 Conn_01x04_Pin, J47 Conn_01x04_Pin, J48 Conn_01x04_Pin, J49 Conn_01x04_Pin, J5 OSTVN02A150, J50 Conn_01x04_Pin, J51 Conn_01x04_Pin, J52 Conn_01x04_Pin, J53 Conn_01x04_Pin, J54 Conn_01x04_Pin, J55 Conn_01x04_Pin, J56 Conn_01x04_Pin, J57 Conn_01x04_Pin, J58 Conn_01x04_Pin, J59 Conn_01x06_Pin, J6 OSTVN02A150, J60 Conn_01x06_Pin, J61 Conn_01x06_Pin, J62 Conn_01x06_Pin, J63 Conn_01x04_Pin, J64 Conn_01x04_Pin, J65 Conn_01x06_Pin, J66 Conn_01x06_Pin, J67 Conn_01x06_Pin, J68 Conn_01x06_Pin, J7 OSTVN02A150, J8 OSTVN02A150, J9 OSTVN02A150, P1 5104338-1, P2 5104338-1, P3 5104338-1, P4 5104338-1, P5 5104338-1, P6 5104338-1, P7 5104338-1, P8 5104338-1, U1 PDQ10-Q48-S5-D, U2 PDQ10-Q48-S5-D, U3 PDQ10-Q48-S3-D, U4 PDQ10-Q48-S5-D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

Commit message: ...
Parts:
- removed PS1, PS6: EHHD010A0B41-HZ, BCRL_power_supply:CONV_EHHD010A0B41-HZ
- removed R14, R15, R16, R17, R18, R19, R20, R21, R22, R23, R37, R38, R39, R40, R41, R42, R43, R44, R45, R46, R47, R48, R49, R50, R52, R53, R54, R56, R57, R60, R61, R64, R65, R66, R67, R68, R69, R70, R71: R, Resistor_SMD:R_0603_1608Metric
- removed R51, R58, R59, R72: 3.4k, Resistor_SMD:R_0603_1608Metric
- added C147: 4.7uf/100v, Capacitor_SMD:C_0603_1608Metric, F.Cu at (290.9, 203.9)
- added C148: 330uf/100v, Capacitor_SMD:C_0603_1608Metric, F.Cu at (290.9, 206.4)
- added C149: 1nf/2kv, Capacitor_SMD:C_0603_1608Metric, F.Cu at (290.9, 208.9)
- added C150: 1nf/2kv, Capacitor_SMD:C_0603_1608Metric, F.Cu at (290.9, 211.4)
- added C151: 47uf/50v, Capacitor_SMD:C_0603_1608Metric, F.Cu at (290.9, 213.9)
- added C152: 680uf/100v, Capacitor_SMD:C_0603_1608Metric, F.Cu at (215.6, 126.7)
- added C153: 4.7uf/100v, Capacitor_SMD:C_0603_1608Metric, F.Cu at (218.1, 126.7)
- added C154: 4.7uf/100v, Capacitor_SMD:C_0603_1608Metric, F.Cu at (220.6, 126.7)
- added C155: 4.7uf/100v, Capacitor_SMD:C_0603_1608Metric, F.Cu at (223.1, 126.7)
- added C156: 4.7uf/100v, Capacitor_SMD:C_0603_1608Metric, F.Cu at (225.7, 126.7)
- added C157: 2.2nf/400vac, Capacitor_SMD:C_0603_1608Metric, F.Cu at (228.2, 126.7)
- added C158: 2.2nf/400vac, Capacitor_SMD:C_0603_1608Metric, F.Cu at (213.1, 122.7)
- added C159: 330uf/63v, Capacitor_SMD:C_0603_1608Metric, F.Cu at (215.6, 122.7)
- added C160: 4.7uf/100v, Capacitor_SMD:C_0603_1608Metric, F.Cu at (310.8, 261.4)
- added C161: 4.7uf/100v, Capacitor_SMD:C_0603_1608Metric, F.Cu at (306.8, 291.5)
- added C162: 330uf/100v, Capacitor_SMD:C_0603_1608Metric, F.Cu at (223.6, 214.3)
- added C163: 4.7uf/100v, Capacitor_SMD:C_0603_1608Metric, F.Cu at (223.6, 216.8)
- added C164: 4.7uf/100v, Capacitor_SMD:C_0603_1608Metric, F.Cu at (227.7, 204.2)
- added C165: 330uf/100v, Capacitor_SMD:C_0603_1608Metric, F.Cu at (227.7, 206.7)
- added C166: 1nf/2kv, Capacitor_SMD:C_0603_1608Metric, F.Cu at (227.7, 209.2)
- added C167: 1nf/2kv, Capacitor_SMD:C_0603_1608Metric, F.Cu at (227.7, 211.8)
- added C168: 47uf/50v, Capacitor_SMD:C_0603_1608Metric, F.Cu at (227.7, 214.3)
- added C169: 4.7uf/100v, Capacitor_SMD:C_0603_1608Metric, F.Cu at (120.4, 210.5)
- added C170: 4.7uf/100v, Capacitor_SMD:C_0603_1608Metric, F.Cu at (120.4, 213.0)
- added C171: 4.7uf/100v, Capacitor_SMD:C_0603_1608Metric, F.Cu at (118.5, 155.6)
- added C172: 4.7uf/100v, Capacitor_SMD:C_0603_1608Metric, F.Cu at (118.5, 158.1)
- added H1: MountingHole, MountingHole:MountingHole_3.5mm_Pad, F.Cu at (396.9, 103.3)
- added H2: MountingHole, MountingHole:MountingHole_3.5mm_Pad, F.Cu at (544.5, 103.3)
- added H3: MountingHole, MountingHole:MountingHole_3.5mm_Pad, F.Cu at (396.9, 315.3)
- added H4: MountingHole, MountingHole:MountingHole_3.5mm_Pad, F.Cu at (544.5, 315.3)
- added H5: MountingHole, MountingHole:MountingHole_3.5mm_Pad, F.Cu at (396.7, 209.1)
- added H6: MountingHole, MountingHole:MountingHole_3.5mm_Pad, F.Cu at (544.4, 209.1)
- added J69: Conn_01x02, Connector_PinHeader_2.54mm:PinHeader_1x02_P2.54mm_Vertical, F.Cu at (120.7, 230.0)
- added J70: Conn_01x02, Connector_PinHeader_2.54mm:PinHeader_1x02_P2.54mm_Vertical, F.Cu at (118.8, 175.1)
- added L41: 2.2mh, Inductor_SMD:L_0603_1608Metric, F.Cu at (244.3, 66.2)
- added L42: 4.7uh/3.1a, Inductor_SMD:L_0603_1608Metric, F.Cu at (295.0, 206.4)
- added L43: 2.2mh, Inductor_SMD:L_0603_1608Metric, F.Cu at (223.1, 122.7)
- added L44: 2.2mh, Inductor_SMD:L_0603_1608Metric, F.Cu at (225.7, 122.7)
- added L45: 4.7uh/3.1a, Inductor_SMD:L_0603_1608Metric, F.Cu at (306.8, 261.4)
- added L46: 4.7uh/3.1a, Inductor_SMD:L_0603_1608Metric, F.Cu at (231.7, 206.7)
- added L47: 4.7uh/3.1a, Inductor_SMD:L_0603_1608Metric, F.Cu at (120.4, 215.5)
- added L48: 4.7uh/3.1a, Inductor_SMD:L_0603_1608Metric, F.Cu at (118.5, 160.6)
- added PS19: PQC50-48-S5-O, BCRL_power_supply:CONV_PQC50-48-S5-O, F.Cu at (213.4, 150.0)
- added PS20: PDQE15-Q48-D24-D, BCRL_power_supply:CONV_PDQE15-Q48-D24-D, F.Cu at (189.6, 216.4)
- added R76: 3.4k, Resistor_SMD:R_0603_1608Metric, F.Cu at (298.7, 266.4)
- added RV1: R_Potentiometer_Trim, Potentiometer_THT:Potentiometer_ACP_CA9-V10_Vertical, F.Cu at (211.7, 275.6)
- added RV10: R_Potentiometer_Trim, Potentiometer_THT:Potentiometer_ACP_CA9-V10_Vertical, F.Cu at (332.8, 323.2)
- added RV11: R_Potentiometer_Trim, Potentiometer_THT:Potentiometer_ACP_CA9-V10_Vertical, F.Cu at (332.8, 311.8)
- added RV12: R_Potentiometer_Trim, Potentiometer_THT:Potentiometer_ACP_CA9-V10_Vertical, F.Cu at (332.8, 300.4)
- added RV13: R_Potentiometer_Trim, Potentiometer_THT:Potentiometer_ACP_CA9-V10_Vertical, F.Cu at (259.9, 130.2)
- added RV14: R_Potentiometer_Trim, Potentiometer_THT:Potentiometer_ACP_CA9-V10_Vertical, F.Cu at (289.6, 71.2)
- added RV15: R_Potentiometer_Trim, Potentiometer_THT:Potentiometer_ACP_CA9-V10_Vertical, F.Cu at (215.0, 74.2)
- added RV16: R_Potentiometer_Trim, Potentiometer_THT:Potentiometer_ACP_CA9-V10_Vertical, F.Cu at (196.4, 130.7)
- added RV2: R_Potentiometer_Trim, Potentiometer_THT:Potentiometer_ACP_CA9-V10_Vertical, F.Cu at (211.7, 287.0)
- added RV3: R_Potentiometer_Trim, Potentiometer_THT:Potentiometer_ACP_CA9-V10_Vertical, F.Cu at (211.7, 298.4)
- added RV4: R_Potentiometer_Trim, Potentiometer_THT:Potentiometer_ACP_CA9-V10_Vertical, F.Cu at (211.7, 309.8)
- added RV5: R_Potentiometer_Trim, Potentiometer_THT:Potentiometer_ACP_CA9-V10_Vertical, F.Cu at (248.5, 130.2)
- added RV6: R_Potentiometer_Trim, Potentiometer_THT:Potentiometer_ACP_CA9-V10_Vertical, F.Cu at (278.2, 71.2)
- added RV7: R_Potentiometer_Trim, Potentiometer_THT:Potentiometer_ACP_CA9-V10_Vertical, F.Cu at (203.6, 74.2)
- added RV8: R_Potentiometer_Trim, Potentiometer_THT:Potentiometer_ACP_CA9-V10_Vertical, F.Cu at (185.0, 130.7)
- added RV9: R_Potentiometer_Trim, Potentiometer_THT:Potentiometer_ACP_CA9-V10_Vertical, F.Cu at (332.8, 334.6)
- added U10: PDQ10-Q48-S5-D, BCRL_power_supply:CONV_PDQ10-Q48-S5-D, F.Cu at (329.5, 356.2)
- added U11: PDQ10-Q48-S5-D, BCRL_power_supply:CONV_PDQ10-Q48-S5-D, F.Cu at (302.6, 356.2)
- added U12: PDQ10-Q48-S5-D, BCRL_power_supply:CONV_PDQ10-Q48-S5-D, F.Cu at (268.9, 254.0)
- added U13: PDQ10-Q48-S5-D, BCRL_power_supply:CONV_PDQ10-Q48-S5-D, F.Cu at (275.6, 356.2)
- added U14: PDQ10-Q48-S5-D, BCRL_power_supply:CONV_PDQ10-Q48-S5-D, F.Cu at (104.9, 224.1)
- added U15: PDQ10-Q48-S5-D, BCRL_power_supply:CONV_PDQ10-Q48-S5-D, F.Cu at (103.0, 169.2)
- C100, C120, C50: value 330uf/63v -> 4.7uf/100v
- C109, C91: value 4.7uf/100v -> 680uf/100v
- C113, C43, C93: value 680uf/100v -> 4.7uf/100v
- C114, C115, C96, C97: value 4.7uf/100v -> 2.2nf/400vac
- C116: value 4.7uf/100v -> 330uf/63v
- C118, C119, C48, C49, C99: value 2.2nf/400vac -> 4.7uf/100v
- C145: value 4.7uf/100v -> 330uf/100v
- C98: value 2.2nf/400vac -> 330uf/63v
- J12: value OSTVN02A150 -> 5034801600; footprint BCRL_power_supply:CONN_OSTVN02A150_OST -> BCRL_power_supply:MOLEX_5034801600
- J23: value 5034801600 -> OSTVN02A150; footprint BCRL_power_supply:MOLEX_5034801600 -> BCRL_power_supply:CONN_OSTVN02A150_OST
- J59, J60: value Conn_01x06_Pin -> Conn_01x04_Pin; footprint Connector_PinHeader_2.54mm:PinHeader_1x06_P2.54mm_Vertical -> Connector_PinHeader_2.54mm:PinHeader_1x04_P2.54mm_Vertical
- J63, J64: value Conn_01x04_Pin -> Conn_01x06_Pin; footprint Connector_PinHeader_2.54mm:PinHeader_1x04_P2.54mm_Vertical -> Connector_PinHeader_2.54mm:PinHeader_1x06_P2.54mm_Vertical
- L13, L14, L15, L16, L29, L34, L35: value 2.2mh -> 4.7uh/3.1a
- L25, L30, L31, L40: value 4.7uh/3.1a -> 2.2mh
- PS18: value PQC50-48-S5-O -> PDQE15-Q48-D24-D; footprint BCRL_power_supply:CONV_PQC50-48-S5-O -> BCRL_power_supply:CONV_PDQE15-Q48-D24-D
- R12, R13, R33, R34, R35, R36, R55, R62, R63: value R -> 3.4k
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Connections:
- net Net-(PS2-VIN) renamed /TxRFswMUXv1 board/PQC50-48-S5-O_EMC_trimmed_1/VIN
- net Net-(PS3-VIN) renamed /TxRFswMUXv1 board/PQC50-48-S5-O_EMC_trimmed_2/VIN
- net Net-(PS4-VIN) renamed /TxRFswMUXv1 board/PQC50-48-S5-O_EMC_trimmed_3/VIN
- net Net-(PS5-VIN) renamed /TxRFswMUXv1 board/PQC50-48-S5-O_EMC_trimmed_4/VIN
- net Net-(U1-+VIN) renamed /TxRFswMUXv1 board/PDQ10-Q48-S5-D_EMC_2/VIN
- net Net-(U2-+VIN) renamed /TxRFswMUXv1 board/PDQ10-Q48-S5-D_EMC_3/VIN
- net Net-(U4-+VIN) renamed /TxRFswMUXv1 board/PDQ10-Q48-S5-D_EMC_4/VIN
- net Net-(U5-+VIN) renamed /Tx_RPi4_HAT_board/PDQ10-Q48-S5-D_EMC_8/VIN
- C100 pad 1: GND -> /RxRFswMUXv1 board/PDQ10-Q48-S5-D_EMC_12/VIN
- C104 pad 1: Net-(PS14-VIN) -> /RxRFswMUXv1 board/PQC50-48-S5-O_EMC_trimmed_14/VIN
- C104 pad 2: Net-(PS14-GND) -> Net-(PS13-GND)
- C105 pad 1: Net-(PS14-VIN) -> /RxRFswMUXv1 board/PQC50-48-S5-O_EMC_trimmed_14/VIN
- C105 pad 2: Net-(PS14-GND) -> Net-(PS13-GND)
- C106 pad 1: Net-(PS14-VIN) -> /RxRFswMUXv1 board/PQC50-48-S5-O_EMC_trimmed_14/VIN
- C106 pad 2: GND -> /RxRFswMUXv1 board/+8V_3
- C107 pad 1: Net-(PS14-GND) -> Net-(PS13-GND)
- C108 pad 1: GND -> /RxRFswMUXv1 board/+8V_3
- C110 pad 1: Net-(U7-+VIN) -> 48V
- C112 pad 1: Net-(U8-+VIN) -> /RxRFswMUXv1 board/PQC50-48-S5-O_EMC_trimmed_11/VIN
- C112 pad 2: GND -> Net-(PS14-GND)
- C113 pad 1: 48V -> /RxRFswMUXv1 board/PQC50-48-S5-O_EMC_trimmed_11/VIN
- C113 pad 2: GND -> Net-(PS14-GND)
- C114 pad 1: 48V -> /RxRFswMUXv1 board/PQC50-48-S5-O_EMC_trimmed_11/VIN
- C114 pad 2: GND -> /RxRFswMUXv1 board/+8V_4
- C115 pad 1: 48V -> Net-(PS14-GND)
- C116 pad 1: Net-(PS15-VIN) -> /RxRFswMUXv1 board/+8V_4
- C116 pad 2: Net-(PS15-GND) -> GND
- C117 pad 1: Net-(PS15-VIN) -> 48V
- C117 pad 2: Net-(PS15-GND) -> GND
- C118 pad 1: Net-(PS15-VIN) -> /RxRFswMUXv1 board/PDQ10-Q48-S5-D_EMC_9/VIN
- C119 pad 1: Net-(PS15-GND) -> 48V
- C120 pad 1: GND -> /TxRFswMUXv1 board/PDQ10-Q48-S5-D_EMC_1/VIN
- C124 pad 1: Net-(PS16-VIN) -> /TxBFN-16C/PQC50-48-S5-O_EMC_trimmed_9/VIN
- C124 pad 2: Net-(PS16-GND) -> Net-(PS15-GND)
- C125 pad 1: Net-(PS16-VIN) -> /TxBFN-16C/PQC50-48-S5-O_EMC_trimmed_9/VIN
- C125 pad 2: Net-(PS16-GND) -> Net-(PS15-GND)
- C126 pad 1: Net-(PS16-VIN) -> /TxBFN-16C/PQC50-48-S5-O_EMC_trimmed_9/VIN
- C126 pad 2: GND -> /TxBFN-16C/+6.5V_1
- C127 pad 1: Net-(PS16-GND) -> Net-(PS15-GND)
- C128 pad 1: GND -> /TxBFN-16C/+6.5V_1
- C132 pad 1: Net-(PS17-VIN) -> /TxBFN-16F/PQC50-48-S5-O_EMC_trimmed_9/VIN
- C132 pad 2: Net-(PS17-GND) -> Net-(PS16-GND)
- C133 pad 1: Net-(PS17-VIN) -> /TxBFN-16F/PQC50-48-S5-O_EMC_trimmed_9/VIN
- C133 pad 2: Net-(PS17-GND) -> Net-(PS16-GND)
- C134 pad 1: Net-(PS17-VIN) -> /TxBFN-16F/PQC50-48-S5-O_EMC_trimmed_9/VIN
- C134 pad 2: GND -> /TxBFN-16F/+6.5V_1
- C135 pad 1: Net-(PS17-GND) -> Net-(PS16-GND)
- C136 pad 1: GND -> /TxBFN-16F/+6.5V_1
- C14 pad 2: GND -> /TxRFswMUXv1 board/+8V_1
- C140 pad 1: Net-(PS18-VIN) -> /RxBFN-16F/PQC50-48-S5-O_EMC_trimmed_9/VIN
- C140 pad 2: Net-(PS18-GND) -> Net-(PS17-GND)
- C141 pad 1: Net-(PS18-VIN) -> /RxBFN-16F/PQC50-48-S5-O_EMC_trimmed_9/VIN
- C141 pad 2: Net-(PS18-GND) -> Net-(PS17-GND)
- C142 pad 1: Net-(PS18-VIN) -> /RxBFN-16F/PQC50-48-S5-O_EMC_trimmed_9/VIN
- C142 pad 2: GND -> /RxBFN-16F/+6.5V_1
- C143 pad 1: Net-(PS18-GND) -> Net-(PS17-GND)
- C144 pad 1: GND -> /RxBFN-16F/+6.5V_1
- C146 pad 1: Net-(U9-+VIN) -> 48V
- C16 pad 1: GND -> /TxRFswMUXv1 board/+8V_1
- C22 pad 2: GND -> /TxRFswMUXv1 board/+8V_2
- C24 pad 1: GND -> /TxRFswMUXv1 board/+8V_2
- C30 pad 2: GND -> /TxRFswMUXv1 board/+8V_3
- C32 pad 1: GND -> /TxRFswMUXv1 board/+8V_3
- C38 pad 2: GND -> /TxRFswMUXv1 board/+8V_4
- C40 pad 1: GND -> /TxRFswMUXv1 board/+8V_4
- C44 pad 1: 48V -> /Tx_RPi4_HAT_board/PDQ10-Q48-S5-D_EMC_7/VIN
- C46 pad 1: Net-(PS7-VIN) -> /Rx_RPi4_HAT_board/PDQ10-Q48-S5-D_EMC_7/VIN
- C46 pad 2: Net-(PS7-GND) -> GND
- C47 pad 1: Net-(PS7-VIN) -> 48V
- C47 pad 2: Net-(PS7-GND) -> GND
- C48 pad 1: Net-(PS7-VIN) -> /Rx_RPi4_HAT_board/PDQ10-Q48-S5-D_EMC_8/VIN
- C49 pad 1: Net-(PS7-GND) -> 48V
- C50 pad 1: GND -> /RxRFswMUXv1 board/PDQ10-Q48-S5-D_EMC_10/VIN
- C54 pad 1: Net-(PS8-VIN) -> /TxBFN-16C/PQC50-48-S5-O_EMC_trimmed_10/VIN
- C54 pad 2: Net-(PS8-GND) -> Net-(PS7-GND)
- C55 pad 1: Net-(PS8-VIN) -> /TxBFN-16C/PQC50-48-S5-O_EMC_trimmed_10/VIN
- C55 pad 2: Net-(PS8-GND) -> Net-(PS7-GND)
- C56 pad 1: Net-(PS8-VIN) -> /TxBFN-16C/PQC50-48-S5-O_EMC_trimmed_10/VIN
- C56 pad 2: GND -> /TxBFN-16C/+6.5V_2
- C57 pad 1: Net-(PS8-GND) -> Net-(PS7-GND)
- C58 pad 1: GND -> /TxBFN-16C/+6.5V_2
- C62 pad 1: Net-(PS9-VIN) -> /TxBFN-16F/PQC50-48-S5-O_EMC_trimmed_10/VIN
- C62 pad 2: Net-(PS9-GND) -> Net-(PS8-GND)
- C63 pad 1: Net-(PS9-VIN) -> /TxBFN-16F/PQC50-48-S5-O_EMC_trimmed_10/VIN
- C63 pad 2: Net-(PS9-GND) -> Net-(PS8-GND)
- C64 pad 1: Net-(PS9-VIN) -> /TxBFN-16F/PQC50-48-S5-O_EMC_trimmed_10/VIN
- C64 pad 2: GND -> /TxBFN-16F/+6.5V_2
- C65 pad 1: Net-(PS9-GND) -> Net-(PS8-GND)
- C66 pad 1: GND -> /TxBFN-16F/+6.5V_2
- C70 pad 1: Net-(PS10-VIN) -> /RxBFN-16F/PQC50-48-S5-O_EMC_trimmed_10/VIN
- C70 pad 2: Net-(PS10-GND) -> Net-(PS9-GND)
- C71 pad 1: Net-(PS10-VIN) -> /RxBFN-16F/PQC50-48-S5-O_EMC_trimmed_10/VIN
- C71 pad 2: Net-(PS10-GND) -> Net-(PS9-GND)
- C72 pad 1: Net-(PS10-VIN) -> /RxBFN-16F/PQC50-48-S5-O_EMC_trimmed_10/VIN
- C72 pad 2: GND -> /RxBFN-16F/+6.5V_2
- C73 pad 1: Net-(PS10-GND) -> Net-(PS9-GND)
- C74 pad 1: GND -> /RxBFN-16F/+6.5V_2
- C78 pad 1: Net-(PS11-VIN) -> /RxBFN-16C/PQC50-48-S5-O_EMC_trimmed_10/VIN
- C78 pad 2: Net-(PS11-GND) -> Net-(PS10-GND)
- C79 pad 1: Net-(PS11-VIN) -> /RxBFN-16C/PQC50-48-S5-O_EMC_trimmed_10/VIN
- C79 pad 2: Net-(PS11-GND) -> Net-(PS10-GND)
- C80 pad 1: Net-(PS11-VIN) -> /RxBFN-16C/PQC50-48-S5-O_EMC_trimmed_10/VIN
- C80 pad 2: GND -> /RxBFN-16C/+6.5V_2
- C81 pad 1: Net-(PS11-GND) -> Net-(PS10-GND)
- C82 pad 1: GND -> /RxBFN-16C/+6.5V_2
- C86 pad 1: Net-(PS12-VIN) -> /RxRFswMUXv1 board/PQC50-48-S5-O_EMC_trimmed_13/VIN
- C86 pad 2: Net-(PS12-GND) -> Net-(PS11-GND)
- C87 pad 1: Net-(PS12-VIN) -> /RxRFswMUXv1 board/PQC50-48-S5-O_EMC_trimmed_13/VIN
- C87 pad 2: Net-(PS12-GND) -> Net-(PS11-GND)
- C88 pad 1: Net-(PS12-VIN) -> /RxRFswMUXv1 board/PQC50-48-S5-O_EMC_trimmed_13/VIN
- C88 pad 2: GND -> /RxRFswMUXv1 board/+8V_2
- C89 pad 1: Net-(PS12-GND) -> Net-(PS11-GND)
- C90 pad 1: GND -> /RxRFswMUXv1 board/+8V_2
- C92 pad 1: Net-(U6-+VIN) -> 48V
- C94 pad 1: 48V -> /RxRFswMUXv1 board/PQC50-48-S5-O_EMC_trimmed_12/VIN
- C94 pad 2: GND -> Net-(PS12-GND)
- C95 pad 1: 48V -> /RxRFswMUXv1 board/PQC50-48-S5-O_EMC_trimmed_12/VIN
- C95 pad 2: GND -> Net-(PS12-GND)
- C96 pad 1: Net-(PS13-VIN) -> /RxRFswMUXv1 board/PQC50-48-S5-O_EMC_trimmed_12/VIN
- C96 pad 2: Net-(PS13-GND) -> /RxRFswMUXv1 board/+8V_1
- C97 pad 1: Net-(PS13-VIN) -> Net-(PS12-GND)
- C97 pad 2: Net-(PS13-GND) -> GND
- C98 pad 1: Net-(PS13-VIN) -> /RxRFswMUXv1 board/+8V_1
- C99 pad 1: Net-(PS13-GND) -> 48V
- D13 pad 2: GND -> /RxRFswMUXv1 board/+8V_1
- D14 pad 2: GND -> /RxRFswMUXv1 board/+8V_3
- D15 pad 2: GND -> /RxRFswMUXv1 board/+8V_2
- D16 pad 2: GND -> /RxRFswMUXv1 board/+8V_4
- D5 pad 2: GND -> /TxRFswMUXv1 board/+8V_1
- D6 pad 2: GND -> /TxRFswMUXv1 board/+8V_3
- D7 pad 2: GND -> /TxRFswMUXv1 board/+8V_2
- D8 pad 2: GND -> /TxRFswMUXv1 board/+8V_4
- J10 pad 1: GND -> /TxRFswMUXv1 board/+8V_3
- J11 pad 1: GND -> /TxRFswMUXv1 board/+8V_4
- J12 pad 1: /TxRFswMUXv1 board/EN_12V_FROM_5V -> unconnected-(J12-Pad1)
- J12 pad 2: GND -> unconnected-(J12-Pad2)
- J23 pad 1: unconnected-(J23-Pad1) -> /Rx_Eth_Switch/+5V
- J23 pad 2: unconnected-(J23-Pad2) -> GND
- J28 pad 1: GND -> /RxRFswMUXv1 board/+8V_1
- J29 pad 1: GND -> /RxRFswMUXv1 board/+8V_2
- J30 pad 1: GND -> /RxRFswMUXv1 board/+8V_3
- J31 pad 1: GND -> /RxRFswMUXv1 board/+8V_4
- J32 pad 1: /RxRFswMUXv1 board/EN_12V_FROM_5V -> /Tx_Eth_Switch/+5V
- J43 pad 2: GND -> /TxBFN-16C/+6.5V_1
- J43 pad 3: GND -> /TxBFN-16C/+6.5V_1
- J44 pad 2: GND -> /TxBFN-16C/+6.5V_1
- J44 pad 3: GND -> /TxBFN-16C/+6.5V_1
- J45 pad 1: GND -> unconnected-(J45-Pin_1-Pad1)
- J45 pad 2: GND -> /TxBFN-16C/+6.5V_2
- J45 pad 3: GND -> /TxBFN-16C/+6.5V_2
- J45 pad 4: GND -> unconnected-(J45-Pin_4-Pad4)
- J46 pad 2: GND -> /TxBFN-16C/+6.5V_2
- J46 pad 3: GND -> /TxBFN-16C/+6.5V_2
- J47 pad 2: GND -> /TxBFN-16F/+6.5V_1
- J47 pad 3: GND -> /TxBFN-16F/+6.5V_1
- J48 pad 2: GND -> /TxBFN-16F/+6.5V_1
- J48 pad 3: GND -> /TxBFN-16F/+6.5V_1
- J49 pad 1: GND -> unconnected-(J49-Pin_1-Pad1)
- J49 pad 2: GND -> /TxBFN-16F/+6.5V_2
- J49 pad 3: GND -> /TxBFN-16F/+6.5V_2
- J49 pad 4: GND -> unconnected-(J49-Pin_4-Pad4)
- J50 pad 2: GND -> /TxBFN-16F/+6.5V_2
- J50 pad 3: GND -> /TxBFN-16F/+6.5V_2
- J51 pad 2: GND -> /RxBFN-16F/+6.5V_1
- J51 pad 3: GND -> /RxBFN-16F/+6.5V_1
- J52 pad 2: GND -> /RxBFN-16F/+6.5V_1
- J52 pad 3: GND -> /RxBFN-16F/+6.5V_1
- J53 pad 1: GND -> unconnected-(J53-Pin_1-Pad1)
- J53 pad 2: GND -> /RxBFN-16F/+6.5V_2
- J53 pad 3: GND -> /RxBFN-16F/+6.5V_2
- J53 pad 4: GND -> unconnected-(J53-Pin_4-Pad4)
- J54 pad 2: GND -> /RxBFN-16F/+6.5V_2
- J54 pad 3: GND -> /RxBFN-16F/+6.5V_2
- J55 pad 2: GND -> /RxBFN-16C/+6.5V_1
- J55 pad 3: GND -> /RxBFN-16C/+6.5V_1
- J56 pad 2: GND -> /RxBFN-16C/+6.5V_1
- J56 pad 3: GND -> /RxBFN-16C/+6.5V_1
- J57 pad 1: GND -> unconnected-(J57-Pin_1-Pad1)
- J57 pad 2: GND -> /RxBFN-16C/+6.5V_2
- J57 pad 3: GND -> /RxBFN-16C/+6.5V_2
- J57 pad 4: GND -> unconnected-(J57-Pin_4-Pad4)
- J58 pad 2: GND -> /RxBFN-16C/+6.5V_2
- J58 pad 3: GND -> /RxBFN-16C/+6.5V_2
- J59 pad 2: +5V -> /Rx_AGC/+6.5V
- J59 pad 3: +24V -> /Rx_AGC/+6.5V
- J60 pad 2: +5V -> /Tx_AGC/+6.5V
- J60 pad 3: +24V -> /Tx_AGC/+6.5V
- J61 pad 2: +5V -> /Tx_RPi4_HAT_board/+5V_1
- J61 pad 3: +24V -> /Tx_RPi4_HAT_board/+24V
- J62 pad 2: +5V -> /Tx_RPi4_HAT_board/+5V_2
- J62 pad 3: +24V -> /Tx_RPi4_HAT_board/+24V
- J63 pad 2: +6.5V -> /Tx_RPi4_HAT_board/+5V_2
- J63 pad 3: +6.5V -> /Tx_RPi4_HAT_board/+24V
- J64 pad 2: +6.5V -> /Tx_RPi4_HAT_board/+5V_1
- J64 pad 3: +6.5V -> /Tx_RPi4_HAT_board/+24V
- J65 pad 2: +5V -> /Rx_RPi4_HAT_board/+5V_1
- J65 pad 3: +24V -> /Rx_RPi4_HAT_board/+24V
- J66 pad 2: +5V -> /Rx_RPi4_HAT_board/+5V_2
- J66 pad 3: +24V -> /Rx_RPi4_HAT_board/+24V
- J67 pad 2: +5V -> /Rx_RPi4_HAT_board/+5V_2
- J67 pad 3: +24V -> /Rx_RPi4_HAT_board/+24V
- J68 pad 2: +5V -> /Rx_RPi4_HAT_board/+5V_1
- J68 pad 3: +24V -> /Rx_RPi4_HAT_board/+24V
- J8 pad 1: GND -> /TxRFswMUXv1 board/+8V_1
- J9 pad 1: GND -> /TxRFswMUXv1 board/+8V_2
- L13 pad 2: Net-(PS7-VIN) -> /Tx_RPi4_HAT_board/PDQ10-Q48-S5-D_EMC_7/VIN
- L14 pad 1: GND -> 48V
- L14 pad 2: Net-(PS7-GND) -> /Rx_RPi4_HAT_board/PDQ10-Q48-S5-D_EMC_7/VIN
- L15 pad 2: Net-(PS8-VIN) -> /Rx_RPi4_HAT_board/PDQ10-Q48-S5-D_EMC_8/VIN
- L16 pad 1: GND -> 48V
- L16 pad 2: Net-(PS8-GND) -> /RxRFswMUXv1 board/PDQ10-Q48-S5-D_EMC_10/VIN
- L17 pad 2: Net-(PS9-VIN) -> /TxBFN-16C/PQC50-48-S5-O_EMC_trimmed_10/VIN
- L18 pad 2: Net-(PS9-GND) -> Net-(PS7-GND)
- L19 pad 2: Net-(PS10-VIN) -> /TxBFN-16F/PQC50-48-S5-O_EMC_trimmed_10/VIN
- L20 pad 2: Net-(PS10-GND) -> Net-(PS8-GND)
- L21 pad 2: Net-(PS11-VIN) -> /RxBFN-16F/PQC50-48-S5-O_EMC_trimmed_10/VIN
- L22 pad 2: Net-(PS11-GND) -> Net-(PS9-GND)
- L23 pad 2: Net-(PS12-VIN) -> /RxBFN-16C/PQC50-48-S5-O_EMC_trimmed_10/VIN
- L24 pad 2: Net-(PS12-GND) -> Net-(PS10-GND)
- L25 pad 2: Net-(U6-+VIN) -> /RxRFswMUXv1 board/PQC50-48-S5-O_EMC_trimmed_13/VIN
- L26 pad 1: 48V -> GND
- L26 pad 2: Net-(PS13-VIN) -> Net-(PS11-GND)
- L27 pad 1: GND -> 48V
- L27 pad 2: Net-(PS13-GND) -> /RxRFswMUXv1 board/PQC50-48-S5-O_EMC_trimmed_12/VIN
- L28 pad 1: 48V -> GND
- L28 pad 2: Net-(PS14-VIN) -> Net-(PS12-GND)
- L29 pad 1: GND -> 48V
- L29 pad 2: Net-(PS14-GND) -> /RxRFswMUXv1 board/PDQ10-Q48-S5-D_EMC_12/VIN
- L30 pad 2: Net-(U7-+VIN) -> /RxRFswMUXv1 board/PQC50-48-S5-O_EMC_trimmed_14/VIN
- L31 pad 1: 48V -> GND
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Other:
- board outline added: 200 x 320 mm

Commit message: almost done schematic
Parts:
- removed PS19: PQC50-48-S5-O, BCRL_power_supply:CONV_PQC50-48-S5-O
- added C173: 680uf/100v, Capacitor_SMD:C_0603_1608Metric, F.Cu at (439.5, 131.1)
- added C174: 4.7uf/100v, Capacitor_SMD:C_0603_1608Metric, F.Cu at (439.5, 133.6)
- added C175: 4.7uf/100v, Capacitor_SMD:C_0603_1608Metric, F.Cu at (439.5, 136.1)
- added C176: 4.7uf/100v, Capacitor_SMD:C_0603_1608Metric, F.Cu at (439.5, 138.6)
- added C177: 4.7uf/100v, Capacitor_SMD:C_0603_1608Metric, F.Cu at (439.5, 141.1)
- added C178: 2.2nf/400vac, Capacitor_SMD:C_0603_1608Metric, F.Cu at (443.5, 131.1)
- added C179: 2.2nf/400vac, Capacitor_SMD:C_0603_1608Metric, F.Cu at (443.5, 133.6)
- added C180: 330uf/63v, Capacitor_SMD:C_0603_1608Metric, F.Cu at (443.5, 136.1)
- added J71: OSTVN02A150, BCRL_power_supply:CONN_OSTVN02A150_OST, F.Cu at (432.5, 109.7)
- added J72: OSTVN02A150, BCRL_power_supply:CONN_OSTVN02A150_OST, F.Cu at (432.5, 118.1)
- added J73: OSTVN02A150, BCRL_power_supply:CONN_OSTVN02A150_OST, F.Cu at (432.5, 126.4)
- added J74: OSTVN02A150, BCRL_power_supply:CONN_OSTVN02A150_OST, F.Cu at (432.5, 134.8)
- added L49: 2.2mh, Inductor_SMD:L_0603_1608Metric, F.Cu at (443.5, 138.6)
- added L50: 2.2mh, Inductor_SMD:L_0603_1608Metric, F.Cu at (443.5, 141.1)
- added PS1: PQC50-48-S5-O, BCRL_power_supply:CONV_PQC50-48-S5-O, F.Cu at (284.4, 118.9)
- added PS6: PQC50-48-S5-O, BCRL_power_supply:CONV_PQC50-48-S5-O, F.Cu at (284.4, 143.3)
- added RV17: R_Potentiometer_Trim, Potentiometer_THT:Potentiometer_ACP_CA9-V10_Vertical, F.Cu at (447.5, 138.0)
- moved PS17 224.7 mm to (455.5, 117.6), turned to 0 degrees
- moved H1 208.1 mm to (198.5, 40.5)
- moved H2 208.1 mm to (346.1, 40.5)
- moved H3 201.9 mm to (198.5, 352.7)
- moved H4 201.9 mm to (346.1, 352.7)
- moved H6 198.6 mm to (346.1, 196.7)
- moved H5 198.6 mm to (198.5, 196.7)
- moved RV8 138.7 mm to (304.2, 60.0), turned to 0 degrees
- moved PS16 118.4 mm to (200.4, 142.8), turned to 0 degrees
- moved C82 114.7 mm to (316.3, 76.7), turned to 0 degrees
- moved J60 112.5 mm to (456.0, 185.9)
- moved C77 108.5 mm to (312.3, 76.7), turned to 0 degrees
- moved C75 105.9 mm to (308.3, 84.2), turned to 0 degrees
- moved L23 105.4 mm to (316.3, 84.2), turned to 0 degrees
- moved C78 105.1 mm to (312.3, 79.2), turned to 0 degrees
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Connections:
- C124 pad 2: Net-(PS15-GND) -> Net-(PS9-GND)
- C125 pad 2: Net-(PS15-GND) -> Net-(PS9-GND)
- C127 pad 1: Net-(PS15-GND) -> Net-(PS9-GND)
- C132 pad 1: /TxBFN-16F/PQC50-48-S5-O_EMC_trimmed_9/VIN -> /TxBFN-16C/PQC50-48-S5-O_EMC_trimmed_10/VIN
- C132 pad 2: Net-(PS16-GND) -> Net-(PS10-GND)
- C133 pad 1: /TxBFN-16F/PQC50-48-S5-O_EMC_trimmed_9/VIN -> /TxBFN-16C/PQC50-48-S5-O_EMC_trimmed_10/VIN
- C133 pad 2: Net-(PS16-GND) -> Net-(PS10-GND)
- C134 pad 1: /TxBFN-16F/PQC50-48-S5-O_EMC_trimmed_9/VIN -> /TxBFN-16C/PQC50-48-S5-O_EMC_trimmed_10/VIN
- C134 pad 2: /TxBFN-16F/+6.5V_1 -> /TxBFN-16C/+6.5V_2
- C135 pad 1: Net-(PS16-GND) -> Net-(PS10-GND)
- C136 pad 1: /TxBFN-16F/+6.5V_1 -> /TxBFN-16C/+6.5V_2
- C140 pad 1: /RxBFN-16F/PQC50-48-S5-O_EMC_trimmed_9/VIN -> /TxBFN-16F/PQC50-48-S5-O_EMC_trimmed_9/VIN
- C140 pad 2: Net-(PS17-GND) -> Net-(PS15-GND)
- C141 pad 1: /RxBFN-16F/PQC50-48-S5-O_EMC_trimmed_9/VIN -> /TxBFN-16F/PQC50-48-S5-O_EMC_trimmed_9/VIN
- C141 pad 2: Net-(PS17-GND) -> Net-(PS15-GND)
- C142 pad 1: /RxBFN-16F/PQC50-48-S5-O_EMC_trimmed_9/VIN -> /TxBFN-16F/PQC50-48-S5-O_EMC_trimmed_9/VIN
- C142 pad 2: /RxBFN-16F/+6.5V_1 -> /TxBFN-16F/+6.5V_1
- C143 pad 1: Net-(PS17-GND) -> Net-(PS15-GND)
- C144 pad 1: /RxBFN-16F/+6.5V_1 -> /TxBFN-16F/+6.5V_1
- C155 pad 1: /RxBFN-16C/PQC50-48-S5-O_EMC_trimmed_9/VIN -> /TxBFN-16F/PQC50-48-S5-O_EMC_trimmed_10/VIN
- C155 pad 2: Net-(PS19-GND) -> Net-(PS16-GND)
- C156 pad 1: /RxBFN-16C/PQC50-48-S5-O_EMC_trimmed_9/VIN -> /TxBFN-16F/PQC50-48-S5-O_EMC_trimmed_10/VIN
- C156 pad 2: Net-(PS19-GND) -> Net-(PS16-GND)
- C157 pad 1: /RxBFN-16C/PQC50-48-S5-O_EMC_trimmed_9/VIN -> /TxBFN-16F/PQC50-48-S5-O_EMC_trimmed_10/VIN
- C157 pad 2: /RxBFN-16C/+6.5V_1 -> /TxBFN-16F/+6.5V_2
- C158 pad 1: Net-(PS19-GND) -> Net-(PS16-GND)
- C159 pad 1: /RxBFN-16C/+6.5V_1 -> /TxBFN-16F/+6.5V_2
- C54 pad 1: /TxBFN-16C/PQC50-48-S5-O_EMC_trimmed_10/VIN -> /RxBFN-16C/PQC50-48-S5-O_EMC_trimmed_9/VIN
- C54 pad 2: Net-(PS7-GND) -> Net-(PS1-GND)
- C55 pad 1: /TxBFN-16C/PQC50-48-S5-O_EMC_trimmed_10/VIN -> /RxBFN-16C/PQC50-48-S5-O_EMC_trimmed_9/VIN
- C55 pad 2: Net-(PS7-GND) -> Net-(PS1-GND)
- C56 pad 1: /TxBFN-16C/PQC50-48-S5-O_EMC_trimmed_10/VIN -> /RxBFN-16C/PQC50-48-S5-O_EMC_trimmed_9/VIN
- C56 pad 2: /TxBFN-16C/+6.5V_2 -> /RxBFN-16C/+6.5V_1
- C57 pad 1: Net-(PS7-GND) -> Net-(PS1-GND)
- C58 pad 1: /TxBFN-16C/+6.5V_2 -> /RxBFN-16C/+6.5V_1
- C62 pad 1: /TxBFN-16F/PQC50-48-S5-O_EMC_trimmed_10/VIN -> /RxBFN-16C/PQC50-48-S5-O_EMC_trimmed_10/VIN
- C62 pad 2: Net-(PS8-GND) -> Net-(PS6-GND)
- C63 pad 1: /TxBFN-16F/PQC50-48-S5-O_EMC_trimmed_10/VIN -> /RxBFN-16C/PQC50-48-S5-O_EMC_trimmed_10/VIN
- C63 pad 2: Net-(PS8-GND) -> Net-(PS6-GND)
- C64 pad 1: /TxBFN-16F/PQC50-48-S5-O_EMC_trimmed_10/VIN -> /RxBFN-16C/PQC50-48-S5-O_EMC_trimmed_10/VIN
- C64 pad 2: /TxBFN-16F/+6.5V_2 -> /RxBFN-16C/+6.5V_2
- C65 pad 1: Net-(PS8-GND) -> Net-(PS6-GND)
- C66 pad 1: /TxBFN-16F/+6.5V_2 -> /RxBFN-16C/+6.5V_2
- C70 pad 1: /RxBFN-16F/PQC50-48-S5-O_EMC_trimmed_10/VIN -> /RxBFN-16F/PQC50-48-S5-O_EMC_trimmed_9/VIN
- C70 pad 2: Net-(PS9-GND) -> Net-(PS7-GND)
- C71 pad 1: /RxBFN-16F/PQC50-48-S5-O_EMC_trimmed_10/VIN -> /RxBFN-16F/PQC50-48-S5-O_EMC_trimmed_9/VIN
- C71 pad 2: Net-(PS9-GND) -> Net-(PS7-GND)
- C72 pad 1: /RxBFN-16F/PQC50-48-S5-O_EMC_trimmed_10/VIN -> /RxBFN-16F/PQC50-48-S5-O_EMC_trimmed_9/VIN
- C72 pad 2: /RxBFN-16F/+6.5V_2 -> /RxBFN-16F/+6.5V_1
- C73 pad 1: Net-(PS9-GND) -> Net-(PS7-GND)
- C74 pad 1: /RxBFN-16F/+6.5V_2 -> /RxBFN-16F/+6.5V_1
- C78 pad 1: /RxBFN-16C/PQC50-48-S5-O_EMC_trimmed_10/VIN -> /RxBFN-16F/PQC50-48-S5-O_EMC_trimmed_10/VIN
- C78 pad 2: Net-(PS10-GND) -> Net-(PS8-GND)
- C79 pad 1: /RxBFN-16C/PQC50-48-S5-O_EMC_trimmed_10/VIN -> /RxBFN-16F/PQC50-48-S5-O_EMC_trimmed_10/VIN
- C79 pad 2: Net-(PS10-GND) -> Net-(PS8-GND)
- C80 pad 1: /RxBFN-16C/PQC50-48-S5-O_EMC_trimmed_10/VIN -> /RxBFN-16F/PQC50-48-S5-O_EMC_trimmed_10/VIN
- C80 pad 2: /RxBFN-16C/+6.5V_2 -> /RxBFN-16F/+6.5V_2
- C81 pad 1: Net-(PS10-GND) -> Net-(PS8-GND)
- C82 pad 1: /RxBFN-16C/+6.5V_2 -> /RxBFN-16F/+6.5V_2
- J43 pad 2: /TxBFN-16C/+6.5V_1 -> /RxBFN-16C/+6.5V_1
- J43 pad 3: /TxBFN-16C/+6.5V_1 -> /RxBFN-16C/+6.5V_1
- J44 pad 2: /TxBFN-16C/+6.5V_1 -> /RxBFN-16C/+6.5V_1
- J44 pad 3: /TxBFN-16C/+6.5V_1 -> /RxBFN-16C/+6.5V_1
- J45 pad 2: /TxBFN-16C/+6.5V_2 -> /RxBFN-16C/+6.5V_2
- J45 pad 3: /TxBFN-16C/+6.5V_2 -> /RxBFN-16C/+6.5V_2
- J46 pad 2: /TxBFN-16C/+6.5V_2 -> /RxBFN-16C/+6.5V_2
- J46 pad 3: /TxBFN-16C/+6.5V_2 -> /RxBFN-16C/+6.5V_2
- J47 pad 2: /TxBFN-16F/+6.5V_1 -> /RxBFN-16F/+6.5V_1
- J47 pad 3: /TxBFN-16F/+6.5V_1 -> /RxBFN-16F/+6.5V_1
- J48 pad 2: /TxBFN-16F/+6.5V_1 -> /RxBFN-16F/+6.5V_1
- J48 pad 3: /TxBFN-16F/+6.5V_1 -> /RxBFN-16F/+6.5V_1
- J49 pad 2: /TxBFN-16F/+6.5V_2 -> /RxBFN-16F/+6.5V_2
- J49 pad 3: /TxBFN-16F/+6.5V_2 -> /RxBFN-16F/+6.5V_2
- J50 pad 2: /TxBFN-16F/+6.5V_2 -> /RxBFN-16F/+6.5V_2
- J50 pad 3: /TxBFN-16F/+6.5V_2 -> /RxBFN-16F/+6.5V_2
- J51 pad 2: /RxBFN-16F/+6.5V_1 -> /TxBFN-16C/+6.5V_1
- J51 pad 3: /RxBFN-16F/+6.5V_1 -> /TxBFN-16C/+6.5V_1
- J52 pad 2: /RxBFN-16F/+6.5V_1 -> /TxBFN-16C/+6.5V_1
- J52 pad 3: /RxBFN-16F/+6.5V_1 -> /TxBFN-16C/+6.5V_1
- J53 pad 2: /RxBFN-16F/+6.5V_2 -> /TxBFN-16C/+6.5V_2
- J53 pad 3: /RxBFN-16F/+6.5V_2 -> /TxBFN-16C/+6.5V_2
- J54 pad 2: /RxBFN-16F/+6.5V_2 -> /TxBFN-16C/+6.5V_2
- J54 pad 3: /RxBFN-16F/+6.5V_2 -> /TxBFN-16C/+6.5V_2
- J55 pad 2: /RxBFN-16C/+6.5V_1 -> /TxBFN-16F/+6.5V_1
- J55 pad 3: /RxBFN-16C/+6.5V_1 -> /TxBFN-16F/+6.5V_1
- J56 pad 2: /RxBFN-16C/+6.5V_1 -> /TxBFN-16F/+6.5V_1
- J56 pad 3: /RxBFN-16C/+6.5V_1 -> /TxBFN-16F/+6.5V_1
- J57 pad 2: /RxBFN-16C/+6.5V_2 -> /TxBFN-16F/+6.5V_2
- J57 pad 3: /RxBFN-16C/+6.5V_2 -> /TxBFN-16F/+6.5V_2
- J58 pad 2: /RxBFN-16C/+6.5V_2 -> /TxBFN-16F/+6.5V_2
- J58 pad 3: /RxBFN-16C/+6.5V_2 -> /TxBFN-16F/+6.5V_2
- J59 pad 2: /Rx_AGC/+6.5V -> /RxBFN-16F/+6.5V_1
- J59 pad 3: /Rx_AGC/+6.5V -> /RxBFN-16F/+6.5V_1
- J60 pad 2: /Tx_AGC/+6.5V -> /TxBFN-16F/+6.5V_1
- J60 pad 3: /Tx_AGC/+6.5V -> /TxBFN-16F/+6.5V_1
- L17 pad 2: /TxBFN-16C/PQC50-48-S5-O_EMC_trimmed_10/VIN -> /RxBFN-16C/PQC50-48-S5-O_EMC_trimmed_9/VIN
- L18 pad 2: Net-(PS7-GND) -> Net-(PS1-GND)
- L19 pad 2: /TxBFN-16F/PQC50-48-S5-O_EMC_trimmed_10/VIN -> /RxBFN-16C/PQC50-48-S5-O_EMC_trimmed_10/VIN
- L20 pad 2: Net-(PS8-GND) -> Net-(PS6-GND)
- L21 pad 2: /RxBFN-16F/PQC50-48-S5-O_EMC_trimmed_10/VIN -> /RxBFN-16F/PQC50-48-S5-O_EMC_trimmed_9/VIN
- L22 pad 2: Net-(PS9-GND) -> Net-(PS7-GND)
- L23 pad 2: /RxBFN-16C/PQC50-48-S5-O_EMC_trimmed_10/VIN -> /RxBFN-16F/PQC50-48-S5-O_EMC_trimmed_10/VIN
- L24 pad 2: Net-(PS10-GND) -> Net-(PS8-GND)
- L37 pad 2: Net-(PS15-GND) -> Net-(PS9-GND)
- L38 pad 2: /TxBFN-16F/PQC50-48-S5-O_EMC_trimmed_9/VIN -> /TxBFN-16C/PQC50-48-S5-O_EMC_trimmed_10/VIN
- L39 pad 2: Net-(PS16-GND) -> Net-(PS10-GND)
- L40 pad 2: /RxBFN-16F/PQC50-48-S5-O_EMC_trimmed_9/VIN -> /TxBFN-16F/PQC50-48-S5-O_EMC_trimmed_9/VIN
- L41 pad 2: Net-(PS17-GND) -> Net-(PS15-GND)
- L43 pad 2: /RxBFN-16C/PQC50-48-S5-O_EMC_trimmed_9/VIN -> /TxBFN-16F/PQC50-48-S5-O_EMC_trimmed_10/VIN
- L44 pad 2: Net-(PS19-GND) -> Net-(PS16-GND)
- PS10 pad 1: /RxBFN-16C/PQC50-48-S5-O_EMC_trimmed_10/VIN -> /TxBFN-16C/PQC50-48-S5-O_EMC_trimmed_10/VIN
- PS10 pad 2: /RxBFN-16C/+6.5V_CTL_2 -> /TxBFN-16C/+6.5V_CTL_2
- PS10 pad 7: /RxBFN-16C/+6.5V_2 -> /TxBFN-16C/+6.5V_2
- PS10 pad 8: /RxBFN-16C/+6.5V_2 -> /TxBFN-16C/+6.5V_2
- PS15 pad 1: /TxBFN-16C/PQC50-48-S5-O_EMC_trimmed_9/VIN -> /TxBFN-16F/PQC50-48-S5-O_EMC_trimmed_9/VIN
- PS15 pad 2: /TxBFN-16C/+6.5V_CTL_1 -> /TxBFN-16F/+6.5V_CTL_1
- PS15 pad 7: /TxBFN-16C/+6.5V_1 -> /TxBFN-16F/+6.5V_1
- PS15 pad 8: /TxBFN-16C/+6.5V_1 -> /TxBFN-16F/+6.5V_1
- PS16 pad 1: /TxBFN-16F/PQC50-48-S5-O_EMC_trimmed_9/VIN -> /TxBFN-16F/PQC50-48-S5-O_EMC_trimmed_10/VIN
- PS16 pad 2: /TxBFN-16F/+6.5V_CTL_1 -> /TxBFN-16F/+6.5V_CTL_2
- PS16 pad 7: /TxBFN-16F/+6.5V_1 -> /TxBFN-16F/+6.5V_2
- PS16 pad 8: /TxBFN-16F/+6.5V_1 -> /TxBFN-16F/+6.5V_2
- PS17 pad 1: /RxBFN-16F/PQC50-48-S5-O_EMC_trimmed_9/VIN -> /fan_20x/PQC50-48-S5-O_EMC_trimmed_15/VIN
- PS17 pad 2: /RxBFN-16F/+6.5V_CTL_1 -> /fan_20x/FAN_CTL
- PS17 pad 7: /RxBFN-16F/+6.5V_1 -> /fan_20x/V_FAN
- PS17 pad 8: /RxBFN-16F/+6.5V_1 -> /fan_20x/V_FAN
- PS7 pad 1: /TxBFN-16C/PQC50-48-S5-O_EMC_trimmed_10/VIN -> /RxBFN-16F/PQC50-48-S5-O_EMC_trimmed_9/VIN
- PS7 pad 2: /TxBFN-16C/+6.5V_CTL_2 -> /RxBFN-16F/+6.5V_CTL_1
- PS7 pad 7: /TxBFN-16C/+6.5V_2 -> /RxBFN-16F/+6.5V_1
- PS7 pad 8: /TxBFN-16C/+6.5V_2 -> /RxBFN-16F/+6.5V_1
- PS8 pad 1: /TxBFN-16F/PQC50-48-S5-O_EMC_trimmed_10/VIN -> /RxBFN-16F/PQC50-48-S5-O_EMC_trimmed_10/VIN
- PS8 pad 2: /TxBFN-16F/+6.5V_CTL_2 -> /RxBFN-16F/+6.5V_CTL_2
- PS8 pad 7: /TxBFN-16F/+6.5V_2 -> /RxBFN-16F/+6.5V_2
- PS8 pad 8: /TxBFN-16F/+6.5V_2 -> /RxBFN-16F/+6.5V_2
- PS9 pad 1: /RxBFN-16F/PQC50-48-S5-O_EMC_trimmed_10/VIN -> /TxBFN-16C/PQC50-48-S5-O_EMC_trimmed_9/VIN
- PS9 pad 2: /RxBFN-16F/+6.5V_CTL_2 -> /TxBFN-16C/+6.5V_CTL_1
- PS9 pad 7: /RxBFN-16F/+6.5V_2 -> /TxBFN-16C/+6.5V_1
- PS9 pad 8: /RxBFN-16F/+6.5V_2 -> /TxBFN-16C/+6.5V_1
- RV13 pad 2: Net-(PS15-TRIM) -> Net-(PS9-TRIM)
- RV14 pad 1: /TxBFN-16F/+6.5V_1 -> /TxBFN-16C/+6.5V_2
- RV14 pad 2: Net-(PS16-TRIM) -> Net-(PS10-TRIM)
- RV15 pad 1: /RxBFN-16F/+6.5V_1 -> /TxBFN-16F/+6.5V_1
- RV15 pad 2: Net-(PS17-TRIM) -> Net-(PS15-TRIM)
- RV16 pad 1: /RxBFN-16C/+6.5V_1 -> /TxBFN-16F/+6.5V_2
- RV16 pad 2: Net-(PS19-TRIM) -> Net-(PS16-TRIM)
- RV5 pad 1: /TxBFN-16C/+6.5V_2 -> /RxBFN-16C/+6.5V_1
- RV5 pad 2: Net-(PS7-TRIM) -> Net-(PS1-TRIM)
- RV6 pad 1: /TxBFN-16F/+6.5V_2 -> /RxBFN-16C/+6.5V_2
- RV6 pad 2: Net-(PS8-TRIM) -> Net-(PS6-TRIM)
- RV7 pad 1: /RxBFN-16F/+6.5V_2 -> /RxBFN-16F/+6.5V_1
- RV7 pad 2: Net-(PS9-TRIM) -> Net-(PS7-TRIM)
- RV8 pad 1: /RxBFN-16C/+6.5V_2 -> /RxBFN-16F/+6.5V_2
- RV8 pad 2: Net-(PS10-TRIM) -> Net-(PS8-TRIM)
Other:
- board size 200 x 320 mm -> 190 x 320 mm

Commit message: schematic done
Parts:
- removed J12: 5034801600, BCRL_power_supply:MOLEX_5034801600
- removed RV1, RV10, RV11, RV12, RV13, RV14, RV15, RV16, RV17, RV2, RV3, RV4, RV5, RV6, RV7, RV8, RV9: R_Potentiometer_Trim, Potentiometer_THT:Potentiometer_ACP_CA9-V10_Vertical
- added D17: LED, LED_SMD:LED_0603_1608Metric, F.Cu at (290.6, 136.3)
- added D18: LED, LED_SMD:LED_0603_1608Metric, F.Cu at (299.6, 73.5)
- added D19: LED, LED_SMD:LED_0603_1608Metric, F.Cu at (218.0, 72.6)
- added D20: LED, LED_SMD:LED_0603_1608Metric, F.Cu at (211.5, 136.7)
- added D21: LED, LED_SMD:LED_0603_1608Metric, F.Cu at (290.6, 138.9)
- added D22: LED, LED_SMD:LED_0603_1608Metric, F.Cu at (299.6, 76.1)
- added D23: LED, LED_SMD:LED_0603_1608Metric, F.Cu at (218.0, 75.2)
- added D24: LED, LED_SMD:LED_0603_1608Metric, F.Cu at (211.5, 139.3)
- added D25: LED, LED_SMD:LED_0603_1608Metric, F.Cu at (122.1, 160.3)
- added D26: LED, LED_SMD:LED_0603_1608Metric, F.Cu at (123.2, 236.0)
- added D27: LED, LED_SMD:LED_0603_1608Metric, F.Cu at (284.0, 220.0)
- added D28: LED, LED_SMD:LED_0603_1608Metric, F.Cu at (218.6, 221.7)
- added D29: LED, LED_SMD:LED_0603_1608Metric, F.Cu at (284.0, 222.6)
- added D30: LED, LED_SMD:LED_0603_1608Metric, F.Cu at (218.6, 224.3)
- added D31: LED, LED_SMD:LED_0603_1608Metric, F.Cu at (284.0, 225.2)
- added D32: LED, LED_SMD:LED_0603_1608Metric, F.Cu at (218.6, 226.9)
- added J75: Conn_01x04_Pin, Connector_PinHeader_2.54mm:PinHeader_1x04_P2.54mm_Vertical, F.Cu at (459.6, 325.7)
- added R14: 168k, Resistor_SMD:R_0603_1608Metric, F.Cu at (233.0, 329.0)
- added R15: 168k, Resistor_SMD:R_0603_1608Metric, F.Cu at (233.0, 331.5)
- added R16: 168k, Resistor_SMD:R_0603_1608Metric, F.Cu at (233.0, 334.0)
- added R17: 168k, Resistor_SMD:R_0603_1608Metric, F.Cu at (233.0, 336.5)
- added R18: 168k, Resistor_SMD:R_0603_1608Metric, F.Cu at (302.6, 126.2)
- added R19: 168k, Resistor_SMD:R_0603_1608Metric, F.Cu at (302.6, 128.7)
- added R20: 168k, Resistor_SMD:R_0603_1608Metric, F.Cu at (230.0, 62.6)
- added R21: 168k, Resistor_SMD:R_0603_1608Metric, F.Cu at (311.6, 63.4)
- added R22: 168k, Resistor_SMD:R_0603_1608Metric, F.Cu at (311.6, 65.9)
- added R23: 168k, Resistor_SMD:R_0603_1608Metric, F.Cu at (230.0, 65.1)
- added R37: 168k, Resistor_SMD:R_0603_1608Metric, F.Cu at (223.5, 126.6)
- added R38: 168k, Resistor_SMD:R_0603_1608Metric, F.Cu at (223.5, 129.1)
- added R39: 168k, Resistor_SMD:R_0603_1608Metric, F.Cu at (428.2, 126.1)
- added R40: 168k, Resistor_SMD:R_0603_1608Metric, F.Cu at (451.2, 327.1)
- added R41: 168k, Resistor_SMD:R_0603_1608Metric, F.Cu at (451.2, 329.7)
- added R42: 168k, Resistor_SMD:R_0603_1608Metric, F.Cu at (451.2, 332.2)
- added R43: 168k, Resistor_SMD:R_0603_1608Metric, F.Cu at (451.2, 334.7)
- added R44: 1k, Resistor_SMD:R_0603_1608Metric, F.Cu at (302.6, 131.2)
- added R45: 1k, Resistor_SMD:R_0603_1608Metric, F.Cu at (311.6, 68.4)
- added R46: 1k, Resistor_SMD:R_0603_1608Metric, F.Cu at (230.0, 67.6)
- added R47: 1k, Resistor_SMD:R_0603_1608Metric, F.Cu at (223.5, 131.6)
- added R48: 1k, Resistor_SMD:R_0603_1608Metric, F.Cu at (302.6, 133.8)
- added R49: 1k, Resistor_SMD:R_0603_1608Metric, F.Cu at (311.6, 70.9)
- added R50: 1k, Resistor_SMD:R_0603_1608Metric, F.Cu at (230.0, 70.1)
- added R51: 1k, Resistor_SMD:R_0603_1608Metric, F.Cu at (223.5, 134.1)
- added R52: 1k, Resistor_SMD:R_0603_1608Metric, F.Cu at (117.4, 149.4)
- added R53: 1k, Resistor_SMD:R_0603_1608Metric, F.Cu at (118.5, 225.1)
- added R54: 1k, Resistor_SMD:R_0603_1608Metric, F.Cu at (279.9, 207.7)
- added R56: 1k, Resistor_SMD:R_0603_1608Metric, F.Cu at (214.6, 209.3)
- added R57: 1k, Resistor_SMD:R_0603_1608Metric, F.Cu at (279.9, 210.2)
- added R58: 1k, Resistor_SMD:R_0603_1608Metric, F.Cu at (214.6, 211.9)
- added R59: 1k, Resistor_SMD:R_0603_1608Metric, F.Cu at (279.9, 212.7)
- added R60: 1k, Resistor_SMD:R_0603_1608Metric, F.Cu at (214.6, 214.4)
- H1, H2, H3, H4, H5, H6: value MountingHole -> MountingHole_Pad
- moved H5 454.7 mm to (616.0, 377.0)
- moved H6 454.7 mm to (763.6, 377.0)
- moved H3 437.7 mm to (616.0, 221.0)
- moved H4 437.7 mm to (763.6, 221.0)
- moved H1 418.2 mm to (616.0, 65.0)
- moved H2 418.2 mm to (763.6, 65.0)
- moved U13 234.0 mm to (488.2, 258.6)
- moved J29 191.9 mm to (466.2, 277.5)
- moved J30 187.2 mm to (466.2, 285.9)
- moved J42 186.8 mm to (467.5, 331.9)
- moved U11 186.4 mm to (461.3, 258.6)
- moved J41 184.1 mm to (467.5, 326.1)
- moved J31 184.0 mm to (466.2, 294.2)
- moved J40 179.6 mm to (464.0, 321.1)
- moved D16 174.9 mm to (455.2, 342.8)
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Connections:
- C106 pad 2: /RxRFswMUXv1 board/+8V_3 -> /RxRFswMUXv1 board/PQC50-48-S5-O_EMC_trimmed_14/+VO
- C108 pad 1: /RxRFswMUXv1 board/+8V_3 -> /RxRFswMUXv1 board/PQC50-48-S5-O_EMC_trimmed_14/+VO
- C88 pad 2: /RxRFswMUXv1 board/+8V_2 -> /RxRFswMUXv1 board/PQC50-48-S5-O_EMC_trimmed_13/+VO
- C90 pad 1: /RxRFswMUXv1 board/+8V_2 -> /RxRFswMUXv1 board/PQC50-48-S5-O_EMC_trimmed_13/+VO
- C96 pad 2: /RxRFswMUXv1 board/+8V_1 -> /RxRFswMUXv1 board/PQC50-48-S5-O_EMC_trimmed_12/+VO
- C98 pad 1: /RxRFswMUXv1 board/+8V_1 -> /RxRFswMUXv1 board/PQC50-48-S5-O_EMC_trimmed_12/+VO
- H1 pad 1: (no net) -> GND
- H2 pad 1: (no net) -> GND
- H3 pad 1: (no net) -> GND
- H4 pad 1: (no net) -> GND
- H5 pad 1: (no net) -> GND
- H6 pad 1: (no net) -> GND
- P5 pad 10: unconnected-(P5-Pad10) -> GND
- P5 pad 7: unconnected-(P5-Pad7) -> /RxRFswMUXv1 board/+5V_1
- P5 pad 8: unconnected-(P5-Pad8) -> /RxRFswMUXv1 board/LNA_SHUTDOWN_1
- P5 pad 9: unconnected-(P5-Pad9) -> GND
- P6 pad 10: unconnected-(P6-Pad10) -> GND
- P6 pad 7: unconnected-(P6-Pad7) -> /RxRFswMUXv1 board/+5V_2
- P6 pad 8: unconnected-(P6-Pad8) -> /RxRFswMUXv1 board/LNA_SHUTDOWN_1
- P6 pad 9: unconnected-(P6-Pad9) -> GND
- P7 pad 10: unconnected-(P7-Pad10) -> GND
- P7 pad 7: unconnected-(P7-Pad7) -> /RxRFswMUXv1 board/+5V_3
- P7 pad 8: unconnected-(P7-Pad8) -> /RxRFswMUXv1 board/LNA_SHUTDOWN_1
- P7 pad 9: unconnected-(P7-Pad9) -> GND
- P8 pad 10: unconnected-(P8-Pad10) -> GND
- P8 pad 7: unconnected-(P8-Pad7) -> /RxRFswMUXv1 board/+5V_4
- P8 pad 8: unconnected-(P8-Pad8) -> /RxRFswMUXv1 board/LNA_SHUTDOWN_1
- P8 pad 9: unconnected-(P8-Pad9) -> GND
- PS11 pad 2: /RxRFswMUXv1 board/RxLNA2_8V_CTL -> /RxRFswMUXv1 board/PQC50-48-S5-O_EMC_trimmed_13/CTRL
- PS11 pad 7: /RxRFswMUXv1 board/+8V_2 -> /RxRFswMUXv1 board/PQC50-48-S5-O_EMC_trimmed_13/+VO
- PS11 pad 8: /RxRFswMUXv1 board/+8V_2 -> /RxRFswMUXv1 board/PQC50-48-S5-O_EMC_trimmed_13/+VO
- PS12 pad 2: /RxRFswMUXv1 board/RxLNA1_8V_CTL -> /RxRFswMUXv1 board/PQC50-48-S5-O_EMC_trimmed_12/CTRL
- PS12 pad 7: /RxRFswMUXv1 board/+8V_1 -> /RxRFswMUXv1 board/PQC50-48-S5-O_EMC_trimmed_12/+VO
- PS12 pad 8: /RxRFswMUXv1 board/+8V_1 -> /RxRFswMUXv1 board/PQC50-48-S5-O_EMC_trimmed_12/+VO
- PS13 pad 2: /RxRFswMUXv1 board/RxLNA3_8V_CTL -> /RxRFswMUXv1 board/PQC50-48-S5-O_EMC_trimmed_14/CTRL
- PS13 pad 7: /RxRFswMUXv1 board/+8V_3 -> /RxRFswMUXv1 board/PQC50-48-S5-O_EMC_trimmed_14/+VO
- PS13 pad 8: /RxRFswMUXv1 board/+8V_3 -> /RxRFswMUXv1 board/PQC50-48-S5-O_EMC_trimmed_14/+VO
- U10 pad 3: /RxRFswMUXv1 board/+5V_4 -> /RxRFswMUXv1 board/PDQ10-Q48-S5-D_EMC_12/+5V
- U10 pad 6: /RxRFswMUXv1 board/RxLNA4_5V_CTL -> /RxRFswMUXv1 board/PDQ10-Q48-S5-D_EMC_12/CTRL
- U11 pad 3: /RxRFswMUXv1 board/+5V_3 -> /RxRFswMUXv1 board/PDQ10-Q48-S5-D_EMC_9/+5V
- U11 pad 6: /RxRFswMUXv1 board/RxLNA3_5V_CTL -> /RxRFswMUXv1 board/PDQ10-Q48-S5-D_EMC_9/CTRL
- U13 pad 3: /RxRFswMUXv1 board/+5V_2 -> /RxRFswMUXv1 board/PDQ10-Q48-S5-D_EMC_11/+5V
- U13 pad 6: /RxRFswMUXv1 board/RxLNA2_5V_CTL -> /RxRFswMUXv1 board/PDQ10-Q48-S5-D_EMC_11/CTRL
- U6 pad 3: /Tx_RPi4_HAT_board/+5V_2 -> /Tx_RPi4_HAT_board/PDQ10-Q48-S5-D_EMC_7/+5V
- U7 pad 3: /Rx_RPi4_HAT_board/+5V_2 -> /Rx_RPi4_HAT_board/PDQ10-Q48-S5-D_EMC_7/+5V
- U9 pad 3: /RxRFswMUXv1 board/+5V_1 -> /RxRFswMUXv1 board/PDQ10-Q48-S5-D_EMC_10/+5V
- U9 pad 6: /RxRFswMUXv1 board/RxLNA1_5V_CTL -> /RxRFswMUXv1 board/PDQ10-Q48-S5-D_EMC_10/CTRL
