File: kicad_files/bcrl_power_supply/bcrl_power_supply.kicad_pcb (KiCad board)
At the start: 2 copper layers, 190 x 320 mm, 447 parts, among them J1 OSTVN02A150, J10 OSTVN02A150, J11 OSTVN02A150, J13 Conn_01x02, J14 Conn_01x02, J15 Conn_01x02, J16 Conn_01x02, J17 Conn_01x02, J18 Conn_01x02, J19 Conn_01x02, J2 OSTVN02A150, J20 Conn_01x02, J21 5034801600, J22 5034801600, J23 OSTVN02A150, J24 OSTVN02A150, J25 OSTVN02A150, J26 OSTVN02A150, J27 OSTVN02A150, J28 OSTVN02A150, J29 OSTVN02A150, J3 Conn_01x02, J30 OSTVN02A150, J31 OSTVN02A150, J32 OSTVN02A150, J33 Conn_01x02, J34 Conn_01x02, J35 Conn_01x02, J36 Conn_01x02, J37 Conn_01x02, J38 Conn_01x02, J39 Conn_01x02, J4 OSTVN02A150, J40 Conn_01x02, J41 5034801600, J42 5034801600, J43 Conn_01x04_Pin, J44 Conn_01x04_Pin, J45 Conn_01x04_Pin, J46 Conn_01x04_Pin, J47 Conn_01x04_Pin, J48 Conn_01x04_Pin, J49 Conn_01x04_Pin, J5 OSTVN02A150, J50 Conn_01x04_Pin, J51 Conn_01x04_Pin, J52 Conn_01x04_Pin, J53 Conn_01x04_Pin, J54 Conn_01x04_Pin, J55 Conn_01x04_Pin, J56 Conn_01x04_Pin, J57 Conn_01x04_Pin, J58 Conn_01x04_Pin, J59 Conn_01x04_Pin, J6 OSTVN02A150, J60 Conn_01x04_Pin, J61 Conn_01x06_Pin, J62 Conn_01x06_Pin, J63 Conn_01x06_Pin, J64 Conn_01x06_Pin, J65 Conn_01x06_Pin, J66 Conn_01x06_Pin, J67 Conn_01x06_Pin, J68 Conn_01x06_Pin, J69 Conn_01x02, J7 OSTVN02A150, J70 Conn_01x02, J71 OSTVN02A150, J72 OSTVN02A150, J73 OSTVN02A150, J74 OSTVN02A150, J75 Conn_01x04_Pin, J8 OSTVN02A150, J9 OSTVN02A150, P1 5104338-1, P2 5104338-1, P3 5104338-1, P4 5104338-1, P5 5104338-1, P6 5104338-1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

Commit message: big changes
Parts:
- removed C100, C102, C103, C104, C105, C160, C161, C163, C164, C174, C175, C176, C177, C76, C77, C78, C84, C85, C86, C87, C92, C93, C94, C95, C99: 4.7uf/100v, Capacitor_SMD:C_0603_1608Metric
- removed C101, C152, C173, C75, C83, C91: 680uf/100v, Capacitor_SMD:C_0603_1608Metric
- removed C106, C178, C179, C88, C89, C96, C97: 2.2nf/400vac, Capacitor_SMD:C_0603_1608Metric
- removed C151, C168: 47uf/50v, Capacitor_SMD:C_0603_1608Metric
- removed C159, C180, C90, C98: 330uf/63v, Capacitor_SMD:C_0603_1608Metric
- removed C162, C165: 330uf/100v, Capacitor_SMD:C_0603_1608Metric
- removed C166, C167: 1nf/2kv, Capacitor_SMD:C_0603_1608Metric
- removed the C39 at (225.0, 321.5)
- removed the C40 at (225.0, 324.0)
- removed the C41 at (271.9, 202.6)
- removed the C42 at (271.9, 205.1)
- removed D20, D21: LED, LED_SMD:LED_0603_1608Metric
- removed the D31 at (284.0, 225.2)
- removed the D32 at (218.6, 226.9)
- removed the J41 at (467.5, 326.1)
- removed the J42 at (467.5, 331.9)
- removed the J43 at (290.9, 110.0)
- removed the J44 at (295.6, 110.0)
- removed the J45 at (300.2, 110.0)
- removed J72, J73, J74: OSTVN02A150, BCRL_power_supply:CONN_OSTVN02A150_OST
- removed L16, L29, L3, L34, L35, L42, L45, L46: 4.7uh/3.1a, Inductor_SMD:L_0603_1608Metric
- removed L17, L20, L21, L22, L23, L24, L25, L27, L28, L30, L31, L32, L33, L36, L37, L38, L39, L4, L40, L41, L43, L44, L49, L5, L50, L6: 2.2mh, Inductor_SMD:L_0603_1608Metric
- removed the L7 at (225.0, 346.6)
- removed the L8 at (225.0, 349.1)
- removed PS10, PS7, PS9: PQC50-48-S5-O, BCRL_power_supply:CONV_PQC50-48-S5-O
- removed the R20 at (230.0, 62.6)
- removed R27, R28, R44, R45: 1k, Resistor_SMD:R_0603_1608Metric
- removed the R29 at (447.2, 347.2)
- removed R42, R43: 168k, Resistor_SMD:R_0603_1608Metric
- removed the R62 at (451.2, 339.7)
- removed R76: 3.4k, Resistor_SMD:R_0603_1608Metric
- removed U12, U9: PDQ10-Q48-S5-D, BCRL_power_supply:CONV_PDQ10-Q48-S5-D
- removed the U4 at (243.1, 256.8)
- removed the U5 at (255.9, 187.9)
- added D25: LED, LED_SMD:LED_0603_1608Metric, F.Cu at (256.8, 254.5)
- added D26: LED, LED_SMD:LED_0603_1608Metric, F.Cu at (256.8, 177.2)
- added D33: LED, LED_SMD:LED_0603_1608Metric, F.Cu at (193.3, 231.4)
- added D34: LED, LED_SMD:LED_0603_1608Metric, F.Cu at (193.3, 234.0)
- added D35: LED, LED_SMD:LED_0603_1608Metric, F.Cu at (193.3, 236.6)
- added D36: LED, LED_SMD:LED_0603_1608Metric, F.Cu at (294.9, 177.2)
- added D37: LED, LED_SMD:LED_0603_1608Metric, F.Cu at (218.7, 254.5)
- added D38: LED, LED_SMD:LED_0603_1608Metric, F.Cu at (218.7, 293.1)
- added J12: Conn_01x02, Connector_PinHeader_2.54mm:PinHeader_1x02_P2.54mm_Vertical, F.Cu at (152.0, 250.0)
- added J23: OSTVN02A150, BCRL_power_supply:CONN_OSTVN02A150_OST, F.Cu at (176.6, 215.6)
- added J32: Conn_01x02, Connector_PinHeader_2.54mm:PinHeader_1x02_P2.54mm_Vertical, F.Cu at (161.3, 198.1)
- added J69: Conn_01x06_Pin, Connector_PinHeader_2.54mm:PinHeader_1x06_P2.54mm_Vertical, F.Cu at (161.3, 302.0)
- added J70: Conn_01x06_Pin, Connector_PinHeader_2.54mm:PinHeader_1x06_P2.54mm_Vertical, F.Cu at (166.0, 302.0)
- added J71: Conn_01x02, Connector_PinHeader_2.54mm:PinHeader_1x02_P2.54mm_Vertical, F.Cu at (189.2, 198.1)
- added J76: Conn_01x06_Pin, Connector_PinHeader_2.54mm:PinHeader_1x06_P2.54mm_Vertical, F.Cu at (175.3, 302.0)
- added J77: Conn_01x06_Pin, Connector_PinHeader_2.54mm:PinHeader_1x06_P2.54mm_Vertical, F.Cu at (179.9, 302.0)
- added J78: Conn_01x06_Pin, Connector_PinHeader_2.54mm:PinHeader_1x06_P2.54mm_Vertical, F.Cu at (184.6, 302.0)
- added PS19: IND108W, BCRL_power_supply:IND108W, F.Cu at (230.7, 244.9)
- added PS21: IND108W, BCRL_power_supply:IND108W, F.Cu at (230.7, 283.6)
- added R12: 1k, Resistor_SMD:R_0603_1608Metric, F.Cu at (181.4, 41.5)
- added R13: 1k, Resistor_SMD:R_0603_1608Metric, F.Cu at (171.4, 44.0)
- added R52: 1k, Resistor_SMD:R_0603_1608Metric, F.Cu at (214.6, 194.7)
- added R53: 9.59k, Resistor_SMD:R_0603_1608Metric, F.Cu at (329.0, 192.2)
- added R64: 1k, Resistor_SMD:R_0603_1608Metric, F.Cu at (214.6, 272.0)
- added R65: 9.59k, Resistor_SMD:R_0603_1608Metric, F.Cu at (214.6, 308.2)
- added R66: 1k, Resistor_SMD:R_0603_1608Metric, F.Cu at (214.6, 310.7)
- added U14: PDQ10-Q48-S5-D, BCRL_power_supply:CONV_PDQ10-Q48-S5-D, F.Cu at (335.3, 251.5)
- added U15: PDQ10-Q48-S5-D, BCRL_power_supply:CONV_PDQ10-Q48-S5-D, F.Cu at (335.3, 312.2)
- C10, C11, C110, C111, C112, C117, C118, C119, C12, C120, C122, C125, C13, C130, C131, C132, C133, C141, C146, C147, C153, C154, C155, C156, C18, C19, C20, C21, C26, C27, C28, C29, C34, C35, C36, C37, C7, C8: value 4.7uf/100v -> 22uf
- C107, C126, C127, C134, C135, C14, C142, C143, C15, C157, C158, C22, C23, C30, C31, C38: value 2.2nf/400vac -> 22uf
- C108, C128, C136, C144, C16, C24, C32: value 330uf/63v -> 22uf
- C109, C121, C129, C17, C25, C33, C9: value 680uf/100v -> 22uf
- C113, C139, C69, C79: value 4.7uf/100v -> 100uf
- C114, C80: value 2.2nf/400vac -> 1uf
- C115, C81: value 2.2nf/400vac -> 100uf
- C116, C82: value 330uf/63v -> 1uf
- C137, C67: value 680uf/100v -> 100uf
- C138, C140, C68, C70: value 4.7uf/100v -> 1uf
- C145, C148: value 330uf/100v -> 22uf
- C149, C150: value 1nf/2kv -> 22uf
- C45, C48, C63: value 4.7uf/100v -> 330uf/100v
- C49, C50: value 4.7uf/100v -> 1nf/2kv
- C51: value 680uf/100v -> 47uf/50v
- C56: value 2.2nf/400vac -> 330uf/100v
- C57, C72, C73: value 2.2nf/400vac -> 4.7uf/100v
- C58, C74: value 330uf/63v -> 4.7uf/100v
- C59: value 680uf/100v -> 4.7uf/100v
- C6: value 4.7uf/100uf -> 4.7uf/100v
- C64, C65: value 2.2nf/400vac -> 1nf/2kv
- C66: value 330uf/63v -> 47uf/50v
- J20, J39, J40: value Conn_01x02 -> 5034801600; footprint Connector_PinHeader_2.54mm:PinHeader_1x02_P2.54mm_Vertical -> BCRL_power_supply:MOLEX_5034801600
- J22: value 5034801600 -> OSTVN02A150; footprint BCRL_power_supply:MOLEX_5034801600 -> BCRL_power_supply:CONN_OSTVN02A150_OST
- J30, J31: value OSTVN02A150 -> Conn_01x02; footprint BCRL_power_supply:CONN_OSTVN02A150_OST -> Connector_PinHeader_2.54mm:PinHeader_1x02_P2.54mm_Vertical
- J46, J47, J48: value Conn_01x04_Pin -> OSTVN02A150; footprint Connector_PinHeader_2.54mm:PinHeader_1x04_P2.54mm_Vertical -> BCRL_power_supply:CONN_OSTVN02A150_OST
- J61, J62, J63, J64, J65, J66: value Conn_01x06_Pin -> Conn_01x04_Pin; footprint Connector_PinHeader_2.54mm:PinHeader_1x06_P2.54mm_Vertical -> Connector_PinHeader_2.54mm:PinHeader_1x04_P2.54mm_Vertical
- J75: value Conn_01x04_Pin -> Conn_01x06_Pin; footprint Connector_PinHeader_2.54mm:PinHeader_1x04_P2.54mm_Vertical -> Connector_PinHeader_2.54mm:PinHeader_1x06_P2.54mm_Vertical
- L10, L11, L18, L19, L26, L9: value 2.2mh -> 4.7uh/3.1a
- PS1, PS12, PS14, PS15, PS16, PS2, PS3, PS4: value PQC50-48-S5-O -> IND108W; footprint BCRL_power_supply:CONV_PQC50-48-S5-O -> BCRL_power_supply:IND108W
- PS11, PS13, PS17, PS8: value PQC50-48-S5-O -> EHHD010A0B41-HZ; footprint BCRL_power_supply:CONV_PQC50-48-S5-O -> BCRL_power_supply:CONV_EHHD010A0B41-HZ
- PS18, PS20: value PDQE15-Q48-D24-D -> IND108W; footprint BCRL_power_supply:CONV_PDQE15-Q48-D24-D -> BCRL_power_supply:IND108W
- PS5, PS6: value PQC50-48-S5-O -> PDQE15-Q48-D24-D; footprint BCRL_power_supply:CONV_PQC50-48-S5-O -> BCRL_power_supply:CONV_PDQE15-Q48-D24-D
- R11, R34, R55: value 3.4k -> 1k
- R14, R16, R18: value 168k -> 9.59k
- R15, R17, R19, R21, R22, R23, R39: value 168k -> 1k
- R31, R48: value 1k -> 3.4k
- R33, R36, R63: value 3.4k -> 9.59k
- R37, R38, R40, R41: value 168k -> 3.4k
- R46, R49, R51, R59: value 1k -> 9.59k
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- renumbered C169 to C39, C170 to C40, C171 to C41, C172 to C42, D25 to D31, D26 to D32, J32 to J41, J70 to J42, J23 to J43, J69 to J44, J71 to J45, L47 to L7, L48 to L8, R12 to R20, R13 to R29, R52 to R61, R53 to R62, U14 to U4, U15 to U5
Connections:
- net /RxRFswMUXv1 board/PQC50-48-S5-O_EMC_trimmed_13/CTRL renamed /BFN/EHHD010A0B41-HZ1/ON/OFF
- net /RxRFswMUXv1 board/PQC50-48-S5-O_EMC_trimmed_14/CTRL renamed /BFN/EHHD010A0B41-HZ2/ON/OFF
- net /Rx_Eth_Switch/CTL renamed /Rx_Eth_Switch/CTRL
- net /Rx_RPi4_HAT_board/PDQ10-Q48-S5-D_EMC_7/CTRL renamed /RPi_HAT/Rx_RPi4_HAT_board1/+5V_CTRL
- net /Tx_Eth_Switch/CTL renamed /Tx_Eth_Switch/CTRL
- net /Tx_RPi4_HAT_board/PDQ10-Q48-S5-D_EMC_7/CTRL renamed /RPi_HAT/Tx_RPi4_HAT_board1/+5V_CTRL
- C10 pad 1: 48V -> /TxRFswMUXv1 board/+12V
- C107 pad 1: Net-(PS13-GND) -> /BFN/IND108W_EMC_6.5V_3/+8V
- C108 pad 1: /RxRFswMUXv1 board/PQC50-48-S5-O_EMC_trimmed_14/+VO -> /BFN/IND108W_EMC_6.5V_3/+8V
- C109 pad 1: 48V -> /BFN/IND108W_EMC_6.5V_3/+8V
- C11 pad 1: 48V -> /TxRFswMUXv1 board/+12V
- C110 pad 1: 48V -> +12V_2
- C111 pad 1: 48V -> +12V_2
- C112 pad 1: /RxRFswMUXv1 board/PQC50-48-S5-O_EMC_trimmed_11/VIN -> +12V_2
- C112 pad 2: Net-(PS14-GND) -> GND
- C113 pad 1: /RxRFswMUXv1 board/PQC50-48-S5-O_EMC_trimmed_11/VIN -> 48V
- C113 pad 2: Net-(PS14-GND) -> GND
- C114 pad 1: /RxRFswMUXv1 board/PQC50-48-S5-O_EMC_trimmed_11/VIN -> 48V
- C114 pad 2: /RxRFswMUXv1 board/+8V_4 -> GND
- C115 pad 1: Net-(PS14-GND) -> +12V_2
- C116 pad 1: /RxRFswMUXv1 board/+8V_4 -> +12V_2
- C117 pad 1: 48V -> /BFN/IND108W_EMC_6.5V_2/+8V
- C118 pad 1: /RxRFswMUXv1 board/PDQ10-Q48-S5-D_EMC_9/VIN -> /BFN/IND108W_EMC_6.5V_2/+8V
- C119 pad 1: 48V -> /BFN/IND108W_EMC_6.5V_2/+8V
- C12 pad 1: /TxRFswMUXv1 board/PQC50-48-S5-O_EMC_trimmed_1/VIN -> /TxRFswMUXv1 board/+12V
- C12 pad 2: Net-(PS2-GND) -> GND
- C120 pad 1: /TxRFswMUXv1 board/PDQ10-Q48-S5-D_EMC_1/VIN -> +12V_1
- C121 pad 1: 48V -> +12V_1
- C122 pad 1: 48V -> +12V_1
- C124 pad 1: /TxBFN-16C/PQC50-48-S5-O_EMC_trimmed_9/VIN -> /TxRFswMUXv1 board/PDQ10-Q48-S5-D_EMC_2/VIN
- C124 pad 2: Net-(PS9-GND) -> GND
- C125 pad 1: /TxBFN-16C/PQC50-48-S5-O_EMC_trimmed_9/VIN -> /BFN/IND108W_EMC_6.5V_1/+8V
- C125 pad 2: Net-(PS9-GND) -> GND
- C126 pad 1: /TxBFN-16C/PQC50-48-S5-O_EMC_trimmed_9/VIN -> /BFN/IND108W_EMC_6.5V_1/+8V
- C126 pad 2: /TxBFN-16C/+6.5V_1 -> GND
- C127 pad 1: Net-(PS9-GND) -> /BFN/IND108W_EMC_6.5V_1/+8V
- C128 pad 1: /TxBFN-16C/+6.5V_1 -> +12V_1
- C129 pad 1: 48V -> +12V_1
- C13 pad 1: /TxRFswMUXv1 board/PQC50-48-S5-O_EMC_trimmed_1/VIN -> /TxRFswMUXv1 board/+8V_3
- C13 pad 2: Net-(PS2-GND) -> GND
- C130 pad 1: 48V -> +12V_1
- C131 pad 1: 48V -> /BFN/IND108W_EMC_6.5V_4/+8V
- C132 pad 1: /TxBFN-16C/PQC50-48-S5-O_EMC_trimmed_10/VIN -> /BFN/IND108W_EMC_6.5V_4/+8V
- C132 pad 2: Net-(PS10-GND) -> GND
- C133 pad 1: /TxBFN-16C/PQC50-48-S5-O_EMC_trimmed_10/VIN -> /BFN/IND108W_EMC_6.5V_4/+8V
- C133 pad 2: Net-(PS10-GND) -> GND
- C134 pad 1: /TxBFN-16C/PQC50-48-S5-O_EMC_trimmed_10/VIN -> +12V_2
- C134 pad 2: /TxBFN-16C/+6.5V_2 -> GND
- C135 pad 1: Net-(PS10-GND) -> +12V_2
- C136 pad 1: /TxBFN-16C/+6.5V_2 -> +12V_2
- C139 pad 1: 48V -> /TxRFswMUXv1 board/+12V
- C14 pad 1: /TxRFswMUXv1 board/PQC50-48-S5-O_EMC_trimmed_1/VIN -> /TxRFswMUXv1 board/+8V_3
- C14 pad 2: /TxRFswMUXv1 board/+8V_1 -> GND
- C140 pad 1: /TxBFN-16F/PQC50-48-S5-O_EMC_trimmed_9/VIN -> /TxRFswMUXv1 board/+12V
- C140 pad 2: Net-(PS15-GND) -> GND
- C141 pad 1: /TxBFN-16F/PQC50-48-S5-O_EMC_trimmed_9/VIN -> /RxRFswMUXv1 board/+8V_3
- C141 pad 2: Net-(PS15-GND) -> GND
- C142 pad 1: /TxBFN-16F/PQC50-48-S5-O_EMC_trimmed_9/VIN -> /RxRFswMUXv1 board/+12V
- C142 pad 2: /TxBFN-16F/+6.5V_1 -> GND
- C143 pad 1: Net-(PS15-GND) -> /RxRFswMUXv1 board/+12V
- C144 pad 1: /TxBFN-16F/+6.5V_1 -> /RxRFswMUXv1 board/+12V
- C145 pad 1: 48V -> /RxRFswMUXv1 board/+8V_4
- C146 pad 1: 48V -> /RxRFswMUXv1 board/+8V_4
- C147 pad 1: /Tx_RPi4_HAT_board/PDQE15-Q48-D24-D_EMC_1/VIN -> /RxRFswMUXv1 board/+8V_4
- C148 pad 1: /Tx_RPi4_HAT_board/PDQE15-Q48-D24-D_EMC_1/VIN -> /RxRFswMUXv1 board/+12V
- C149 pad 1: /Tx_RPi4_HAT_board/PDQE15-Q48-D24-D_EMC_1/VIN -> /RxRFswMUXv1 board/+12V
- C149 pad 2: /Tx_RPi4_HAT_board/+24V -> GND
- C15 pad 1: Net-(PS2-GND) -> /TxRFswMUXv1 board/+8V_3
- C150 pad 1: GND -> /RxRFswMUXv1 board/+12V
- C153 pad 1: 48V -> /TxRFswMUXv1 board/+8V_1
- C154 pad 1: 48V -> /TxRFswMUXv1 board/+8V_1
- C155 pad 1: /TxBFN-16F/PQC50-48-S5-O_EMC_trimmed_10/VIN -> /TxRFswMUXv1 board/+8V_1
- C155 pad 2: Net-(PS16-GND) -> GND
- C156 pad 1: /TxBFN-16F/PQC50-48-S5-O_EMC_trimmed_10/VIN -> /TxRFswMUXv1 board/+12V
- C156 pad 2: Net-(PS16-GND) -> GND
- C157 pad 1: /TxBFN-16F/PQC50-48-S5-O_EMC_trimmed_10/VIN -> /TxRFswMUXv1 board/+12V
- C157 pad 2: /TxBFN-16F/+6.5V_2 -> GND
- C158 pad 1: Net-(PS16-GND) -> /TxRFswMUXv1 board/+12V
- C16 pad 1: /TxRFswMUXv1 board/+8V_1 -> /TxRFswMUXv1 board/+12V
- C17 pad 1: 48V -> /TxRFswMUXv1 board/+12V
- C18 pad 1: 48V -> /TxRFswMUXv1 board/+12V
- C19 pad 1: 48V -> /TxRFswMUXv1 board/+8V_4
- C2 pad 1: /TxRFswMUXv1 board/PDQ10-Q48-S5-D_EMC_2/VIN -> /TxRFswMUXv1 board/PDQ10-Q48-S5-D_EMC_3/VIN
- C20 pad 1: /TxRFswMUXv1 board/PQC50-48-S5-O_EMC_trimmed_2/VIN -> /TxRFswMUXv1 board/+8V_4
- C20 pad 2: Net-(PS3-GND) -> GND
- C21 pad 1: /TxRFswMUXv1 board/PQC50-48-S5-O_EMC_trimmed_2/VIN -> /TxRFswMUXv1 board/+8V_4
- C21 pad 2: Net-(PS3-GND) -> GND
- C22 pad 1: /TxRFswMUXv1 board/PQC50-48-S5-O_EMC_trimmed_2/VIN -> /TxRFswMUXv1 board/+12V
- C22 pad 2: /TxRFswMUXv1 board/+8V_2 -> GND
- C23 pad 1: Net-(PS3-GND) -> /TxRFswMUXv1 board/+12V
- C24 pad 1: /TxRFswMUXv1 board/+8V_2 -> /TxRFswMUXv1 board/+12V
- C25 pad 1: 48V -> /RxRFswMUXv1 board/+8V_1
- C26 pad 1: 48V -> /RxRFswMUXv1 board/+8V_1
- C27 pad 1: 48V -> /RxRFswMUXv1 board/+8V_1
- C28 pad 1: /TxRFswMUXv1 board/PQC50-48-S5-O_EMC_trimmed_3/VIN -> /RxRFswMUXv1 board/+12V
- C28 pad 2: Net-(PS4-GND) -> GND
- C29 pad 1: /TxRFswMUXv1 board/PQC50-48-S5-O_EMC_trimmed_3/VIN -> /RxRFswMUXv1 board/+12V
- C29 pad 2: Net-(PS4-GND) -> GND
- C30 pad 1: /TxRFswMUXv1 board/PQC50-48-S5-O_EMC_trimmed_3/VIN -> /RxRFswMUXv1 board/+12V
- C30 pad 2: /TxRFswMUXv1 board/+8V_3 -> GND
- C31 pad 1: Net-(PS4-GND) -> /RxRFswMUXv1 board/+8V_2
- C32 pad 1: /TxRFswMUXv1 board/+8V_3 -> /RxRFswMUXv1 board/+8V_2
- C33 pad 1: 48V -> /RxRFswMUXv1 board/+8V_2
- C34 pad 1: 48V -> /RxRFswMUXv1 board/+12V
- C35 pad 1: 48V -> /RxRFswMUXv1 board/+12V
- C36 pad 1: /TxRFswMUXv1 board/PQC50-48-S5-O_EMC_trimmed_4/VIN -> /RxRFswMUXv1 board/+12V
- C36 pad 2: Net-(PS5-GND) -> GND
- C37 pad 1: /TxRFswMUXv1 board/PQC50-48-S5-O_EMC_trimmed_4/VIN -> /RxRFswMUXv1 board/+8V_3
- C37 pad 2: Net-(PS5-GND) -> GND
- C38 pad 1: /TxRFswMUXv1 board/PQC50-48-S5-O_EMC_trimmed_4/VIN -> /RxRFswMUXv1 board/+8V_3
- C38 pad 2: /TxRFswMUXv1 board/+8V_4 -> GND
- C4 pad 1: /TxRFswMUXv1 board/PDQ10-Q48-S5-D_EMC_3/VIN -> /TxRFswMUXv1 board/PDQ10-Q48-S5-D_EMC_4/VIN
- C44 pad 1: /Tx_RPi4_HAT_board/PDQ10-Q48-S5-D_EMC_7/VIN -> /RPi_HAT/Tx_RPi4_HAT_board1/PDQ10-Q48-S5-D_EMC_8/VIN
- C46 pad 1: /Rx_RPi4_HAT_board/PDQ10-Q48-S5-D_EMC_7/VIN -> 48V
- C47 pad 1: 48V -> /RPi_HAT/Rx_RPi4_HAT_board1/PDQE15-Q48-D24-D_EMC_1/VIN
- C48 pad 1: /Rx_RPi4_HAT_board/PDQ10-Q48-S5-D_EMC_8/VIN -> /RPi_HAT/Rx_RPi4_HAT_board1/PDQE15-Q48-D24-D_EMC_1/VIN
- C49 pad 1: 48V -> /RPi_HAT/Rx_RPi4_HAT_board1/PDQE15-Q48-D24-D_EMC_1/VIN
- C49 pad 2: GND -> /RPi_HAT/+24V_Rx_RPi4_HAT
- C50 pad 1: /RxRFswMUXv1 board/PDQ10-Q48-S5-D_EMC_10/VIN -> GND
- C51 pad 1: 48V -> /RPi_HAT/+24V_Rx_RPi4_HAT
- C53 pad 1: 48V -> /RPi_HAT/Rx_RPi4_HAT_board1/PDQ10-Q48-S5-D_EMC_8/VIN
- C54 pad 1: /RxBFN-16C/PQC50-48-S5-O_EMC_trimmed_9/VIN -> 48V
- C54 pad 2: Net-(PS1-GND) -> GND
- C55 pad 1: /RxBFN-16C/PQC50-48-S5-O_EMC_trimmed_9/VIN -> /RxRFswMUXv1 board/PDQ10-Q48-S5-D_EMC_14/VIN
- C55 pad 2: Net-(PS1-GND) -> GND
- C56 pad 1: /RxBFN-16C/PQC50-48-S5-O_EMC_trimmed_9/VIN -> 48V
- C56 pad 2: /RxBFN-16C/+6.5V_1 -> GND
- C57 pad 1: Net-(PS1-GND) -> 48V
- C58 pad 1: /RxBFN-16C/+6.5V_1 -> 48V
- C59 pad 1: 48V -> /RxRFswMUXv1 board/PDQ10-Q48-S5-D_EMC_15/VIN
- C61 pad 1: 48V -> /TxRFswMUXv1 board/PDQ10-Q48-S5-D_EMC_1/VIN
- C62 pad 1: /RxBFN-16C/PQC50-48-S5-O_EMC_trimmed_10/VIN -> /RPi_HAT/Tx_RPi4_HAT_board1/PDQE15-Q48-D24-D_EMC_1/VIN
- C62 pad 2: Net-(PS6-GND) -> GND
- C63 pad 1: /RxBFN-16C/PQC50-48-S5-O_EMC_trimmed_10/VIN -> /RPi_HAT/Tx_RPi4_HAT_board1/PDQE15-Q48-D24-D_EMC_1/VIN
- C63 pad 2: Net-(PS6-GND) -> GND
- C64 pad 1: /RxBFN-16C/PQC50-48-S5-O_EMC_trimmed_10/VIN -> /RPi_HAT/Tx_RPi4_HAT_board1/PDQE15-Q48-D24-D_EMC_1/VIN
- C64 pad 2: /RxBFN-16C/+6.5V_2 -> /RPi_HAT/+24V_Tx_RPi4_HAT
- C65 pad 1: Net-(PS6-GND) -> GND
- C66 pad 1: /RxBFN-16C/+6.5V_2 -> /RPi_HAT/+24V_Tx_RPi4_HAT
- C69 pad 1: 48V -> +12V_1
- C7 pad 1: 48V -> /TxRFswMUXv1 board/+8V_2
- C70 pad 1: /RxBFN-16F/PQC50-48-S5-O_EMC_trimmed_9/VIN -> +12V_1
- C70 pad 2: Net-(PS7-GND) -> GND
- C71 pad 1: /RxBFN-16F/PQC50-48-S5-O_EMC_trimmed_9/VIN -> 48V
- C71 pad 2: Net-(PS7-GND) -> GND
- C72 pad 1: /RxBFN-16F/PQC50-48-S5-O_EMC_trimmed_9/VIN -> /RxRFswMUXv1 board/PDQ10-Q48-S5-D_EMC_16/VIN
- C72 pad 2: /RxBFN-16F/+6.5V_1 -> GND
- C73 pad 1: Net-(PS7-GND) -> 48V
- C74 pad 1: /RxBFN-16F/+6.5V_1 -> /RxRFswMUXv1 board/PDQ10-Q48-S5-D_EMC_17/VIN
- C79 pad 1: /RxBFN-16F/PQC50-48-S5-O_EMC_trimmed_10/VIN -> 48V
- C79 pad 2: Net-(PS8-GND) -> GND
- C8 pad 1: /TxRFswMUXv1 board/PDQ10-Q48-S5-D_EMC_4/VIN -> /TxRFswMUXv1 board/+8V_2
- C80 pad 1: /RxBFN-16F/PQC50-48-S5-O_EMC_trimmed_10/VIN -> 48V
- C80 pad 2: /RxBFN-16F/+6.5V_2 -> GND
- C81 pad 1: Net-(PS8-GND) -> /RxRFswMUXv1 board/+12V
- C82 pad 1: /RxBFN-16F/+6.5V_2 -> /RxRFswMUXv1 board/+12V
- C9 pad 1: 48V -> /TxRFswMUXv1 board/+8V_2
- D10 pad 2: /RxRFswMUXv1 board/+5V_2 -> /RPi_HAT/+5V_Tx_RPi4_HAT
- D11 pad 2: /RxRFswMUXv1 board/+5V_3 -> /RPi_HAT/+24V_Rx_RPi4_HAT
- D12 pad 2: /RxRFswMUXv1 board/+5V_4 -> /BFN/IND108W_EMC_6.5V_3/+8V
- D13 pad 2: /RxRFswMUXv1 board/+8V_1 -> /BFN/IND108W_EMC_6.5V_2/+8V
- D14 pad 2: /RxRFswMUXv1 board/+8V_3 -> /RxRFswMUXv1 board/+5V_1
- D15 pad 2: /RxRFswMUXv1 board/+8V_2 -> /RxRFswMUXv1 board/+5V_2
- D16 pad 2: /RxRFswMUXv1 board/+8V_4 -> /RxRFswMUXv1 board/+5V_3
- D17 pad 2: /RxBFN-16C/+6.5V_1 -> /RxRFswMUXv1 board/+5V_4
- D18 pad 2: /RxBFN-16F/+6.5V_1 -> /TxRFswMUXv1 board/+12V
- D19 pad 2: /TxBFN-16C/+6.5V_1 -> /RxRFswMUXv1 board/+12V
- D22 pad 2: /RxBFN-16F/+6.5V_2 -> /RPi_HAT/+24V_Tx_RPi4_HAT
- D23 pad 2: /TxBFN-16C/+6.5V_2 -> /BFN/IND108W_EMC_6.5V_1/+8V
- D24 pad 2: /TxBFN-16F/+6.5V_2 -> /BFN/IND108W_EMC_6.5V_4/+8V
- D27 pad 2: /Tx_RPi4_HAT_board/+5V_1 -> /TxRFswMUXv1 board/+8V_1
- D28 pad 2: /Rx_RPi4_HAT_board/+5V_1 -> /TxRFswMUXv1 board/+8V_4
- D29 pad 2: /Tx_RPi4_HAT_board/+24V -> /RxRFswMUXv1 board/+8V_1
- D30 pad 2: /Rx_RPi4_HAT_board/+24V -> /RxRFswMUXv1 board/+8V_1
- D9 pad 2: /RxRFswMUXv1 board/+5V_1 -> /RPi_HAT/+5V_Rx_RPi4_HAT
- J13 pad 1: /TxRFswMUXv1 board/TxPA1_5V_CTL -> /TxRFswMUXv1 board/TxPA2_5V_CTRL
- J14 pad 1: /TxRFswMUXv1 board/TxPA2_5V_CTL -> /TxRFswMUXv1 board/TxPA3_5V_CTRL
- J15 pad 1: /TxRFswMUXv1 board/TxPA3_5V_CTL -> /TxRFswMUXv1 board/TxPA4_5V_CTRL
- J16 pad 1: /TxRFswMUXv1 board/TxPA4_5V_CTL -> /TxRFswMUXv1 board/TxPA1_8V_CTRL
- J17 pad 1: /TxRFswMUXv1 board/TxPA1_8V_CTL -> /TxRFswMUXv1 board/TxPA2_8V_CTRL
- J18 pad 1: /TxRFswMUXv1 board/TxPA2_8V_CTL -> /TxRFswMUXv1 board/TxPA3_8V_CTRL
- J19 pad 1: /TxRFswMUXv1 board/TxPA3_8V_CTL -> /TxRFswMUXv1 board/TxPA4_8V_CTRL
- J20 pad 1: /TxRFswMUXv1 board/TxPA4_8V_CTL -> GND
- J20 pad 2: GND -> /TxRFswMUXv1 board/P1.1_VCTRL2_SW1
- J21 pad 10: /TxRFswMUXv1 board/P3.1_VCTL2_SW1 -> /TxRFswMUXv1 board/TxPA1_8V_CTRL
- J21 pad 11: /TxRFswMUXv1 board/P3.1_VCTL2_SW1 -> /TxRFswMUXv1 board/TxPA2_8V_CTRL
- J21 pad 12: /TxRFswMUXv1 board/P3.3_VCTL1 -> /TxRFswMUXv1 board/TxPA3_8V_CTRL
- J21 pad 13: /TxRFswMUXv1 board/P4.1_VCTL2_SW1 -> /TxRFswMUXv1 board/TxPA4_8V_CTRL
- J21 pad 14: /TxRFswMUXv1 board/P4.1_VCTL2_SW1 -> unconnected-(J21-Pad14)
- J21 pad 15: /TxRFswMUXv1 board/P4.3_VCTL1 -> unconnected-(J21-Pad15)
- J21 pad 2: /TxRFswMUXv1 board/P1.1_VCTL2_SW1 -> /TxRFswMUXv1 board/TxPA1_5V_CTRL
- J21 pad 3: /TxRFswMUXv1 board/P1.2_VCTL2_SW2 -> /TxRFswMUXv1 board/TxPA2_5V_CTRL
- J21 pad 4: /TxRFswMUXv1 board/P1.3_VCTL1 -> /TxRFswMUXv1 board/TxPA3_5V_CTRL
- J21 pad 5: /TxRFswMUXv1 board/P2.1_VCTL2_SW1 -> /TxRFswMUXv1 board/TxPA4_5V_CTRL
- J21 pad 6: /TxRFswMUXv1 board/P2.1_VCTL2_SW1 -> unconnected-(J21-Pad6)
- J21 pad 7: /TxRFswMUXv1 board/P2.3_VCTL1 -> unconnected-(J21-Pad7)
- J22 pad 1: GND -> /RxRFswMUXv1 board/+5V_1
- J22 pad 2: /TxRFswMUXv1 board/TxPA1_5V_CTL -> GND
- J24 pad 1: /RxRFswMUXv1 board/+5V_1 -> /RxRFswMUXv1 board/+5V_3
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
Commit message: board review
Parts:
- removed C141, C142, C143, C144, C145, C146, C147, C148, C149, C150, C153, C154, C155, C156, C157, C158: 22uf, Capacitor_SMD:C_0603_1608Metric
- removed the C31 at (290.8, 177.2)
- removed the C32 at (290.8, 179.7)
- removed the C33 at (290.8, 182.2)
- removed the C34 at (290.8, 184.7)
- removed the C37 at (214.6, 254.5)
- removed the C38 at (214.6, 257.0)
- removed C46, C47, C52, C53, C57: 4.7uf/100v, Capacitor_SMD:C_0603_1608Metric
- removed C48, C56: 330uf/100v, Capacitor_SMD:C_0603_1608Metric
- removed C49: 1nf/2kv, Capacitor_SMD:C_0603_1608Metric
- removed the C50 at (280.2, 318.0)
- removed the C51 at (280.2, 320.5)
- removed the C62 at (280.2, 281.6)
- removed the C63 at (280.2, 284.1)
- removed the C64 at (280.2, 286.6)
- removed the C65 at (280.2, 289.1)
- removed the C66 at (280.2, 291.6)
- removed the D22 at (177.4, 44.1)
- removed the D23 at (218.7, 331.8)
- removed the D24 at (294.9, 215.9)
- removed D25, D26, D27, D28, D29, D32, D36: LED, LED_SMD:LED_0603_1608Metric
- removed the D9 at (167.4, 41.6)
- removed the J43 at (102.9, 209.6)
- removed the J67 at (152.0, 302.0)
- removed the J68 at (156.7, 302.0)
- removed the L10 at (280.2, 323.1)
- removed the L11 at (350.8, 333.9)
- removed the L13 at (280.2, 294.1)
- removed L7, L9: 4.7uh/3.1a, Inductor_SMD:L_0603_1608Metric
- removed the PS13 at (180.6, 135.1)
- removed PS20, PS21: IND108W, BCRL_power_supply:IND108W
- removed the PS5 at (264.8, 317.7)
- removed the R11 at (171.4, 41.5)
- removed the R30 at (181.4, 44.0)
- removed the R31 at (350.8, 336.4)
- removed the R32 at (367.4, 131.8)
- removed R34, R47, R50, R52, R54, R60, R64, R66: 1k, Resistor_SMD:R_0603_1608Metric
- removed the R39 at (200.3, 40.2)
- removed the R49 at (214.6, 230.9)
- removed the R59 at (290.8, 192.2)
- removed R65: 9.59k, Resistor_SMD:R_0603_1608Metric
- removed U4, U7: PDQ10-Q48-S5-D, BCRL_power_supply:CONV_PDQ10-Q48-S5-D
- added C105: 22u, Capacitor_SMD:C_0603_1608Metric, F.Cu at (450.5, 198.4)
- added C106: 22u, Capacitor_SMD:C_0603_1608Metric, F.Cu at (450.5, 200.9)
- added C107: 22u, Capacitor_SMD:C_0603_1608Metric, F.Cu at (450.5, 203.4)
- added C108: 22u, Capacitor_SMD:C_0603_1608Metric, F.Cu at (450.5, 205.9)
- added C109: 22u, Capacitor_SMD:C_0603_1608Metric, F.Cu at (450.5, 208.4)
- added C110: 22u, Capacitor_SMD:C_0603_1608Metric, F.Cu at (450.5, 210.9)
- added C111: 22u, Capacitor_SMD:C_0603_1608Metric, F.Cu at (488.6, 198.4)
- added C112: 22u, Capacitor_SMD:C_0603_1608Metric, F.Cu at (488.6, 200.9)
- added C117: 22u, Capacitor_SMD:C_0603_1608Metric, F.Cu at (450.5, 237.0)
- added C118: 22u, Capacitor_SMD:C_0603_1608Metric, F.Cu at (450.5, 239.5)
- added C119: 22u, Capacitor_SMD:C_0603_1608Metric, F.Cu at (450.5, 242.0)
- added C120: 22u, Capacitor_SMD:C_0603_1608Metric, F.Cu at (450.5, 244.5)
- added C121: 22u, Capacitor_SMD:C_0603_1608Metric, F.Cu at (450.5, 247.0)
- added C122: 22u, Capacitor_SMD:C_0603_1608Metric, F.Cu at (450.5, 249.6)
- added C123: 22u, Capacitor_SMD:C_0603_1608Metric, F.Cu at (412.4, 237.0)
- added C124: 22u, Capacitor_SMD:C_0603_1608Metric, F.Cu at (412.4, 239.5)
- added C125: 22u, Capacitor_SMD:C_0603_1608Metric, F.Cu at (412.4, 242.0)
- added C126: 22u, Capacitor_SMD:C_0603_1608Metric, F.Cu at (412.4, 244.5)
- added C127: 22u, Capacitor_SMD:C_0603_1608Metric, F.Cu at (412.4, 247.0)
- added C128: 22u, Capacitor_SMD:C_0603_1608Metric, F.Cu at (412.4, 249.6)
- added C129: 4.7u, Capacitor_SMD:C_0603_1608Metric, F.Cu at (477.4, 297.7)
- added C130: 4.7u, Capacitor_SMD:C_0603_1608Metric, F.Cu at (477.4, 300.2)
- added C131: 330u, Capacitor_SMD:C_0603_1608Metric, F.Cu at (439.9, 297.7)
- added C132: 4.7u, Capacitor_SMD:C_0603_1608Metric, F.Cu at (439.9, 300.2)
- added C133: 4.7u, Capacitor_SMD:C_0603_1608Metric, F.Cu at (439.9, 302.7)
- added C134: 330u, Capacitor_SMD:C_0603_1608Metric, F.Cu at (439.9, 305.2)
- added C135: 1nf, Capacitor_SMD:C_0603_1608Metric, F.Cu at (439.9, 307.8)
- added C136: 1nf, Capacitor_SMD:C_0603_1608Metric, F.Cu at (439.9, 310.3)
- added C137: 47u, Capacitor_SMD:C_0603_1608Metric, F.Cu at (439.9, 312.8)
- added C41: 2.2u, Capacitor_SMD:C_0603_1608Metric, F.Cu at (517.7, 300.5)
- added C42: 100u, Capacitor_SMD:C_0603_1608Metric, F.Cu at (488.6, 283.4)
- added D14: LED 0603, LED_SMD:LED_0603_1608Metric, F.Cu at (213.3, 233.9)
- added FL1: FLT007A0Z, BCRL_power_supply:FLT007A0Z, F.Cu at (491.6, 318.4)
- added J45: Conn_01x02, Connector_PinHeader_2.54mm:PinHeader_1x02_P2.54mm_Vertical, F.Cu at (531.7, 235.9)
- added J71: Conn_01x02, Connector_PinHeader_2.54mm:PinHeader_1x02_P2.54mm_Vertical, F.Cu at (545.7, 235.9)
- added J72: Conn_01x02, Connector_PinHeader_2.54mm:PinHeader_1x02_P2.54mm_Vertical, F.Cu at (550.3, 235.9)
- added J73: Conn_01x06_Pin, Connector_PinHeader_2.54mm:PinHeader_1x06_P2.54mm_Vertical, F.Cu at (213.6, 207.8)
- added J74: Conn_01x06_Pin, Connector_PinHeader_2.54mm:PinHeader_1x06_P2.54mm_Vertical, F.Cu at (218.2, 207.8)
- added J75: Conn_01x06_Pin, Connector_PinHeader_2.54mm:PinHeader_1x06_P2.54mm_Vertical, F.Cu at (222.9, 207.8)
- added J79: Conn_01x02, Connector_PinHeader_2.54mm:PinHeader_1x02_P2.54mm_Vertical, F.Cu at (547.9, 221.5)
- added J80: Conn_01x06_Pin, Connector_PinHeader_2.54mm:PinHeader_1x06_P2.54mm_Vertical, F.Cu at (227.6, 207.8)
- added J81: Conn_01x06_Pin, Connector_PinHeader_2.54mm:PinHeader_1x06_P2.54mm_Vertical, F.Cu at (232.2, 207.8)
- added J82: Conn_01x06_Pin, Connector_PinHeader_2.54mm:PinHeader_1x06_P2.54mm_Vertical, F.Cu at (236.8, 207.8)
- added J83: Conn_01x06_Pin, Connector_PinHeader_2.54mm:PinHeader_1x06_P2.54mm_Vertical, F.Cu at (241.5, 207.8)
- added L15: 4.7u, Inductor_SMD:L_0603_1608Metric, F.Cu at (477.4, 302.7)
- added L16: 4.7u, Inductor_SMD:L_0603_1608Metric, F.Cu at (439.9, 315.3)
- added L5: 4.7u, Inductor_SMD:L_0603_1608Metric, F.Cu at (550.7, 300.5)
- added PS15: IND108W, BCRL_power_supply:IND108W, F.Cu at (466.6, 188.8)
- added PS16: IND108W, BCRL_power_supply:IND108W, F.Cu at (504.7, 188.8)
- added PS17: IND108W, BCRL_power_supply:IND108W, F.Cu at (466.6, 227.5)
- added R18: 9.59k, Resistor_SMD:R_0603_1608Metric, F.Cu at (412.4, 290.7)
- added R21: 1k, Resistor_SMD:R_0603_1608Metric, F.Cu at (217.3, 233.6)
- added R55: 9.59k, Resistor_SMD:R_0603_1608Metric, F.Cu at (450.5, 252.1)
- added R57: 9.59k, Resistor_SMD:R_0603_1608Metric, F.Cu at (412.4, 252.1)
- added R61: 3.4k, Resistor_SMD:R_0603_1608Metric, F.Cu at (477.4, 305.2)
- added U14: PDQ10-Q48-S5-D, BCRL_power_supply:CONV_PDQ10-Q48-S5-D, F.Cu at (462.0, 311.3)
- C1, C2, C3, C39, C4, C40, C5, C6: value 4.7uf/100v -> 4.7u
- C10, C11, C12, C13, C14, C15, C16, C17, C18, C19, C20, C21, C22, C23, C24, C25, C26, C27, C28, C29, C30, C7, C8, C9: value 22uf -> 22u
- C100: renamed from C136; value 22uf -> 22u
- C101: renamed from C137; value 100uf -> 100u
- C102: renamed from C138; value 1uf -> 1u
- C103: renamed from C139; value 100uf -> 100u
- C104: renamed from C140; value 1uf -> 1u
- C113, C115: value 100uf -> 22u
- C114, C116: value 1uf -> 22u
- C31: renamed from C67; value 100uf -> 100u
- C32: renamed from C68; value 1uf -> 1u
- C33: renamed from C69; value 100uf -> 100u
- C34: renamed from C70; value 1uf -> 1u
- C35, C36: value 22uf -> 2.2u
- C37: renamed from C41; value 4.7uf/100v -> 4.7u
- C38: renamed from C42; value 4.7uf/100v -> 4.7u
- C43: value 4.7uf/100v -> 1u
- C44: value 4.7uf/100v -> 100u
- C45: value 330uf/100v -> 1u
- C50: renamed from C54; value 4.7uf/100v -> 4.7u
- C51: renamed from C55; value 4.7uf/100v -> 4.7u
- C59: renamed from C58; value 4.7uf/100v -> 4.7u
- C60: renamed from C59; value 4.7uf/100v -> 4.7u
- C61: renamed from C60; value 4.7uf/100v -> 4.7u
- C62: renamed from C61; value 4.7uf/100v -> 4.7u
- C63: renamed from C107; value 22uf -> 22u
- C64: renamed from C108; value 22uf -> 22u
- C65: renamed from C109; value 22uf -> 22u
- C66: renamed from C110; value 22uf -> 22u
- C67: renamed from C111; value 22uf -> 22u
- C68: renamed from C112; value 22uf -> 22u
- C73: renamed from C71; value 4.7uf/100v -> 4.7u
- C74: renamed from C72; value 4.7uf/100v -> 4.7u
- C75: renamed from C73; value 4.7uf/100v -> 4.7u
- C76: renamed from C74; value 4.7uf/100v -> 4.7u
- C77: renamed from C79; value 100uf -> 100u
- C78: renamed from C80; value 1uf -> 1u
- C79: renamed from C81; value 100uf -> 100u
- C80: renamed from C82; value 1uf -> 1u
- C81: renamed from C117; value 22uf -> 22u
- C82: renamed from C118; value 22uf -> 22u
- C83: renamed from C119; value 22uf -> 22u
- C84: renamed from C120; value 22uf -> 22u
- C85: renamed from C121; value 22uf -> 22u
- C86: renamed from C122; value 22uf -> 22u
- C87: renamed from C125; value 22uf -> 22u
- C88: renamed from C126; value 22uf -> 22u
- C89: renamed from C127; value 22uf -> 22u
- C90: renamed from C128; value 22uf -> 22u
- C91: renamed from C129; value 22uf -> 22u
- C92: renamed from C130; value 22uf -> 22u
- C93: renamed from C123; value 4.7uf/100v -> 4.7u
- C94: renamed from C124; value 4.7uf/100v -> 4.7u
- C95: renamed from C131; value 22uf -> 22u
- C96: renamed from C132; value 22uf -> 22u
- C97: renamed from C133; value 22uf -> 22u
- C98: renamed from C134; value 22uf -> 22u
- C99: renamed from C135; value 22uf -> 22u
- D1: renamed from D18; value LED -> LED 0603
- D10, D11, D12, D13, D37, D38: value LED -> LED 0603
- D16: renamed from D19; value LED -> LED 0603
- D17: renamed from D14; value LED -> LED 0603
- D18: renamed from D15; value LED -> LED 0603
- D19: renamed from D16; value LED -> LED 0603
- D2: renamed from D1; value LED -> LED 0603
- D20: renamed from D17; value LED -> LED 0603
- D21: renamed from D30; value LED -> LED 0603
- D22: renamed from D33; value LED -> LED 0603
- D23: renamed from D34; value LED -> LED 0603
- D24: renamed from D35; value LED -> LED 0603
- D3: renamed from D2; value LED -> LED 0603
- D35: renamed from D31; value LED -> LED 0603
- D4: renamed from D3; value LED -> LED 0603
- D5: renamed from D4; value LED -> LED 0603
- D6: renamed from D5; value LED -> LED 0603
- D7: renamed from D6; value LED -> LED 0603
- D8: renamed from D7; value LED -> LED 0603
- D9: renamed from D8; value LED -> LED 0603
- J69, J70, J76, J77: value Conn_01x06_Pin -> Conn_01x02; footprint Connector_PinHeader_2.54mm:PinHeader_1x06_P2.54mm_Vertical -> Connector_PinHeader_2.54mm:PinHeader_1x02_P2.54mm_Vertical
- J78: value Conn_01x06_Pin -> OSTVN02A150; footprint Connector_PinHeader_2.54mm:PinHeader_1x06_P2.54mm_Vertical -> BCRL_power_supply:CONN_OSTVN02A150_OST
- L1, L2: value 4.7uh/3.1a -> 4.7u
- L10: renamed from L14; value 4.7uh/3.1a -> 4.7u
- L11: renamed from L15; value 4.7uh/3.1a -> 4.7u
- L12: renamed from L18; value 4.7uh/3.1a -> 4.7u
- L13: renamed from L19; value 4.7uh/3.1a -> 4.7u
- L14: renamed from L26; value 4.7uh/3.1a -> 4.7u
- L4: renamed from L8; value 4.7uh/3.1a -> 4.7u
- L8: renamed from L12; value 4.7uh/3.1a -> 4.7u
- PS19: value IND108W -> PDQE15-Q48-D24-D; footprint BCRL_power_supply:IND108W -> BCRL_power_supply:CONV_PDQE15-Q48-D24-D
- PS6: value PDQE15-Q48-D24-D -> EHHD010A0B41-HZ; footprint BCRL_power_supply:CONV_PDQE15-Q48-D24-D -> BCRL_power_supply:CONV_EHHD010A0B41-HZ
- R12: value 1k -> 3.4k
- R20: value 3.4k -> 9.59k
- R40: renamed from R18; value 9.59k -> 12.06k
- R44: renamed from R33; value 9.59k -> 12.06k
- R46: renamed from R36; value 9.59k -> 12.06k
- R49: renamed from R46; value 9.59k -> 12.06k
- R63: value 9.59k -> 1k
- moved R12 452.4 mm to (550.7, 303.0)
- moved C39 439.6 mm to (550.7, 295.5)
- moved C40 439.6 mm to (550.7, 298.0)
- moved D10 414.4 mm to (547.6, 227.7)
- moved R62 412.3 mm to (530.8, 227.6)
- moved R13 410.6 mm to (538.0, 228.8)
- moved J44 408.2 mm to (527.1, 235.9)
- moved J69 380.8 mm to (536.4, 235.9)
- moved J70 380.8 mm to (541.0, 235.9)
- moved J78 364.6 mm to (540.5, 223.5)
- moved J77 360.9 mm to (531.7, 221.5)
- moved J76 360.9 mm to (527.1, 221.5)
- moved C113 341.4 mm to (488.6, 203.4)
- moved C114 341.4 mm to (488.6, 205.9)
- moved C115 341.4 mm to (488.6, 208.4)
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- renumbered J38 to J20, J20 to J21, J21 to J22, J22 to J23, J23 to J24, J24 to J25, J25 to J26, J26 to J27, J27 to J28, J28 to J29, J29 to J30, J30 to J31, J31 to J32, J32 to J33, J33 to J34, J34 to J35, J35 to J36, J36 to J37, J37 to J38, J71 to J39, J39 to J40, J40 to J41, J41 to J42, J42 to J43, J45 to J46, J46 to J47, J47 to J48, J48 to J49, J49 to J51, J51 to J52, J52 to J53, J53 to J54, J54 to J55, J55 to J56, J56 to J57, J57 to J58, J58 to J59, J59 to J60, J65 to J62, J62 to J63, J63 to J64, J60 to J65, J64 to J66, J66 to J67, J75 to J68, PS8 to PS10, PS14 to PS11, PS15 to PS12, PS16 to PS13, PS17 to PS14, PS11 to PS5, PS12 to PS8, R25 to R1, R9 to R10, R10 to R11, R1 to R2, R26 to R23, R21 to R24, R22 to R25, R23 to R26, R24 to R27, R55 to R28, R56 to R29, R2 to R3, R57 to R30, R58 to R31, R29 to R32, R35 to R37, R37 to R38, R38 to R39, R3 to R4, R40 to R42, R41 to R43, R4 to R5, R61 to R59, R5 to R6, R6 to R7, R7 to R8, R8 to R9, U11 to U10, U13 to U11, U14 to U12, U15 to U13, U10 to U9
Connections:
- net /Tx_Eth_Switch/CTRL renamed /Eth_Switch/CTRL_Tx
- net /Tx_Eth_Switch/PDQ10-Q48-S5-D_EMC_13/VIN renamed /Eth_Switch/PDQ10-Q48-S5-D_EMC_13/VIN
- C101 pad 1: 48V -> +48V
- C102 pad 1: 48V -> +48V
- C113 pad 1: 48V -> /RxRFswMUXv1 board/+8V_3
- C114 pad 1: 48V -> /RxRFswMUXv1 board/+12V
- C115 pad 1: +12V_2 -> /RxRFswMUXv1 board/+12V
- C116 pad 1: +12V_2 -> /RxRFswMUXv1 board/+12V
- C31 pad 1: 48V -> +48V
- C32 pad 1: 48V -> +48V
- C35 pad 1: /RxRFswMUXv1 board/+12V -> GND
- C35 pad 2: GND -> +48V_unfiltered
- C36 pad 1: /RxRFswMUXv1 board/+12V -> GND
- C36 pad 2: GND -> +48V_unfiltered
- C40 pad 1: /Rx_Eth_Switch/PDQ10-Q48-S5-D_EMC_13/VIN -> /Eth_Switch/PDQ10-Q48-S5-D_EMC_18/VIN
- C43 pad 1: 48V -> +48V
- C44 pad 1: /RPi_HAT/Tx_RPi4_HAT_board1/PDQ10-Q48-S5-D_EMC_8/VIN -> +12V_2
- C45 pad 1: 48V -> +12V_2
- C63 pad 1: /BFN/IND108W_EMC_6.5V_3/+8V -> /BFN/+6.5V_TxBFN_C
- C64 pad 1: /BFN/IND108W_EMC_6.5V_3/+8V -> /BFN/+6.5V_TxBFN_C
- C65 pad 1: /BFN/IND108W_EMC_6.5V_3/+8V -> /BFN/+6.5V_TxBFN_C
- C77 pad 1: 48V -> +48V
- C78 pad 1: 48V -> +48V
- C81 pad 1: /BFN/IND108W_EMC_6.5V_2/+8V -> /BFN/+6.5V_RxBFN_F
- C82 pad 1: /BFN/IND108W_EMC_6.5V_2/+8V -> /BFN/+6.5V_RxBFN_F
- C83 pad 1: /BFN/IND108W_EMC_6.5V_2/+8V -> /BFN/+6.5V_RxBFN_F
- C87 pad 1: /BFN/IND108W_EMC_6.5V_1/+8V -> /BFN/+6.5V_RxBFN_C
- C88 pad 1: /BFN/IND108W_EMC_6.5V_1/+8V -> /BFN/+6.5V_RxBFN_C
- C89 pad 1: /BFN/IND108W_EMC_6.5V_1/+8V -> /BFN/+6.5V_RxBFN_C
- C95 pad 1: /BFN/IND108W_EMC_6.5V_4/+8V -> /BFN/+6.5V_TxBFN_F
- C96 pad 1: /BFN/IND108W_EMC_6.5V_4/+8V -> /BFN/+6.5V_TxBFN_F
- C97 pad 1: /BFN/IND108W_EMC_6.5V_4/+8V -> /BFN/+6.5V_TxBFN_F
- D10 pad 2: /RPi_HAT/+5V_Tx_RPi4_HAT -> /Eth_Switch/+5V_Rx
- D11 pad 2: /RPi_HAT/+24V_Rx_RPi4_HAT -> /BFN/+6.5V_RxBFN_C
- D12 pad 2: /BFN/IND108W_EMC_6.5V_3/+8V -> /BFN/+6.5V_RxBFN_F
- D13 pad 2: /BFN/IND108W_EMC_6.5V_2/+8V -> /BFN/+6.5V_TxBFN_C
- D35 pad 2: /Tx_Eth_Switch/+5V -> /Eth_Switch/+5V_Tx
- D37 pad 2: /RxRFswMUXv1 board/+8V_3 -> /RPi_HAT/+5V
- D38 pad 2: /RxRFswMUXv1 board/+8V_4 -> /RPi_HAT/+24V
- J1 pad 1: +48V -> +48V_unfiltered
- J2 pad 1: +48V -> +48V_unfiltered
- J42 pad 1: /Tx_Eth_Switch/+5V -> /Eth_Switch/+5V_Tx
- J44 pad 1: /Rx_Eth_Switch/CTRL -> /BFN/+12V_CTRL_RxBFN
- J68 pad 2: /RPi_HAT/+5V_Rx_RPi4_HAT -> /RPi_HAT/+5V
- J68 pad 3: /RPi_HAT/+24V_Rx_RPi4_HAT -> /RPi_HAT/+24V
- J69 pad 1: GND -> /BFN/+6.5V_CTRL_RxBFN_F
- J69 pad 2: /RPi_HAT/+5V_Tx_RPi4_HAT -> GND
- J70 pad 1: GND -> /BFN/+12V_CTRL_TxBFN
- J70 pad 2: /RPi_HAT/+5V_Tx_RPi4_HAT -> GND
- J76 pad 1: GND -> /RPi_HAT/+5V_CTRL
- J76 pad 2: /RPi_HAT/+5V_Rx_RPi4_HAT -> GND
- J77 pad 1: GND -> /RPi_HAT/+24V_CTRL
- J77 pad 2: /RPi_HAT/+5V_Rx_RPi4_HAT -> GND
- J78 pad 1: GND -> /Eth_Switch/+5V_Rx
- J78 pad 2: /RPi_HAT/+5V_Rx_RPi4_HAT -> GND
- PS10 pad 1: 48V -> +48V
- PS11 pad 1: /BFN/IND108W_EMC_6.5V_2/+8V_CTRL -> /BFN/+6.5V_CTRL_RxBFN_F
- PS11 pad 3: /BFN/IND108W_EMC_6.5V_2/+8V -> /BFN/+6.5V_RxBFN_F
- PS11 pad 5: /BFN/IND108W_EMC_6.5V_2/+8V -> /BFN/+6.5V_RxBFN_F
- PS12 pad 1: /BFN/IND108W_EMC_6.5V_1/+8V_CTRL -> /BFN/+6.5V_CTRL_RxBFN_C
- PS12 pad 3: /BFN/IND108W_EMC_6.5V_1/+8V -> /BFN/+6.5V_RxBFN_C
- PS12 pad 5: /BFN/IND108W_EMC_6.5V_1/+8V -> /BFN/+6.5V_RxBFN_C
- PS13 pad 1: /BFN/IND108W_EMC_6.5V_4/+8V_CTRL -> /BFN/+6.5V_CTRL_TxBFN_F
- PS13 pad 3: /BFN/IND108W_EMC_6.5V_4/+8V -> /BFN/+6.5V_TxBFN_F
- PS13 pad 5: /BFN/IND108W_EMC_6.5V_4/+8V -> /BFN/+6.5V_TxBFN_F
- PS14 pad 1: 48V -> +48V
- PS18 pad 1: /RxRFswMUXv1 board/RxLNA2_8V_CTRL -> /RxRFswMUXv1 board/RxLNA4_8V_CTRL
- PS18 pad 3: /RxRFswMUXv1 board/+8V_2 -> /RxRFswMUXv1 board/+8V_4
- PS18 pad 5: /RxRFswMUXv1 board/+8V_2 -> /RxRFswMUXv1 board/+8V_4
- PS19 pad 1: /RxRFswMUXv1 board/RxLNA3_8V_CTRL -> /RPi_HAT/+24V_CTRL
- PS19 pad 3: /RxRFswMUXv1 board/+8V_3 -> /RPi_HAT/PDQE15-Q48-D24-D_EMC_2/VIN
- PS19 pad 4: Net-(PS19-TRIM) -> /RPi_HAT/+24V
- PS19 pad 5: /RxRFswMUXv1 board/+8V_3 -> GND
- PS19 pad 6: GND -> unconnected-(PS19--VO-Pad6)
- PS5 pad 1: 48V -> +48V
- PS5 pad 2: /BFN/EHHD010A0B41-HZ1/ON/OFF -> /BFN/+12V_CTRL_RxBFN
- PS6 pad 1: /RPi_HAT/Tx_RPi4_HAT_board1/+24V_CTRL -> +48V
- PS6 pad 2: GND -> /BFN/+12V_CTRL_TxBFN
- PS6 pad 3: /RPi_HAT/Tx_RPi4_HAT_board1/PDQE15-Q48-D24-D_EMC_1/VIN -> GND
- PS6 pad 4: /RPi_HAT/+24V_Tx_RPi4_HAT -> GND
- PS6 pad 5: GND -> unconnected-(PS6-SENSE--Pad5)
- PS8 pad 1: /BFN/IND108W_EMC_6.5V_3/+8V_CTRL -> /BFN/+6.5V_CTRL_TxBFN_C
- PS8 pad 3: /BFN/IND108W_EMC_6.5V_3/+8V -> /BFN/+6.5V_TxBFN_C
- PS8 pad 5: /BFN/IND108W_EMC_6.5V_3/+8V -> /BFN/+6.5V_TxBFN_C
- R12 pad 2: Net-(D10-K) -> Net-(U6-TRIM)
- R13 pad 2: Net-(D11-K) -> Net-(D10-K)
- R15 pad 2: Net-(D25-K) -> Net-(D11-K)
- R17 pad 2: Net-(D26-K) -> Net-(D12-K)
- R19 pad 2: Net-(D12-K) -> Net-(D13-K)
- R20 pad 1: GND -> Net-(PS4-TRIM)
- R20 pad 2: Net-(U4-TRIM) -> GND
- R51 pad 1: Net-(PS4-TRIM) -> Net-(PS15-TRIM)
- R62 pad 2: Net-(D32-K) -> Net-(D37-K)
- R63 pad 1: Net-(PS19-TRIM) -> GND
- R63 pad 2: GND -> Net-(D38-K)
- U5 pad 3: /Tx_Eth_Switch/+5V -> /Eth_Switch/PDQ10-Q48-S5-D_EMC_13/+5V
- U6 pad 1: /RPi_HAT/Tx_RPi4_HAT_board1/PDQ10-Q48-S5-D_EMC_8/VIN -> /Eth_Switch/PDQ10-Q48-S5-D_EMC_18/VIN
- U6 pad 3: /RPi_HAT/+5V_Tx_RPi4_HAT -> /Eth_Switch/+5V_Rx
- U6 pad 6: /RPi_HAT/Tx_RPi4_HAT_board1/+5V_CTRL -> /Eth_Switch/CTRL_Rx

Commit message: digikey BOM
Parts:
- removed C131, C134: 330u, Capacitor_SMD:C_0603_1608Metric
- removed C137: 47u, Capacitor_SMD:C_0603_1608Metric
- added C46: 330u, Capacitor_THT:CP_Radial_D12.5mm_P5.00mm, F.Cu at (373.5, 139.7)
- added C47: 330u, Capacitor_THT:CP_Radial_D12.5mm_P5.00mm, F.Cu at (373.5, 153.8)
- added C48: 47u, Capacitor_THT:CP_Radial_D12.5mm_P5.00mm, F.Cu at (373.5, 167.8)
- C1, C129, C130, C132, C133, C2, C3, C37, C38, C39, C4, C40, C5, C50, C51, C59, C6, C60, C61, C62, C73, C74, C75, C76, C93, C94: value 4.7u -> 4.7u; footprint Capacitor_SMD:C_0603_1608Metric -> Capacitor_SMD:C_1206_3216Metric
- C10, C100, C105, C106, C107, C108, C109, C11, C110, C111, C112, C113, C114, C115, C116, C117, C118, C119, C12, C120, C121, C122, C123, C124, C125, C126, C127, C128, C13, C14, C15, C16, C17, C18, C19, C20, C21, C22, C23, C24, C25, C26, C27, C28, C29, C30, C35, C36, C41, C63, C64, C65, C66, C67, C68, C7, C8, C81, C82, C83, C84, C85, C86, C87, C88, C89, C9, C90, C91, C92, C95, C96, C97, C98, C99: footprint Capacitor_SMD:C_0603_1608Metric -> Capacitor_SMD:C_1206_3216Metric
- C101, C103, C31, C33, C42, C44, C77, C79: value 100u -> 47u; footprint Capacitor_SMD:C_0603_1608Metric -> Capacitor_THT:CP_Radial_D12.5mm_P5.00mm
