File: kicad_files/bcrl_power_supply/PDQE15-Q48-D24-D_EMC.kicad_sch (KiCad schematic)
At the start: 9 parts

Commit message: ...
Parts:
- PS18: renamed from PS19; footprint PDQE15-Q48-D24-D:CONV_PDQE15-Q48-D24-D -> BCRL_power_supply:CONV_PDQE15-Q48-D24-D
- renumbered C1 to C146, C2 to C147, C147 to C148, C91 to C149, C109 to C150, C41 to C151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
Connections:
- net VIN: now reaches C147.1, C148.1, C149.1, L42.2, PS18.3 (VIN)
