File: kicad_files/bcrl_power_supply/PDQE15-Q48-D24-D_EMC.kicad_sch (KiCad schematic)
At the start: 9 parts

Commit message: big reorg
Parts:
- renumbered C145 to C45, C146 to C46, C147 to C47, C148 to C48, C149 to C49, C150 to C50, C151 to C51, L42 to L10, PS18 to PS5
Changed lines of the file:
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@@
 		(dnp no)
 		(fields_autoplaced yes)
-		(property "Reference" "#PWR0210"
+		(property "Reference" "#PWR0201"
 			(at 41.275 110.49 0)
 			(effects
@@
 		(instances
 			(project "bcrl_power_supply"
-				(path "/77f0f57c-9586-4625-9281-fa8cbd8015db/a85e3a44-afc6-43fc-a4d8-d3c8f12cb5cc/90beb04a-7ddb-4e1c-b4d9-8871b13e8ee0"
-					(reference "#PWR0210")
-					(unit 1)
-				)
-				(path "/77f0f57c-9586-4625-9281-fa8cbd8015db/b08c53be-3c36-4aa7-b4db-fe44d17a238c/90beb04a-7ddb-4e1c-b4d9-8871b13e8ee0"
-					(reference "#PWR0249")
+				(path "/77f0f57c-9586-4625-9281-fa8cbd8015db/74d0f335-4d3b-4aa7-8bba-06f11ca9d6fc/90beb04a-7ddb-4e1c-b4d9-8871b13e8ee0"
+					(reference "#PWR0201")
+					(unit 1)
+				)
+				(path "/77f0f57c-9586-4625-9281-fa8cbd8015db/3e577bd7-c793-4d4a-9991-32d1d0bab64c/90beb04a-7ddb-4e1c-b4d9-8871b13e8ee0"
+					(reference "#PWR0304")
 					(unit 1)
 				)
@@
 		(dnp no)
 		(fields_autoplaced yes)
-		(property "Reference" "#PWR0211"
+		(property "Reference" "#PWR0202"
 			(at 153.67 102.87 0)
 			(effects
@@
 		(instances
 			(project "bcrl_power_supply"
-				(path "/77f0f57c-9586-4625-9281-fa8cbd8015db/a85e3a44-afc6-43fc-a4d8-d3c8f12cb5cc/90beb04a-7ddb-4e1c-b4d9-8871b13e8ee0"
-					(reference "#PWR0211")
-					(unit 1)
-				)
-				(path "/77f0f57c-9586-4625-9281-fa8cbd8015db/b08c53be-3c36-4aa7-b4db-fe44d17a238c/90beb04a-7ddb-4e1c-b4d9-8871b13e8ee0"
-					(reference "#PWR0250")
+				(path "/77f0f57c-9586-4625-9281-fa8cbd8015db/74d0f335-4d3b-4aa7-8bba-06f11ca9d6fc/90beb04a-7ddb-4e1c-b4d9-8871b13e8ee0"
+					(reference "#PWR0202")
+					(unit 1)
+				)
+				(path "/77f0f57c-9586-4625-9281-fa8cbd8015db/3e577bd7-c793-4d4a-9991-32d1d0bab64c/90beb04a-7ddb-4e1c-b4d9-8871b13e8ee0"
+					(reference "#PWR0305")
 					(unit 1)
 				)
@@
 		(dnp no)
 		(fields_autoplaced yes)
-		(property "Reference" "C146"
+		(property "Reference" "C46"
 			(at 67.31 95.25 0)
 			(effects
@@
 		(instances
 			(project "bcrl_power_supply"
-				(path "/77f0f57c-9586-4625-9281-fa8cbd8015db/a85e3a44-afc6-43fc-a4d8-d3c8f12cb5cc/90beb04a-7ddb-4e1c-b4d9-8871b13e8ee0"
-					(reference "C146")
-					(unit 1)
-				)
-				(path "/77f0f57c-9586-4625-9281-fa8cbd8015db/b08c53be-3c36-4aa7-b4db-fe44d17a238c/90beb04a-7ddb-4e1c-b4d9-8871b13e8ee0"
-					(reference "C163")
+				(path "/77f0f57c-9586-4625-9281-fa8cbd8015db/74d0f335-4d3b-4aa7-8bba-06f11ca9d6fc/90beb04a-7ddb-4e1c-b4d9-8871b13e8ee0"
+					(reference "C46")
+					(unit 1)
+				)
+				(path "/77f0f57c-9586-4625-9281-fa8cbd8015db/3e577bd7-c793-4d4a-9991-32d1d0bab64c/90beb04a-7ddb-4e1c-b4d9-8871b13e8ee0"
+					(reference "C188")
 					(unit 1)
 				)
@@
 		(dnp no)
 		(fields_autoplaced yes)
-		(property "Reference" "C151"
+		(property "Reference" "C51"
 			(at 157.48 91.44 0)
 			(effects
@@
 		(instances
 			(project "bcrl_power_supply"
-				(path "/77f0f57c-9586-4625-9281-fa8cbd8015db/a85e3a44-afc6-43fc-a4d8-d3c8f12cb5cc/90beb04a-7ddb-4e1c-b4d9-8871b13e8ee0"
-					(reference "C151")
-					(unit 1)
-				)
-				(path "/77f0f57c-9586-4625-9281-fa8cbd8015db/b08c53be-3c36-4aa7-b4db-fe44d17a238c/90beb04a-7ddb-4e1c-b4d9-8871b13e8ee0"
-					(reference "C168")
+				(path "/77f0f57c-9586-4625-9281-fa8cbd8015db/74d0f335-4d3b-4aa7-8bba-06f11ca9d6fc/90beb04a-7ddb-4e1c-b4d9-8871b13e8ee0"
+					(reference "C51")
+					(unit 1)
+				)
+				(path "/77f0f57c-9586-4625-9281-fa8cbd8015db/3e577bd7-c793-4d4a-9991-32d1d0bab64c/90beb04a-7ddb-4e1c-b4d9-8871b13e8ee0"
+					(reference "C193")
 					(unit 1)
 				)
@@
 		(dnp no)
 		(fields_autoplaced yes)
-		(property "Reference" "C149"
+		(property "Reference" "C49"
 			(at 132.715 67.31 90)
 			(effects
@@
 		(instances
 			(project "bcrl_power_supply"
-				(path "/77f0f57c-9586-4625-9281-fa8cbd8015db/a85e3a44-afc6-43fc-a4d8-d3c8f12cb5cc/90beb04a-7ddb-4e1c-b4d9-8871b13e8ee0"
-					(reference "C149")
-					(unit 1)
-				)
-				(path "/77f0f57c-9586-4625-9281-fa8cbd8015db/b08c53be-3c36-4aa7-b4db-fe44d17a238c/90beb04a-7ddb-4e1c-b4d9-8871b13e8ee0"
-					(reference "C166")
+				(path "/77f0f57c-9586-4625-9281-fa8cbd8015db/74d0f335-4d3b-4aa7-8bba-06f11ca9d6fc/90beb04a-7ddb-4e1c-b4d9-8871b13e8ee0"
+					(reference "C49")
+					(unit 1)
+				)
+				(path "/77f0f57c-9586-4625-9281-fa8cbd8015db/3e577bd7-c793-4d4a-9991-32d1d0bab64c/90beb04a-7ddb-4e1c-b4d9-8871b13e8ee0"
+					(reference "C191")
 					(unit 1)
 				)
@@
 		(dnp no)
 		(fields_autoplaced yes)
-		(property "Reference" "PS18"
+		(property "Reference" "PS5"
 			(at 132.715 81.28 0)
 			(effects
@@
 		(instances
 			(project "bcrl_power_supply"
-				(path "/77f0f57c-9586-4625-9281-fa8cbd8015db/a85e3a44-afc6-43fc-a4d8-d3c8f12cb5cc/90beb04a-7ddb-4e1c-b4d9-8871b13e8ee0"
-					(reference "PS18")
-					(unit 1)
-				)
-				(path "/77f0f57c-9586-4625-9281-fa8cbd8015db/b08c53be-3c36-4aa7-b4db-fe44d17a238c/90beb04a-7ddb-4e1c-b4d9-8871b13e8ee0"
-					(reference "PS20")
+				(path "/77f0f57c-9586-4625-9281-fa8cbd8015db/74d0f335-4d3b-4aa7-8bba-06f11ca9d6fc/90beb04a-7ddb-4e1c-b4d9-8871b13e8ee0"
+					(reference "PS5")
+					(unit 1)
+				)
+				(path "/77f0f57c-9586-4625-9281-fa8cbd8015db/3e577bd7-c793-4d4a-9991-32d1d0bab64c/90beb04a-7ddb-4e1c-b4d9-8871b13e8ee0"
+					(reference "PS21")
 					(unit 1)
 				)
@@
 		(dnp no)
 		(fields_autoplaced yes)
-		(property "Reference" "C150"
+		(property "Reference" "C50"
 			(at 134.62 104.14 90)
 			(effects
@@
 		(instances
 			(project "bcrl_power_supply"
-				(path "/77f0f57c-9586-4625-9281-fa8cbd8015db/a85e3a44-afc6-43fc-a4d8-d3c8f12cb5cc/90beb04a-7ddb-4e1c-b4d9-8871b13e8ee0"
-					(reference "C150")
-					(unit 1)
-				)
-				(path "/77f0f57c-9586-4625-9281-fa8cbd8015db/b08c53be-3c36-4aa7-b4db-fe44d17a238c/90beb04a-7ddb-4e1c-b4d9-8871b13e8ee0"
-					(reference "C167")
+				(path "/77f0f57c-9586-4625-9281-fa8cbd8015db/74d0f335-4d3b-4aa7-8bba-06f11ca9d6fc/90beb04a-7ddb-4e1c-b4d9-8871b13e8ee0"
+					(reference "C50")
+					(unit 1)
+				)
+				(path "/77f0f57c-9586-4625-9281-fa8cbd8015db/3e577bd7-c793-4d4a-9991-32d1d0bab64c/90beb04a-7ddb-4e1c-b4d9-8871b13e8ee0"
+					(reference "C192")
 					(unit 1)
 				)
@@
 		(dnp no)
 		(fields_autoplaced yes)
-		(property "Reference" "C148"
+		(property "Reference" "C48"
 			(at 102.235 95.25 0)
 			(effects
@@
 		(instances
 			(project "bcrl_power_supply"
-				(path "/77f0f57c-9586-4625-9281-fa8cbd8015db/a85e3a44-afc6-43fc-a4d8-d3c8f12cb5cc/90beb04a-7ddb-4e1c-b4d9-8871b13e8ee0"
-					(reference "C148")
-					(unit 1)
-				)
-				(path "/77f0f57c-9586-4625-9281-fa8cbd8015db/b08c53be-3c36-4aa7-b4db-fe44d17a238c/90beb04a-7ddb-4e1c-b4d9-8871b13e8ee0"
-					(reference "C165")
+				(path "/77f0f57c-9586-4625-9281-fa8cbd8015db/74d0f335-4d3b-4aa7-8bba-06f11ca9d6fc/90beb04a-7ddb-4e1c-b4d9-8871b13e8ee0"
+					(reference "C48")
+					(unit 1)
+				)
+				(path "/77f0f57c-9586-4625-9281-fa8cbd8015db/3e577bd7-c793-4d4a-9991-32d1d0bab64c/90beb04a-7ddb-4e1c-b4d9-8871b13e8ee0"
+					(reference "C190")
 					(unit 1)
 				)
@@
 		(dnp no)
 		(fields_autoplaced yes)
-		(property "Reference" "L42"
+		(property "Reference" "L10"
 			(at 72.39 83.82 90)
 			(effects
@@
 		(instances
 			(project "bcrl_power_supply"
-				(path "/77f0f57c-9586-4625-9281-fa8cbd8015db/a85e3a44-afc6-43fc-a4d8-d3c8f12cb5cc/90beb04a-7ddb-4e1c-b4d9-8871b13e8ee0"
-					(reference "L42")
-					(unit 1)
-				)
-				(path "/77f0f57c-9586-4625-9281-fa8cbd8015db/b08c53be-3c36-4aa7-b4db-fe44d17a238c/90beb04a-7ddb-4e1c-b4d9-8871b13e8ee0"
-					(reference "L46")
+				(path "/77f0f57c-9586-4625-9281-fa8cbd8015db/74d0f335-4d3b-4aa7-8bba-06f11ca9d6fc/90beb04a-7ddb-4e1c-b4d9-8871b13e8ee0"
+					(reference "L10")
+					(unit 1)
+				)
+				(path "/77f0f57c-9586-4625-9281-fa8cbd8015db/3e577bd7-c793-4d4a-9991-32d1d0bab64c/90beb04a-7ddb-4e1c-b4d9-8871b13e8ee0"
+					(reference "L35")
 					(unit 1)
 				)
@@
 		(dnp no)
 		(fields_autoplaced yes)
-		(property "Reference" "C145"
+		(property "Reference" "C45"
 			(at 48.895 95.885 0)
 			(effects
@@
 		(instances
 			(project "bcrl_power_supply"
-				(path "/77f0f57c-9586-4625-9281-fa8cbd8015db/a85e3a44-afc6-43fc-a4d8-d3c8f12cb5cc/90beb04a-7ddb-4e1c-b4d9-8871b13e8ee0"
-					(reference "C145")
-					(unit 1)
-				)
-				(path "/77f0f57c-9586-4625-9281-fa8cbd8015db/b08c53be-3c36-4aa7-b4db-fe44d17a238c/90beb04a-7ddb-4e1c-b4d9-8871b13e8ee0"
-					(reference "C162")
+				(path "/77f0f57c-9586-4625-9281-fa8cbd8015db/74d0f335-4d3b-4aa7-8bba-06f11ca9d6fc/90beb04a-7ddb-4e1c-b4d9-8871b13e8ee0"
+					(reference "C45")
+					(unit 1)
+				)
+				(path "/77f0f57c-9586-4625-9281-fa8cbd8015db/3e577bd7-c793-4d4a-9991-32d1d0bab64c/90beb04a-7ddb-4e1c-b4d9-8871b13e8ee0"
+					(reference "C187")
 					(unit 1)
 				)
@@
 		(dnp no)
 		(fields_autoplaced yes)
-		(property "Reference" "C147"
+		(property "Reference" "C47"
 			(at 83.82 95.25 0)
 			(effects
@@
 		(instances
 			(project "bcrl_power_supply"
-				(path "/77f0f57c-9586-4625-9281-fa8cbd8015db/a85e3a44-afc6-43fc-a4d8-d3c8f12cb5cc/90beb04a-7ddb-4e1c-b4d9-8871b13e8ee0"
-					(reference "C147")
-					(unit 1)
-				)
-				(path "/77f0f57c-9586-4625-9281-fa8cbd8015db/b08c53be-3c36-4aa7-b4db-fe44d17a238c/90beb04a-7ddb-4e1c-b4d9-8871b13e8ee0"
-					(reference "C164")
-					(unit 1)
-				)
+				(path "/77f0f57c-9586-4625-9281-fa8cbd8015db/74d0f335-4d3b-4aa7-8bba-06f11ca9d6fc/90beb04a-7ddb-4e1c-b4d9-8871b13e8ee0"
+					(reference "C47")
+					(unit 1)
+				)
+				(path "/77f0f57c-9586-4625-9281-fa8cbd8015db/3e577bd7-c793-4d4a-9991-32d1d0bab64c/90beb04a-7ddb-4e1c-b4d9-8871b13e8ee0"
+					(reference "C189")
+					(unit 1)
+				)
