File: kicad_files/bcrl_power_supply/PDQE15-Q48-D24-D_EMC.kicad_sch (KiCad schematic)
At the start: 9 parts

Commit message: almost done schematic
Parts:
- C131: renamed from C45; value 330uf/100v -> 330u; rating (none) -> 100v
- C132: renamed from C46; value 4.7uf/100v -> 4.7u; rating (none) -> 100v
- C133: renamed from C47; value 4.7uf/100v -> 4.7u; rating (none) -> 100v
- C134: renamed from C48; value 330uf/100v -> 330u; rating (none) -> 100v
- C135: renamed from C49; value 1nf/2kv -> 1nf; rating (none) -> 2kv
- C136: renamed from C50; value 1nf/2kv -> 1nf; rating (none) -> 2kv
- C137: renamed from C51; value 47uf/50v -> 47u; rating (none) -> 50v
- L16: renamed from L10; value 4.7uh/3.1a -> 4.7u; rating (none) -> 3.1a
- renumbered PS5 to PS19

Commit message: digikey BOM
Parts:
- removed C131, C134: 330u, Capacitor_SMD:C_0603_1608Metric, symbol Device:C
- removed C137: 47u, Capacitor_SMD:C_0603_1608Metric, symbol Device:C
- added C46, C47: 330u, Capacitor_THT:CP_Radial_D12.5mm_P5.00mm, symbol Device:C_Polarized
- added C48: 47u, Capacitor_THT:CP_Radial_D12.5mm_P5.00mm, symbol Device:C_Polarized
- C132, C133: value 4.7u -> 4.7u; footprint Capacitor_SMD:C_0603_1608Metric -> Capacitor_SMD:C_1206_3216Metric; DigiKey_Part_Number (none) -> GRM31CC72A475KE11L
- C135, C136: DigiKey_Part_Number (none) -> CGP5C102KGYDAA7301
- L16: DigiKey_Part_Number (none) -> MGAH06034R7M-10
- PS19: DigiKey_Part_Number (none) -> PDQE15-Q48-D24-D
Connections:
- net +24V: now also C48.1
- net 48V: now also C46.1
- net GND: now also C46.2, C47.2, C48.2
- net VIN: now also C47.1
Other:
- note added: "https://www.cui.com/product/resource/pdqe15-d.pdf"
- moved on the sheet: C135, PS19
