File: kicad_files/bcrl_power_supply/AGC_board.kicad_sch (KiCad schematic)
At the start: 1 part, among them J75 Conn_01x04_Pin

Commit message: WIP
Connections:
- net VCC_shared: no longer names the net of J75.3 (Pin_3)
Changed lines of the file:
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@@
     (stroke (width 0) (type default))
-  )
-  (label "VCC_shared" (at 50.165 47.625 0) (fields_autoplaced)
-    (effects (font (size 1.27 1.27)) (justify left bottom))
   )
   (label "+6.5V" (at 49.53 45.085 0) (fields_autoplaced)

Commit message: cleanup PCB
Parts:
- J63: renamed from J75; footprint (none) -> Connector_PinHeader_2.54mm:PinHeader_1x04_P2.54mm_Vertical
Connections:
- net +6.5V: now also J63.3 (Pin_3)
Changed lines of the file:
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@@
 (kicad_sch (version 20230121) (generator eeschema)
   (paper "A4")
+  (junction (at 37.465 45.085) (diameter 0) (color 0 0 0 0)
+  )
   (wire (pts (xy 49.53 45.085) (xy 37.465 45.085))
     (stroke (width 0) (type default))
@@
     (stroke (width 0) (type default))
   )
-  (wire (pts (xy 37.465 47.625) (xy 50.165 47.625))
-    (stroke (width 0) (type default))
-  )
   (wire (pts (xy 39.37 42.545) (xy 37.465 42.545))
     (stroke (width 0) (type default))
   )
-  (label "+6.5V" (at 49.53 45.085 0) (fields_autoplaced)
-    (effects (font (size 1.27 1.27)) (justify left bottom))
+  (wire (pts (xy 37.465 45.085) (xy 37.465 47.625))
+    (stroke (width 0) (type default))
+  )
+  (hierarchical_label "+6.5V" (shape input) (at 49.53 45.085 0) (fields_autoplaced)
+    (effects (font (size 1.27 1.27)) (justify left))
   )
   (symbol (lib_id "Connector:Conn_01x04_Pin") (at 32.385 45.085 0) (unit 1)
     (in_bom yes) (on_board yes) (dnp no) (fields_autoplaced)
-    (property "Reference" "J75" (at 33.02 37.465 0)
+    (property "Reference" "J63" (at 33.02 37.465 0)
       (effects (font (size 1.27 1.27)))
     )
@@
       (effects (font (size 1.27 1.27)))
     )
-    (property "Footprint" "" (at 32.385 45.085 0)
+    (property "Footprint" "Connector_PinHeader_2.54mm:PinHeader_1x04_P2.54mm_Vertical" (at 32.385 45.085 0)
       (effects (font (size 1.27 1.27)) hide)
     )
@@
       (project "bcrl_power_supply"
         (path "/77f0f57c-9586-4625-9281-fa8cbd8015db/7ab5448f-bd34-4432-b359-f13f98fccb68"
-          (reference "J75") (unit 1)
+          (reference "J63") (unit 1)
         )
         (path "/77f0f57c-9586-4625-9281-fa8cbd8015db/3eea0769-b0fa-4084-b012-c895759d5215"
-          (reference "J76") (unit 1)
+          (reference "J64") (unit 1)
         )
       )
@@
   (symbol (lib_id "power:GND") (at 39.37 50.165 90) (unit 1)
     (in_bom yes) (on_board yes) (dnp no) (fields_autoplaced)
-    (property "Reference" "#PWR0254" (at 45.72 50.165 0)
+    (property "Reference" "#PWR0220" (at 45.72 50.165 0)
       (effects (font (size 1.27 1.27)) hide)
     )
@@
       (project "bcrl_power_supply"
         (path "/77f0f57c-9586-4625-9281-fa8cbd8015db/7ab5448f-bd34-4432-b359-f13f98fccb68"
-          (reference "#PWR0254") (unit 1)
+          (reference "#PWR0220") (unit 1)
         )
         (path "/77f0f57c-9586-4625-9281-fa8cbd8015db/3eea0769-b0fa-4084-b012-c895759d5215"
-          (reference "#PWR0256") (unit 1)
+          (reference "#PWR0224") (unit 1)
         )
       )
@@
   (symbol (lib_id "power:GND") (at 39.37 42.545 90) (unit 1)
     (in_bom yes) (on_board yes) (dnp no) (fields_autoplaced)
-    (property "Reference" "#PWR0253" (at 45.72 42.545 0)
+    (property "Reference" "#PWR0219" (at 45.72 42.545 0)
       (effects (font (size 1.27 1.27)) hide)
     )
@@
       (project "bcrl_power_supply"
         (path "/77f0f57c-9586-4625-9281-fa8cbd8015db/7ab5448f-bd34-4432-b359-f13f98fccb68"
-          (reference "#PWR0253") (unit 1)
+          (reference "#PWR0219") (unit 1)
         )
         (path "/77f0f57c-9586-4625-9281-fa8cbd8015db/3eea0769-b0fa-4084-b012-c895759d5215"
-          (reference "#PWR0255") (unit 1)
+          (reference "#PWR0223") (unit 1)
         )
       )

Commit message: ...
Parts:
- renumbered J63 to J59

Commit message: schematic done
Other:
- moved on the sheet: J59
Changed lines of the file:
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@@
 	(paper "A4")
 	(junction
-		(at 37.465 45.085)
+		(at 38.1 45.72)
 		(diameter 0)
 		(color 0 0 0 0)
@@
 	(wire
 		(pts
-			(xy 49.53 45.085) (xy 37.465 45.085)
-		)
-		(stroke
-			(width 0)
-			(type default)
-		)
-	)
-	(wire
-		(pts
-			(xy 39.37 50.165) (xy 37.465 50.165)
-		)
-		(stroke
-			(width 0)
-			(type default)
-		)
-	)
-	(wire
-		(pts
-			(xy 39.37 42.545) (xy 37.465 42.545)
-		)
-		(stroke
-			(width 0)
-			(type default)
-		)
-	)
-	(wire
-		(pts
-			(xy 37.465 45.085) (xy 37.465 47.625)
+			(xy 49.53 45.72) (xy 38.1 45.72)
+		)
+		(stroke
+			(width 0)
+			(type default)
+		)
+	)
+	(wire
+		(pts
+			(xy 39.37 50.8) (xy 38.1 50.8)
+		)
+		(stroke
+			(width 0)
+			(type default)
+		)
+	)
+	(wire
+		(pts
+			(xy 39.37 43.18) (xy 38.1 43.18)
+		)
+		(stroke
+			(width 0)
+			(type default)
+		)
+	)
+	(wire
+		(pts
+			(xy 38.1 45.72) (xy 38.1 48.26)
 		)
 		(stroke
@@
 	(hierarchical_label "+6.5V"
 		(shape input)
-		(at 49.53 45.085 0)
+		(at 49.53 45.72 0)
 		(fields_autoplaced yes)
 		(effects
@@
 	(symbol
 		(lib_id "Connector:Conn_01x04_Pin")
-		(at 32.385 45.085 0)
+		(at 33.02 45.72 0)
 		(unit 1)
 		(exclude_from_sim no)
@@
 		(fields_autoplaced yes)
 		(property "Reference" "J59"
-			(at 33.02 37.465 0)
+			(at 33.655 38.1 0)
 			(effects
 				(font
@@
 		)
 		(property "Value" "Conn_01x04_Pin"
-			(at 33.02 40.005 0)
+			(at 33.655 40.64 0)
 			(effects
 				(font
@@
 		)
 		(property "Footprint" "Connector_PinHeader_2.54mm:PinHeader_1x04_P2.54mm_Vertical"
-			(at 32.385 45.085 0)
+			(at 33.02 45.72 0)
 			(effects
 				(font
@@
 		)
 		(property "Datasheet" "~"
-			(at 32.385 45.085 0)
+			(at 33.02 45.72 0)
 			(effects
 				(font
@@
 		)
 		(property "Description" ""
-			(at 32.385 45.085 0)
+			(at 33.02 45.72 0)
 			(effects
 				(font
@@
 	(symbol
 		(lib_id "power:GND")
-		(at 39.37 50.165 90)
+		(at 39.37 50.8 90)
 		(unit 1)
 		(exclude_from_sim no)
@@
 		(fields_autoplaced yes)
 		(property "Reference" "#PWR0196"
-			(at 45.72 50.165 0)
+			(at 45.72 50.8 0)
 			(effects
 				(font
@@
 		)
 		(property "Value" "GND"
-			(at 43.18 50.165 90)
+			(at 43.18 50.8 90)
 			(effects
 				(font
@@
 		)
 		(property "Footprint" ""
-			(at 39.37 50.165 0)
+			(at 39.37 50.8 0)
 			(effects
 				(font
@@
 		)
 		(property "Datasheet" ""
-			(at 39.37 50.165 0)
+			(at 39.37 50.8 0)
 			(effects
 				(font
@@
 		)
 		(property "Description" ""
-			(at 39.37 50.165 0)
+			(at 39.37 50.8 0)
 			(effects
 				(font
@@
 	(symbol
 		(lib_id "power:GND")
-		(at 39.37 42.545 90)
+		(at 39.37 43.18 90)
 		(unit 1)
 		(exclude_from_sim no)
@@
 		(fields_autoplaced yes)
 		(property "Reference" "#PWR0195"
-			(at 45.72 42.545 0)
+			(at 45.72 43.18 0)
 			(effects
 				(font
@@
 		)
 		(property "Value" "GND"
-			(at 43.18 42.545 90)
+			(at 43.18 43.18 90)
 			(effects
 				(font
@@
 		)
 		(property "Footprint" ""
-			(at 39.37 42.545 0)
+			(at 39.37 43.18 0)
 			(effects
 				(font
@@
 		)
 		(property "Datasheet" ""
-			(at 39.37 42.545 0)
+			(at 39.37 43.18 0)
 			(effects
 				(font
@@
 		)
 		(property "Description" ""
-			(at 39.37 42.545 0)
-			(effects
-				(font
+			(at 39.37 43.18 0)
+			(effects
+				(font

Commit message: big reorg
Parts:
- removed J59: Conn_01x04_Pin, Connector_PinHeader_2.54mm:PinHeader_1x04_P2.54mm_Vertical, symbol Connector:Conn_01x04_Pin
