File: kicad_files/bcrl_power_supply/PQC50-48-S5-O_EMC_trimmed.kicad_sch (KiCad schematic)
At the start: 15 parts

Commit message: cleanup PCB
Parts:
- L4: renamed from L5; footprint (none) -> Inductor_SMD:L_0603_1608Metric
- L5: renamed from L6; footprint (none) -> Inductor_SMD:L_0603_1608Metric
- RV1: footprint (none) -> Potentiometer_THT:Potentiometer_ACP_CA9-V10_Vertical
- renumbered C28 to C10, C29 to C11, C30 to C12, C31 to C13, C32 to C14, C33 to C15, C34 to C16, C27 to C9, PS6 to PS2, R1 to R12, R2 to R13, R3 to R14
Connections:
- net GND: no longer C14.2, C16.1, PS2.7 (SENSE+), PS2.8 (+VO), R13.1
- new net +VO: C14.2, C16.1, PS2.7 (SENSE+), PS2.8 (+VO), R13.1

Commit message: ...
Parts:
- removed R12, R13, R14: R, Resistor_SMD:R_0603_1608Metric, symbol Device:R
Connections:
- net +VO: now also RV1.1
- net GND: no longer RV1.1
- net VIN: now reaches C12.1, C13.1, C14.1, L4.2, PS2.1 (VIN)
- no-connect marks 0 -> 1
Other:
- moved on the sheet: RV1

Commit message: almost done schematic
Parts:
- removed RV1: R_Potentiometer_Trim, Potentiometer_THT:Potentiometer_ACP_CA9-V10_Vertical, symbol Device:R_Potentiometer_Trim
- added R39: 168k, symbol Device:R
Connections:
- net +VO: now also R39.1
- net at PS2.6 (TRIM): now also R39.2
- no-connect marks 1 -> 0

Commit message: schematic done
Parts:
- R39: footprint (none) -> Resistor_SMD:R_0603_1608Metric
Changed lines of the file:
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@@
 			)
 		)
-		(property "Footprint" ""
+		(property "Footprint" "Resistor_SMD:R_0603_1608Metric"
 			(at 196.342 91.44 90)
 			(effects

Commit message: started LCSC, fixing DCDC
Parts:
- removed L4, L5: 2.2mh, Inductor_SMD:L_0603_1608Metric, symbol Device:L
- added L62: L_Coupled_Small_1423, symbol Device:L_Coupled_Small_1423
- C10, C11, C12, C13: LCSC (none) -> C784420
- C9: LCSC (none) -> C18255877
Connections:
- net 48V: now also L62.1
- net GND: now also L62.2
- net VIN: now also L62.4
- net at C12.2, C13.2, C15.1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: now also L62.3

Commit message: big reorg
Parts:
- renumbered C9 to C62, C10 to C63, C11 to C64, C12 to C65, C13 to C66, C14 to C67, C15 to C68, C16 to C69, L62 to L16, PS2 to PS6, R39 to R36
