File: kicad_files/bcrl_power_supply/PQC50-48-S5-O_EMC_trimmed.kicad_sch (KiCad schematic)
At the start: 11 parts

Commit message: big changes
Parts:
- renumbered C62 to C75, C63 to C76, C64 to C77, C65 to C78, C66 to C79, C67 to C80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
