File: kicad_files/bcrl_power_supply/PYBE20-Q48-S9_8V_trim.kicad_sch (KiCad schematic)
At the start: 9 parts

Commit message: started LCSC, fixing DCDC
Parts:
- removed C145, C148: 330uf/100v, Capacitor_SMD:C_0603_1608Metric, symbol Device:C
- removed C146, C147: 4.7uf/100v, Capacitor_SMD:C_0603_1608Metric, symbol Device:C
- removed C149, C150: 1nf/2kv, Capacitor_SMD:C_0603_1608Metric, symbol Device:C
- removed C151: 47uf/50v, Capacitor_SMD:C_0603_1608Metric, symbol Device:C
- removed L42: 4.7uh/3.1a, Inductor_SMD:L_0603_1608Metric, symbol Device:L
- removed PS18: PDQE15-Q48-D24-D, BCRL_power_supply:CONV_PDQE15-Q48-D24-D, symbol BCRL_power_supply:PDQE15-Q48-D24-D
- added C181: 330uf/100v, Capacitor_SMD:C_0603_1608Metric, symbol Device:C_Polarized
- added C182, C183: 100uf, Capacitor_SMD:C_0603_1608Metric, symbol Device:C
- added C184, C185: 1nf/2kv, Capacitor_SMD:C_0603_1608Metric, symbol Device:C
- added C186: 470uf, Capacitor_SMD:C_0603_1608Metric, symbol Device:C
- added L51: 4.7uh/3.1a, symbol Device:L
- added PS21: PYBE20-Q48-S9, symbol BCRL_power_supply:PYBE20-Q48-S9
Connections:
- net 48V: now also C181.1, C182.1, L51.1
- net CTRL: now also PS21.6 (CTRL)
- net GND: now also C181.2, C182.2, C183.2, C185.1, C185.2, C186.2, PS21.1 (GND), PS21.5 (0V)
- new net: C183.1, C184.1, L51.2, PS21.2 (VIN)
- new net +9V: C184.2, C186.1, PS21.3 (+VO)
- no-connect marks 0 -> 1

Commit message: big reorg
Parts:
- renumbered C181 to C39, C182 to C40, C183 to C60, C184 to C61, C185 to C70, C186 to C71, L51 to L7, PS21 to PS7
Changed lines of the file:
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@@
 		(dnp no)
 		(fields_autoplaced yes)
-		(property "Reference" "PS21"
+		(property "Reference" "PS7"
 			(at 146.05 82.55 0)
 			(effects
@@
 		(instances
 			(project "bcrl_power_supply"
-				(path "/77f0f57c-9586-4625-9281-fa8cbd8015db/94fee228-5462-46f6-ad6c-1e47c0f1b343/a1e164ce-9ade-499f-8629-2721619051ad"
-					(reference "PS21")
+				(path "/77f0f57c-9586-4625-9281-fa8cbd8015db/94fee228-5462-46f6-ad6c-1e47c0f1b343/1f2fcd3d-ee32-476b-8353-2d2feab2ada6"
+					(reference "PS7")
 					(unit 1)
 				)
@@
 		(dnp no)
 		(fields_autoplaced yes)
-		(property "Reference" "C185"
+		(property "Reference" "C70"
 			(at 146.05 116.84 90)
 			(effects
@@
 		(instances
 			(project "bcrl_power_supply"
-				(path "/77f0f57c-9586-4625-9281-fa8cbd8015db/94fee228-5462-46f6-ad6c-1e47c0f1b343/a1e164ce-9ade-499f-8629-2721619051ad"
-					(reference "C185")
+				(path "/77f0f57c-9586-4625-9281-fa8cbd8015db/94fee228-5462-46f6-ad6c-1e47c0f1b343/1f2fcd3d-ee32-476b-8353-2d2feab2ada6"
+					(reference "C70")
 					(unit 1)
 				)
@@
 		(dnp no)
 		(fields_autoplaced yes)
-		(property "Reference" "C183"
+		(property "Reference" "C60"
 			(at 115.57 99.06 0)
 			(effects
@@
 		(instances
 			(project "bcrl_power_supply"
-				(path "/77f0f57c-9586-4625-9281-fa8cbd8015db/94fee228-5462-46f6-ad6c-1e47c0f1b343/a1e164ce-9ade-499f-8629-2721619051ad"
-					(reference "C183")
+				(path "/77f0f57c-9586-4625-9281-fa8cbd8015db/94fee228-5462-46f6-ad6c-1e47c0f1b343/1f2fcd3d-ee32-476b-8353-2d2feab2ada6"
+					(reference "C60")
 					(unit 1)
 				)
@@
 		(dnp no)
 		(fields_autoplaced yes)
-		(property "Reference" "C186"
+		(property "Reference" "C71"
 			(at 175.26 99.06 0)
 			(effects
@@
 		(instances
 			(project "bcrl_power_supply"
-				(path "/77f0f57c-9586-4625-9281-fa8cbd8015db/94fee228-5462-46f6-ad6c-1e47c0f1b343/a1e164ce-9ade-499f-8629-2721619051ad"
-					(reference "C186")
+				(path "/77f0f57c-9586-4625-9281-fa8cbd8015db/94fee228-5462-46f6-ad6c-1e47c0f1b343/1f2fcd3d-ee32-476b-8353-2d2feab2ada6"
+					(reference "C71")
 					(unit 1)
 				)
@@
 		(dnp no)
 		(fields_autoplaced yes)
-		(property "Reference" "C181"
+		(property "Reference" "C39"
 			(at 88.9 98.171 0)
 			(effects
@@
 		(instances
 			(project "bcrl_power_supply"
-				(path "/77f0f57c-9586-4625-9281-fa8cbd8015db/94fee228-5462-46f6-ad6c-1e47c0f1b343/a1e164ce-9ade-499f-8629-2721619051ad"
-					(reference "C181")
+				(path "/77f0f57c-9586-4625-9281-fa8cbd8015db/94fee228-5462-46f6-ad6c-1e47c0f1b343/1f2fcd3d-ee32-476b-8353-2d2feab2ada6"
+					(reference "C39")
 					(unit 1)
 				)
@@
 		(dnp no)
 		(fields_autoplaced yes)
-		(property "Reference" "#PWR0284"
+		(property "Reference" "#PWR0138"
 			(at 171.45 114.3 0)
 			(effects
@@
 		(instances
 			(project "bcrl_power_supply"
-				(path "/77f0f57c-9586-4625-9281-fa8cbd8015db/94fee228-5462-46f6-ad6c-1e47c0f1b343/a1e164ce-9ade-499f-8629-2721619051ad"
-					(reference "#PWR0284")
+				(path "/77f0f57c-9586-4625-9281-fa8cbd8015db/94fee228-5462-46f6-ad6c-1e47c0f1b343/1f2fcd3d-ee32-476b-8353-2d2feab2ada6"
+					(reference "#PWR0138")
 					(unit 1)
 				)
@@
 		(dnp no)
 		(fields_autoplaced yes)
-		(property "Reference" "C184"
+		(property "Reference" "C61"
 			(at 146.05 67.31 90)
 			(effects
@@
 		(instances
 			(project "bcrl_power_supply"
-				(path "/77f0f57c-9586-4625-9281-fa8cbd8015db/94fee228-5462-46f6-ad6c-1e47c0f1b343/a1e164ce-9ade-499f-8629-2721619051ad"
-					(reference "C184")
+				(path "/77f0f57c-9586-4625-9281-fa8cbd8015db/94fee228-5462-46f6-ad6c-1e47c0f1b343/1f2fcd3d-ee32-476b-8353-2d2feab2ada6"
+					(reference "C61")
 					(unit 1)
 				)
@@
 		(dnp no)
 		(fields_autoplaced yes)
-		(property "Reference" "L51"
+		(property "Reference" "L7"
 			(at 104.14 87.63 90)
 			(effects
@@
 		(instances
 			(project "bcrl_power_supply"
-				(path "/77f0f57c-9586-4625-9281-fa8cbd8015db/94fee228-5462-46f6-ad6c-1e47c0f1b343/a1e164ce-9ade-499f-8629-2721619051ad"
-					(reference "L51")
+				(path "/77f0f57c-9586-4625-9281-fa8cbd8015db/94fee228-5462-46f6-ad6c-1e47c0f1b343/1f2fcd3d-ee32-476b-8353-2d2feab2ada6"
+					(reference "L7")
 					(unit 1)
 				)
@@
 		(dnp no)
 		(fields_autoplaced yes)
-		(property "Reference" "#PWR0283"
+		(property "Reference" "#PWR0137"
 			(at 80.01 114.3 0)
 			(effects
@@
 		(instances
 			(project "bcrl_power_supply"
-				(path "/77f0f57c-9586-4625-9281-fa8cbd8015db/94fee228-5462-46f6-ad6c-1e47c0f1b343/a1e164ce-9ade-499f-8629-2721619051ad"
-					(reference "#PWR0283")
+				(path "/77f0f57c-9586-4625-9281-fa8cbd8015db/94fee228-5462-46f6-ad6c-1e47c0f1b343/1f2fcd3d-ee32-476b-8353-2d2feab2ada6"
+					(reference "#PWR0137")
 					(unit 1)
 				)
@@
 		(dnp no)
 		(fields_autoplaced yes)
-		(property "Reference" "C182"
+		(property "Reference" "C40"
 			(at 99.06 99.06 0)
 			(effects
@@
 		(instances
 			(project "bcrl_power_supply"
-				(path "/77f0f57c-9586-4625-9281-fa8cbd8015db/94fee228-5462-46f6-ad6c-1e47c0f1b343/a1e164ce-9ade-499f-8629-2721619051ad"
-					(reference "C182")
-					(unit 1)
-				)
+				(path "/77f0f57c-9586-4625-9281-fa8cbd8015db/94fee228-5462-46f6-ad6c-1e47c0f1b343/1f2fcd3d-ee32-476b-8353-2d2feab2ada6"
+					(reference "C40")
+					(unit 1)
+				)
