File: kicad_files/bcrl_power_supply/RxRFswMUXv1_board.kicad_sch (KiCad schematic)
At the start: 27 parts, among them J1 OSTVN02A150, J11 5034801600, J2 OSTVN02A150, J3 OSTVN02A150, J4 OSTVN02A150, J5 OSTVN02A150, J6 OSTVN02A150, J7 OSTVN02A150, J8 OSTVN02A150, J9 5034801600, P1 5104338-1, P2 5104338-1, P3 Conn_01x10, P4 Conn_01x10, U1 PDQ10-Q48-S3-D

Commit message: added more circuits
Parts:
- removed CJ1, CJ2, CJ3, CJ4: Conn_01x10, Connector_PinSocket_2.54mm:PinSocket_1x10_P2.54mm_Vertical, symbol Connector_Generic:Conn_01x10
- removed J1, J2, J3, J4, J5, J6, J7, J8: OSTVN02A150, BCRL_power_supply:CONN_OSTVN02A150_OST, symbol 2024-02-14_22-22-09:OSTVN02A150
- removed J11, J9: 5034801600, symbol BCRL_power_supply:5034801600
- removed P1, P2: 5104338-1, symbol BCRL_power_supply:5104338-1
- removed P3, P4: Conn_01x10, Connector_PinSocket_1.27mm:PinSocket_1x10_P1.27mm_Vertical, symbol Connector_Generic:Conn_01x10
- removed PS1, PS2, PS3, PS4: PYBE20-Q48-S9, symbol BCRL_power_supply:PYBE20-Q48-S9
- removed PS5, PS6, PS7, PS8: PYBE20-Q48-S5, PYBE20-Q48-S5:CONV_PYBE20-Q48-S5, symbol BCRL_power_supply:PYBE20-Q48-S5
- removed U1: PDQ10-Q48-S3-D, PDQ10-Q48-S3-D:CONV_PDQ10-Q48-S3-D, symbol BCRL_power_supply:PDQ10-Q48-S3-D
- added J15, J16, J17, J18, J19, J20, J21, J22, J23, J24: OSTVN02A150, BCRL_power_supply:CONN_OSTVN02A150_OST, symbol 2024-02-14_22-22-09:OSTVN02A150
- added J25, J26: 5034801600, BCRL_power_supply:MOLEX_5034801600, symbol BCRL_power_supply:5034801600
- added P5, P6, P7, P8: 5104338-1, BCRL_power_supply:TE_5104338-1, symbol BCRL_power_supply:5104338-1
Connections:
- net GND: now also J15.2, J16.2, J17.2, J18.2, J19.2, J20.2, J21.2, J22.2, J23.2, J24.2, J25.1, J25.16, J25.8, J25.9, J25.S1 (SHIELD), J25.S2 (SHIELD__1), J26.1, J26.16, J26.8, J26.9, J26.S1 (SHIELD), J26.S2 (SHIELD__1), P5.4, P5.6, P6.4, P6.6, P7.4, P7.6, P8.4, P8.6
- new net +3.3V: P5.5, P6.5, P7.5, P8.5
- new net +5V: J15.1, J16.1, J17.1, J18.1
- new net +8V: J19.1, J20.1, J21.1, J22.1
- new net EN_12V_FROM_5V: J23.1
- new net EN_3.3V_FROM_5V: J24.1
- new net P1.1_VCTL2_SW1: J25.2, P5.1
- new net P1.2_VCTL2_SW2: J25.3, P5.2
- new net P1.3_VCTL1: J25.4, P5.3
- new net P2.1_VCTL2_SW1: J25.5, J25.6, P6.1, P6.2
- new net P2.3_VCTL1: J25.7, P6.3
- new net P3.1_VCTL2_SW1: J25.10, J25.11, P7.1, P7.2
- new net P3.3_VCTL1: J25.12, P7.3
- new net P4.1_VCTL2_SW1: J25.13, J25.14, P8.1, P8.2
- new net P4.3_VCTL1: J25.15, P8.3
- new net RxLNA1_OnOFF: J26.2
- new net RxLNA2_OnOFF: J26.3
- new net RxLNA3_OnOFF: J26.4
- new net RxLNA4_OnOFF: J26.5
- new net RxPAx4_8VOnOFF: J26.6
- no-connect marks 0 -> 23
Other:
- added sheet EHHD010A0B41-HZ_EMC1 (EHHD010A0B41-HZ.kicad_sch)
- added sheet PDQ10-Q48-S3-D_EMC_2 (PDQ10-Q48-S3-D_EMC.kicad_sch)
- added sheet PQC50-48-S5-O_EMC_trimmed_5 (PQC50-48-S5-O_EMC_trimmed.kicad_sch)
- added sheet PQC50-48-S5-O_EMC_trimmed_6 (PQC50-48-S5-O_EMC_trimmed.kicad_sch)
- added sheet PQC50-48-S5-O_EMC_trimmed_7 (PQC50-48-S5-O_EMC_trimmed.kicad_sch)
- added sheet PQC50-48-S5-O_EMC_trimmed_8 (PQC50-48-S5-O_EMC_trimmed.kicad_sch)
- added sheet PYBE20-Q48-S5_EMC_5 (PYBE20-Q48-S5_EMC.kicad_sch)
- added sheet PYBE20-Q48-S5_EMC_6 (PYBE20-Q48-S5_EMC.kicad_sch)
- added sheet PYBE20-Q48-S5_EMC_7 (PYBE20-Q48-S5_EMC.kicad_sch)
- added sheet PYBE20-Q48-S5_EMC_8 (PYBE20-Q48-S5_EMC.kicad_sch)

Commit message: WIP
Parts:
- added J51, J52, J53: OSTVN02A150, BCRL_power_supply:CONN_OSTVN02A150_OST, symbol 2024-02-14_22-22-09:OSTVN02A150
- added J54: 5034801600, BCRL_power_supply:MOLEX_5034801600, symbol BCRL_power_supply:5034801600
Connections:
- net RxPAx4_8VOnOFF: no longer J26.6
- new net RxPAx4_8VOnOFF_1: J26.6
- no-connect marks 23 -> 22
Changed lines of the file:
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@@
   (no_connect (at 125.73 80.645))
   (no_connect (at 181.61 121.285))
-  (no_connect (at 125.73 48.895))
   (no_connect (at 125.73 78.105))
   (no_connect (at 125.73 83.185))
@@
     (effects (font (size 1.27 1.27)) (justify left bottom))
   )
+  (label "LNA_SHUTDOWN" (at 110.49 49.53 0) (fields_autoplaced)
+    (effects (font (size 1.27 1.27)) (justify left bottom))
+  )
   (label "P3.3_VCTL1" (at 107.95 94.615 0) (fields_autoplaced)
     (effects (font (size 1.27 1.27)) (justify left bottom))
@@
     (effects (font (size 1.27 1.27)) (justify left bottom))
   )
-  (label "RxPAx4_8VOnOFF" (at 167.64 98.425 0) (fields_autoplaced)
+  (label "RxPAx4_8VOnOFF_1" (at 167.64 98.425 0) (fields_autoplaced)
     (effects (font (size 1.27 1.27)) (justify left bottom))
   )
@@
         (path "/77f0f57c-9586-4625-9281-fa8cbd8015db/86d69f20-72a8-480c-899a-1cc522974f16"
           (reference "#PWR0105") (unit 1)
+        )
+      )
+    )
+  )
+  (symbol (lib_id "2024-02-14_22-22-09:OSTVN02A150") (at 40.64 200.66 0) (unit 1)
+    (in_bom yes) (on_board yes) (dnp no) (fields_autoplaced)
+    (property "Reference" "J51" (at 54.61 200.66 0)
+      (effects (font (size 1.524 1.524)) (justify left))
+    )
+    (property "Value" "OSTVN02A150" (at 54.61 203.2 0)
+      (effects (font (size 1.524 1.524)) (justify left))
+    )
+    (property "Footprint" "BCRL_power_supply:CONN_OSTVN02A150_OST" (at 30.48 195.58 0)
+      (effects (font (size 1.27 1.27) italic) hide)
+    )
+    (property "Datasheet" "" (at 34.29 198.12 0)
+      (effects (font (size 1.27 1.27) italic) hide)
+    )
+    (pin "2")
+    (pin "1")
+    (instances
+      (project "bcrl_power_supply"
+        (path "/77f0f57c-9586-4625-9281-fa8cbd8015db/86d69f20-72a8-480c-899a-1cc522974f16"
+          (reference "J51") (unit 1)
         )
       )
@@
     )
   )
+  (symbol (lib_id "BCRL_power_supply:5034801600") (at 191.77 168.91 0) (unit 1)
+    (in_bom yes) (on_board yes) (dnp no) (fields_autoplaced)
+    (property "Reference" "J54" (at 198.12 170.18 0)
+      (effects (font (size 1.27 1.27)) (justify left))
+    )
+    (property "Value" "5034801600" (at 198.12 172.72 0)
+      (effects (font (size 1.27 1.27)) (justify left))
+    )
+    (property "Footprint" "BCRL_power_supply:MOLEX_5034801600" (at 191.77 168.91 0)
+      (effects (font (size 1.27 1.27)) (justify bottom) hide)
+    )
+    (property "Datasheet" "" (at 191.77 168.91 0)
+      (effects (font (size 1.27 1.27)) hide)
+    )
+    (property "PARTREV" "" (at 207.01 162.56 0)
+      (effects (font (size 1.27 1.27)) (justify bottom) hide)
+    )
+    (property "STANDARD" "" (at 191.77 168.91 0)
+      (effects (font (size 1.27 1.27)) (justify bottom) hide)
+    )
+    (property "MAXIMUM_PACKAGE_HEIGHT" "1.87 mm" (at 194.31 170.18 90)
+      (effects (font (size 1.27 1.27)) (justify bottom) hide)
+    )
+    (property "MANUFACTURER" "Molex" (at 193.04 149.86 0)
+      (effects (font (size 1.27 1.27)) (justify bottom) hide)
+    )
+    (pin "7")
+    (pin "15")
+    (pin "S1")
+    (pin "8")
+    (pin "11")
+    (pin "12")
+    (pin "10")
+    (pin "14")
+    (pin "13")
+    (pin "6")
+    (pin "1")
+    (pin "4")
+    (pin "16")
+    (pin "2")
+    (pin "5")
+    (pin "S2")
+    (pin "3")
+    (pin "9")
+    (instances
+      (project "bcrl_power_supply"
+        (path "/77f0f57c-9586-4625-9281-fa8cbd8015db/86d69f20-72a8-480c-899a-1cc522974f16"
+          (reference "J54") (unit 1)
+        )
+      )
+    )
+  )
   (symbol (lib_id "2024-02-14_22-22-09:OSTVN02A150") (at 30.48 116.205 0) (unit 1)
     (in_bom yes) (on_board yes) (dnp no) (fields_autoplaced)
@@
     )
   )
+  (symbol (lib_id "2024-02-14_22-22-09:OSTVN02A150") (at 40.64 215.9 0) (unit 1)
+    (in_bom yes) (on_board yes) (dnp no) (fields_autoplaced)
+    (property "Reference" "J52" (at 54.61 215.9 0)
+      (effects (font (size 1.524 1.524)) (justify left))
+    )
+    (property "Value" "OSTVN02A150" (at 54.61 218.44 0)
+      (effects (font (size 1.524 1.524)) (justify left))
+    )
+    (property "Footprint" "BCRL_power_supply:CONN_OSTVN02A150_OST" (at 30.48 210.82 0)
+      (effects (font (size 1.27 1.27) italic) hide)
+    )
+    (property "Datasheet" "" (at 34.29 213.36 0)
+      (effects (font (size 1.27 1.27) italic) hide)
+    )
+    (pin "2")
+    (pin "1")
+    (instances
+      (project "bcrl_power_supply"
+        (path "/77f0f57c-9586-4625-9281-fa8cbd8015db/86d69f20-72a8-480c-899a-1cc522974f16"
+          (reference "J52") (unit 1)
+        )
+      )
+    )
+  )
   (symbol (lib_id "power:GND") (at 168.91 69.215 270) (unit 1)
     (in_bom yes) (on_board yes) (dnp no) (fields_autoplaced)
@@
         )
       )
+    )
+  )
+  (symbol (lib_id "2024-02-14_22-22-09:OSTVN02A150") (at 40.64 231.14 0) (unit 1)
+    (in_bom yes) (on_board yes) (dnp no) (fields_autoplaced)
+    (property "Reference" "J53" (at 54.61 231.14 0)
+      (effects (font (size 1.524 1.524)) (justify left))
+    )
+    (property "Value" "OSTVN02A150" (at 54.61 233.68 0)
+      (effects (font (size 1.524 1.524)) (justify left))
+    )
+    (property "Footprint" "BCRL_power_supply:CONN_OSTVN02A150_OST" (at 30.48 226.06 0)
+      (effects (font (size 1.27 1.27) italic) hide)
+    )
+    (property "Datasheet" "" (at 34.29 228.6 0)
+      (effects (font (size 1.27 1.27) italic) hide)
+    )
+    (pin "2")
+    (pin "1")
+    (instances
+      (project "bcrl_power_supply"
+        (path "/77f0f57c-9586-4625-9281-fa8cbd8015db/86d69f20-72a8-480c-899a-1cc522974f16"
+          (reference "J53") (unit 1)
+        )
+      )

Commit message: cleanup PCB
Parts:
- removed J15, J16, J17, J18, J19, J20, J21, J22, J51, J52, J53: OSTVN02A150, BCRL_power_supply:CONN_OSTVN02A150_OST, symbol 2024-02-14_22-22-09:OSTVN02A150
- removed J26, J54: 5034801600, BCRL_power_supply:MOLEX_5034801600, symbol BCRL_power_supply:5034801600
- added D10, D11, D12, D13, D14, D15, D16, D9: LED, LED_SMD:LED_0603_1608Metric, symbol Device:LED
- added J25, J26, J27, J28, J29, J30, J31: OSTVN02A150, BCRL_power_supply:CONN_OSTVN02A150_OST, symbol 2024-02-14_22-22-09:OSTVN02A150
- added J33, J34, J35, J36, J37, J38, J39, J40: Conn_01x02, Connector_PinHeader_2.54mm:PinHeader_1x02_P2.54mm_Vertical, symbol Connector_Generic:Conn_01x02
- added J42: 5034801600, BCRL_power_supply:MOLEX_5034801600, symbol BCRL_power_supply:5034801600
- added R24, R25, R26, R27, R28, R29, R30, R31: 1k, Resistor_SMD:R_0603_1608Metric, symbol Device:R
- renumbered J23 to J32, J25 to J41
Connections:
- net GND: now also J25.2, J26.2, J27.2, J28.2, J29.2, J30.2, J31.2, J33.2 (Pin_2), J34.2 (Pin_2), J35.2 (Pin_2), J36.2 (Pin_2), J37.2 (Pin_2), J38.2 (Pin_2), J39.2 (Pin_2), J40.2 (Pin_2), J42.1, J42.16, J42.8, J42.9, J42.S1 (SHIELD), J42.S2 (SHIELD__1), R24.1, R25.1, R26.1, R27.1, R28.1, R29.1, R30.1, R31.1
- net EN_3.3V_FROM_5V renamed +5V_1
- net +5V_1: now also D9.2 (A)
- new net: D11.1 (K), R26.2
- new net: D16.1 (K), R31.2
- new net: D14.1 (K), R29.2
- new net: D10.1 (K), R25.2
- new net: D12.1 (K), R27.2
- new net: D13.1 (K), R28.2
- new net: D9.1 (K), R24.2
- new net: D15.1 (K), R30.2
- new net +5V_2: D10.2 (A), J25.1
- new net +5V_3: D11.2 (A), J26.1
- new net +5V_4: D12.2 (A), J27.1
- new net +8V_1: D13.2 (A), J28.1
- new net +8V_2: D15.2 (A), J29.1
- new net +8V_3: D14.2 (A), J30.1
- new net +8V_4: D16.2 (A), J31.1
- new net RxLNA1_5V_CTL: J33.1 (Pin_1), J42.2
- new net RxLNA1_8V_CTL: J37.1 (Pin_1), J42.10
- new net RxLNA2_5V_CTL: J34.1 (Pin_1), J42.3
- new net RxLNA2_8V_CTL: J38.1 (Pin_1), J42.11
- new net RxLNA3_5V_CTL: J35.1 (Pin_1), J42.4
- new net RxLNA3_8V_CTL: J39.1 (Pin_1), J42.12
- new net RxLNA4_5V_CTL: J36.1 (Pin_1), J42.5
- new net RxLNA4_8V_CTL: J40.1 (Pin_1), J42.13
- no-connect marks 22 -> 19
Other:
- removed sheet PDQ10-Q48-S3-D_EMC_2
- removed sheet PQC50-48-S5-O_EMC_trimmed_5
- removed sheet PQC50-48-S5-O_EMC_trimmed_6
- removed sheet PQC50-48-S5-O_EMC_trimmed_7
- removed sheet PQC50-48-S5-O_EMC_trimmed_8
- removed sheet PYBE20-Q48-S5_EMC_5
- removed sheet PYBE20-Q48-S5_EMC_6
- removed sheet PYBE20-Q48-S5_EMC_7
- removed sheet PYBE20-Q48-S5_EMC_8
- added sheet PDQ10-Q48-S5-D_EMC_10 (PDQ10-Q48-S5-D_EMC.kicad_sch)
- added sheet PDQ10-Q48-S5-D_EMC_11 (PDQ10-Q48-S5-D_EMC.kicad_sch)
- added sheet PDQ10-Q48-S5-D_EMC_12 (PDQ10-Q48-S5-D_EMC.kicad_sch)
- added sheet PDQ10-Q48-S5-D_EMC_9 (PDQ10-Q48-S5-D_EMC.kicad_sch)
- added sheet PQC50-48-S5-O_EMC_trimmed_11 (PQC50-48-S5-O_EMC_trimmed.kicad_sch)
- added sheet PQC50-48-S5-O_EMC_trimmed_12 (PQC50-48-S5-O_EMC_trimmed.kicad_sch)
- added sheet PQC50-48-S5-O_EMC_trimmed_13 (PQC50-48-S5-O_EMC_trimmed.kicad_sch)
- added sheet PQC50-48-S5-O_EMC_trimmed_14 (PQC50-48-S5-O_EMC_trimmed.kicad_sch)

Commit message: ...
Parts:
- removed J32: OSTVN02A150, BCRL_power_supply:CONN_OSTVN02A150_OST, symbol 2024-02-14_22-22-09:OSTVN02A150
Other:
- removed sheet EHHD010A0B41-HZ_EMC1

Commit message: almost done schematic
Parts:
- added J12: 5034801600, BCRL_power_supply:MOLEX_5034801600, symbol BCRL_power_supply:5034801600
- added J75: Conn_01x04_Pin, Connector_PinHeader_2.54mm:PinHeader_1x04_P2.54mm_Vertical, symbol Connector:Conn_01x04_Pin
Connections:
- net GND: now also J75.1 (Pin_1), J75.4 (Pin_4)
- new net +6.5V_1: J75.2 (Pin_2), J75.3 (Pin_3)

Commit message: schematic done
Parts:
- removed J12: 5034801600, BCRL_power_supply:MOLEX_5034801600, symbol BCRL_power_supply:5034801600
Connections:
- net +5V_1: now also P5.7
- net +5V_2: now also P6.7
- net +5V_3: now also P7.7
- net +5V_4: now also P8.7
- net GND: now also P5.10, P5.9, P6.10, P6.9, P7.10, P7.9, P8.10, P8.9
- net LNA_SHUTDOWN_1: now reaches P7.8
- net LNA_SHUTDOWN_1: now also P5.8, P6.8, P8.8
- no-connect marks 19 -> 4
Other:
- moved on the sheet: D13, D14, D15, J33, J34, J35, J36, J37, J38, J39, J40, J41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

Commit message: big reorg
Parts:
- removed D10, D11, D12, D13, D14, D15, D16, D9: LED, LED_SMD:LED_0603_1608Metric, symbol Device:LED
- removed J26, J27, J28, J29, J30, J31: OSTVN02A150, BCRL_power_supply:CONN_OSTVN02A150_OST, symbol 2024-02-14_22-22-09:OSTVN02A150
- removed J33, J34, J35, J36, J37, J38, J39, J40: Conn_01x02, Connector_PinHeader_2.54mm:PinHeader_1x02_P2.54mm_Vertical, symbol Connector_Generic:Conn_01x02
- removed J41, J42: 5034801600, BCRL_power_supply:MOLEX_5034801600, symbol BCRL_power_supply:5034801600
- removed J75: Conn_01x04_Pin, Connector_PinHeader_2.54mm:PinHeader_1x04_P2.54mm_Vertical, symbol Connector:Conn_01x04_Pin
- removed P5, P6, P7, P8: 5104338-1, BCRL_power_supply:TE_5104338-1, symbol BCRL_power_supply:5104338-1
- removed R24, R25, R26, R27, R28, R29, R31: 1k, Resistor_SMD:R_0603_1608Metric, symbol Device:R
- added D30, D31, D32, D36, D37, D38, D39, D40: LED, LED_SMD:LED_0603_1608Metric, symbol Device:LED
- added J22, J23, J79, J80, J81, J82: OSTVN02A150, BCRL_power_supply:CONN_OSTVN02A150_OST, symbol 2024-02-14_22-22-09:OSTVN02A150
- added J83, J84, J85, J86, J87, J88, J89, J90: Conn_01x02, Connector_PinHeader_2.54mm:PinHeader_1x02_P2.54mm_Vertical, symbol Connector_Generic:Conn_01x02
- added J91: Conn_01x04_Pin, Connector_PinHeader_2.54mm:PinHeader_1x04_P2.54mm_Vertical, symbol Connector:Conn_01x04_Pin
- added J92, J93: 5034801600, BCRL_power_supply:MOLEX_5034801600, symbol BCRL_power_supply:5034801600
- added P10, P11, P12, P9: 5104338-1, BCRL_power_supply:TE_5104338-1, symbol BCRL_power_supply:5104338-1
- added R32, R61, R62, R63, R69, R70, R71: 1k, Resistor_SMD:R_0603_1608Metric, symbol Device:R
Connections:
- net +3.3V: now also P10.5, P11.5, P12.5, P9.5
- net +5V_1: now also D30.2 (A), J22.1, P9.7; no longer J24.1
- net +5V_2: now also D31.2 (A), J23.1, P10.7; no longer J25.1
- net +5V_3: now also J24.1, D32.2 (A), P11.7
- net +5V_4: now also J25.1, D36.2 (A), P12.7
- net +6.5V_1: now also J91.2 (Pin_2), J91.3 (Pin_3)
- net +8V_1: now also D37.2 (A), J79.1
- net +8V_2: now also D39.2 (A), J80.1
- net +8V_3: now also D38.2 (A), J81.1
- net +8V_4: now also D40.2 (A), J82.1
- net GND: now also J22.2, J23.2, J79.2, J80.2, J81.2, J82.2, J83.2 (Pin_2), J84.2 (Pin_2), J85.2 (Pin_2), J86.2 (Pin_2), J87.2 (Pin_2), J88.2 (Pin_2), J89.2 (Pin_2), J90.2 (Pin_2), J91.1 (Pin_1), J91.4 (Pin_4), J92.1, J92.16, J92.8, J92.9, J92.S1 (SHIELD), J92.S2 (SHIELD__1), J93.1, J93.16, J93.8, J93.9, J93.S1 (SHIELD), J93.S2 (SHIELD__1), P10.10, P10.4, P10.6, P10.9, P11.10, P11.4, P11.6, P11.9, P12.10, P12.4, P12.6, P12.9, P9.10, P9.4, P9.6, P9.9, R32.1, R61.1, R62.1, R63.1, R69.1, R70.1, R71.1
- net LNA_SHUTDOWN_1: now also J93.12, P9.8
- net at R30.2: now also D30.1 (K)
- new net: D36.1 (K), R62.2
- new net: D38.1 (K), R69.2
- new net: D37.1 (K), R63.2
- new net: D39.1 (K), R70.2
- new net: D40.1 (K), R71.2
- new net: D32.1 (K), R61.2
- new net: D31.1 (K), R32.2
- new net LNA_SHUTDOWN_2: J93.13, P10.8
- new net LNA_SHUTDOWN_3: J93.14, P11.8
- new net LNA_SHUTDOWN_4: J93.15, P12.8
- new net P1.1_VCTRL2_SW1: J92.2, P9.1
- new net P1.2_VCTRL2_SW2: J92.3, P9.2
- new net P1.3_VCTRL1: J92.4, P9.3
- new net P2.1_VCTRL2_SW1: J92.5, J92.6, P10.1, P10.2
- new net P2.3_VCTRL1: J92.7, P10.3
- new net P3.1_VCTRL2_SW1: J92.10, J92.11, P11.1, P11.2
- new net P3.3_VCTRL1: J92.12, P11.3
- new net P4.1_VCTRL2_SW1: J92.13, J92.14, P12.1, P12.2
- new net P4.3_VCTRL1: J92.15, P12.3
- new net RxLNA1_5V_CTRL: J83.1 (Pin_1), J93.2
- new net RxLNA1_8V_CTRL: J87.1 (Pin_1), J93.6
- new net RxLNA2_5V_CTRL: J84.1 (Pin_1), J93.3
- new net RxLNA2_8V_CTRL: J88.1 (Pin_1), J93.7
- new net RxLNA3_5V_CTRL: J85.1 (Pin_1), J93.4
- new net RxLNA3_8V_CTRL: J89.1 (Pin_1), J93.10
- new net RxLNA4_5V_CTRL: J86.1 (Pin_1), J93.5
- new net RxLNA4_8V_CTRL: J90.1 (Pin_1), J93.11
- no-connect marks 4 -> 0
Other:
- removed sheet PDQ10-Q48-S5-D_EMC_10
- removed sheet PDQ10-Q48-S5-D_EMC_11
- removed sheet PDQ10-Q48-S5-D_EMC_12
- removed sheet PDQ10-Q48-S5-D_EMC_9
- removed sheet PQC50-48-S5-O_EMC_trimmed_11
- removed sheet PQC50-48-S5-O_EMC_trimmed_12
- removed sheet PQC50-48-S5-O_EMC_trimmed_13
- removed sheet PQC50-48-S5-O_EMC_trimmed_14
- added sheet EHHD010A0B41-HZ_1 (EHHD010A0B41-HZ.kicad_sch)
- added sheet PDQ10-Q48-S5-D_EMC_14 (PDQ10-Q48-S5-D_EMC.kicad_sch)
- added sheet PDQ10-Q48-S5-D_EMC_15 (PDQ10-Q48-S5-D_EMC.kicad_sch)
- added sheet PDQ10-Q48-S5-D_EMC_16 (PDQ10-Q48-S5-D_EMC.kicad_sch)
- added sheet PDQ10-Q48-S5-D_EMC_17 (PDQ10-Q48-S5-D_EMC.kicad_sch)
- added sheet PQC50-48-S5-O_EMC_trimmed_16 (PQC50-48-S5-O_EMC_trimmed.kicad_sch)
- added sheet PQC50-48-S5-O_EMC_trimmed_17 (PQC50-48-S5-O_EMC_trimmed.kicad_sch)
- added sheet PQC50-48-S5-O_EMC_trimmed_18 (PQC50-48-S5-O_EMC_trimmed.kicad_sch)
- added sheet PQC50-48-S5-O_EMC_trimmed_19 (PQC50-48-S5-O_EMC_trimmed.kicad_sch)
