File: kicad_files/bcrl_power_supply/RxRFswMUXv1_board.kicad_sch (KiCad schematic)
At the start: 39 parts, among them J22 OSTVN02A150, J23 OSTVN02A150, J24 OSTVN02A150, J25 OSTVN02A150, J79 OSTVN02A150, J80 OSTVN02A150, J81 OSTVN02A150, J82 OSTVN02A150, J83 Conn_01x02, J84 Conn_01x02, J85 Conn_01x02, J86 Conn_01x02, J87 Conn_01x02, J88 Conn_01x02, J89 Conn_01x02, J90 Conn_01x02, J91 Conn_01x04_Pin, J92 5034801600, J93 5034801600, P10 5104338-1, P11 5104338-1, P12 5104338-1, P9 5104338-1

Commit message: big changes
Parts:
- removed D37, D38, D39, D40: LED, LED_SMD:LED_0603_1608Metric, symbol Device:LED
- removed J91: Conn_01x04_Pin, Connector_PinHeader_2.54mm:PinHeader_1x04_P2.54mm_Vertical, symbol Connector:Conn_01x04_Pin
- removed R63, R69, R70, R71: 1k, Resistor_SMD:R_0603_1608Metric, symbol Device:R
- added D19, D30, D33, D34, D35: LED, LED_SMD:LED_0603_1608Metric, symbol Device:LED
- added J71: Conn_01x02, Connector_PinHeader_2.54mm:PinHeader_1x02_P2.54mm_Vertical, symbol Connector_Generic:Conn_01x02
- added R26, R55, R56, R57, R58: 1k, Resistor_SMD:R_0603_1608Metric, symbol Device:R
- renumbered D30 to D14, D31 to D15, D32 to D16, D36 to D17, J79 to J26, J80 to J27, J81 to J28, J82 to J29, J83 to J30, J84 to J31, J85 to J32, J86 to J33, J87 to J34, J88 to J35, J89 to J36, J90 to J37, J92 to J39, J93 to J40, P9 to P5, P10 to P6, P11 to P7, P12 to P8, R30 to R21, R32 to R22, R61 to R23, R62 to R24
Connections:
- net +8V_1: now also D30.2 (A)
- net +8V_2: now also D34.2 (A)
- net +8V_3: now also D33.2 (A)
- net +8V_4: now also D35.2 (A)
- net GND: now also J71.2 (Pin_2), R26.1, R55.1, R56.1, R57.1, R58.1
- new net: D30.1 (K), R55.2
- new net: D35.1 (K), R58.2
- new net: D34.1 (K), R57.2
- new net: D33.1 (K), R56.2
- new net: D19.1 (K), R26.2
- new net +12V: D19.2 (A)
- new net +12V_CTRL: J71.1 (Pin_1)
Other:
- removed sheet EHHD010A0B41-HZ_1
- removed sheet PQC50-48-S5-O_EMC_trimmed_16
- removed sheet PQC50-48-S5-O_EMC_trimmed_17
- removed sheet PQC50-48-S5-O_EMC_trimmed_18
- removed sheet PQC50-48-S5-O_EMC_trimmed_19
- added sheet EHHD010A0B41-HZ5 (EHHD010A0B41-HZ.kicad_sch)
- added sheet IND108W_EMC_8V_10 (IND108W_EMC_8V.kicad_sch)
- added sheet IND108W_EMC_8V_11 (IND108W_EMC_8V.kicad_sch)
- added sheet IND108W_EMC_8V_12 (IND108W_EMC_8V.kicad_sch)
- added sheet IND108W_EMC_8V_9 (IND108W_EMC_8V.kicad_sch)
