File: kicad_files/bcrl_power_supply/RxRFswMUXv1_board.kicad_sch (KiCad schematic)
At the start: 41 parts, among them J22 OSTVN02A150, J23 OSTVN02A150, J24 OSTVN02A150, J25 OSTVN02A150, J26 OSTVN02A150, J27 OSTVN02A150, J28 OSTVN02A150, J29 OSTVN02A150, J30 Conn_01x02, J31 Conn_01x02, J32 Conn_01x02, J33 Conn_01x02, J34 Conn_01x02, J35 Conn_01x02, J36 Conn_01x02, J37 Conn_01x02, J39 5034801600, J40 5034801600, J71 Conn_01x02, P5 5104338-1, P6 5104338-1, P7 5104338-1, P8 5104338-1

Commit message: almost done schematic
Parts:
- renumbered D19 to D16, D14 to D17, D15 to D18, D16 to D19, D17 to D20, D30 to D21, D33 to D22, D34 to D23, D35 to D24, J22 to J23, J23 to J24, J24 to J25, J25 to J26, J26 to J27, J27 to J28, J28 to J29, J29 to J30, J30 to J31, J31 to J32, J32 to J33, J33 to J34, J34 to J35, J35 to J36, J36 to J37, J37 to J38, J71 to J39, J39 to J40, J40 to J41, R26 to R23, R21 to R24, R22 to R25, R23 to R26, R24 to R27, R55 to R28, R56 to R29, R57 to R30, R58 to R31

Commit message: board review
Parts:
- D16, D17, D18, D19, D20, D21, D22, D23, D24: value LED -> LED 0603
Changed lines of the file:
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@@
 			)
 		)
-		(property "Value" "LED"
+		(property "Value" "LED 0603"
 			(at 259.3975 101.6 0)
 			(effects
@@
 			)
 		)
-		(property "Value" "LED"
+		(property "Value" "LED 0603"
 			(at 260.6675 165.1 0)
 			(effects
@@
 			)
 		)
-		(property "Value" "LED"
+		(property "Value" "LED 0603"
 			(at 254.3175 22.86 0)
 			(effects
@@
 			)
 		)
-		(property "Value" "LED"
+		(property "Value" "LED 0603"
 			(at 260.6675 123.19 0)
 			(effects
@@
 			)
 		)
-		(property "Value" "LED"
+		(property "Value" "LED 0603"
 			(at 259.3975 144.78 0)
 			(effects
@@
 			)
 		)
-		(property "Value" "LED"
+		(property "Value" "LED 0603"
 			(at 255.5875 63.5 0)
 			(effects
@@
 			)
 		)
-		(property "Value" "LED"
+		(property "Value" "LED 0603"
 			(at 255.5875 82.55 0)
 			(effects
@@
 			)
 		)
-		(property "Value" "LED"
+		(property "Value" "LED 0603"
 			(at 175.5775 153.67 0)
 			(effects
@@
 			)
 		)
-		(property "Value" "LED"
+		(property "Value" "LED 0603"
 			(at 255.5875 44.45 0)
 			(effects

Commit message: digikey BOM
Parts:
- D16, D17, D18, D19, D20, D21, D22, D23, D24: DigiKey_Part_Number (none) -> 150060GS75000
- J23, J24, J25, J26, J27, J28, J29, J30: DigiKey_Part_Number (none) -> OSTVN02A150
- J40, J41: DigiKey_Part_Number (none) -> 5034801600
- P5, P6, P7, P8: DigiKey_Part_Number (none) -> 5104338-1
- R23, R24, R25, R26, R27, R28, R29, R30, R31: DigiKey_Part_Number (none) -> ESR03EZPF1001
