File: kicad_files/bcrl_power_supply/BFN_board.kicad_sch (KiCad schematic)
At the start: 3 parts, among them J28 Conn_01x04_Pin, J29 Conn_01x04_Pin, J39 Conn_01x04_Pin

Commit message: WIP
Parts:
- added J39: Conn_01x04_Pin, symbol Connector:Conn_01x04_Pin
- renumbered J39 to J27
Connections:
- net +6.5V: no longer J27.2 (Pin_2), J28.2 (Pin_2), J29.2 (Pin_2)
- net GND: now also J39.1 (Pin_1), J39.4 (Pin_4)
- removed net VCC_shared: J27.3 (Pin_3), J28.3 (Pin_3), J29.3 (Pin_3)
- new net +6.5V_1: J27.2 (Pin_2)
Other:
- added sheet PQC50-48-S5-O_EMC_trimmed_10 (PQC50-48-S5-O_EMC_trimmed.kicad_sch)

Commit message: cleanup PCB
Parts:
- removed J28, J29, J39: Conn_01x04_Pin, symbol Connector:Conn_01x04_Pin
- added J44, J45, J46: Conn_01x04_Pin, Connector_PinHeader_2.54mm:PinHeader_1x04_P2.54mm_Vertical, symbol Connector:Conn_01x04_Pin
- J43: renamed from J27; footprint (none) -> Connector_PinHeader_2.54mm:PinHeader_1x04_P2.54mm_Vertical
Connections:
- net +6.5V_1: now also J43.3 (Pin_3), J44.2 (Pin_2), J44.3 (Pin_3)
- net GND: now also J44.1 (Pin_1), J44.4 (Pin_4), J46.1 (Pin_1), J46.4 (Pin_4)
- new net +6.5V_2: J45.2 (Pin_2), J45.3 (Pin_3), J46.2 (Pin_2), J46.3 (Pin_3)

Commit message: schematic done
Parts:
- added D17, D21: LED, LED_SMD:LED_0603_1608Metric, symbol Device:LED
- added R44, R48: 1k, Resistor_SMD:R_0603_1608Metric, symbol Device:R
Connections:
- net +6.5V_1: now also D17.2 (A)
- net +6.5V_2: now also D21.2 (A)
- net GND: now also R44.1, R48.1
- new net: D17.1 (K), R44.2
- new net: D21.1 (K), R48.2
Other:
- moved on the sheet: J45, J46

Commit message: big reorg
Parts:
- removed J43, J44, J45, J46: Conn_01x04_Pin, Connector_PinHeader_2.54mm:PinHeader_1x04_P2.54mm_Vertical, symbol Connector:Conn_01x04_Pin
- renumbered D17 to D20, R44 to R34, R48 to R35

Commit message: big changes
Parts:
- removed D20, D21: LED, LED_SMD:LED_0603_1608Metric, symbol Device:LED
- removed R34, R35: 1k, Resistor_SMD:R_0603_1608Metric, symbol Device:R
Other:
- removed sheet PQC50-48-S5-O_EMC_trimmed_10
- removed sheet PQC50-48-S5-O_EMC_trimmed_9
- added sheet EHHD010A0B41-HZ (EHHD010A0B41-HZ.kicad_sch)
- added sheet IND108W_EMC_1 (IND108W_EMC.kicad_sch)
