File: kicad_files/bcrl_power_supply/EHHD010A0B41-HZ.kicad_sch (KiCad schematic)
At the start: 1 part

Commit message: cleanup PCB
Parts:
- renumbered PS4 to PS1
Changed lines of the file:
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@@
         )
         (path "/77f0f57c-9586-4625-9281-fa8cbd8015db/86d69f20-72a8-480c-899a-1cc522974f16/8cfea22d-80b8-49d7-b970-46c0a7f512d1"
-          (reference "#PWR0145") (unit 1)
+          (reference "#PWR0132") (unit 1)
         )
       )
@@
         )
         (path "/77f0f57c-9586-4625-9281-fa8cbd8015db/86d69f20-72a8-480c-899a-1cc522974f16/8cfea22d-80b8-49d7-b970-46c0a7f512d1"
-          (reference "#PWR0144") (unit 1)
+          (reference "#PWR0131") (unit 1)
         )
       )
@@
   (symbol (lib_id "BCRL_power_supply:EHHD010A0B41-HZ") (at 132.08 101.6 0) (unit 1)
     (in_bom yes) (on_board yes) (dnp no) (fields_autoplaced)
-    (property "Reference" "PS4" (at 132.08 83.82 0)
+    (property "Reference" "PS1" (at 132.08 83.82 0)
       (effects (font (size 1.27 1.27)))
     )
@@
       (project "bcrl_power_supply"
         (path "/77f0f57c-9586-4625-9281-fa8cbd8015db/94fee228-5462-46f6-ad6c-1e47c0f1b343/b51a450f-a417-4376-bdb4-fbea692f0aa4"
-          (reference "PS4") (unit 1)
+          (reference "PS1") (unit 1)
         )
         (path "/77f0f57c-9586-4625-9281-fa8cbd8015db/86d69f20-72a8-480c-899a-1cc522974f16/8cfea22d-80b8-49d7-b970-46c0a7f512d1"
-          (reference "PS14") (unit 1)
+          (reference "PS6") (unit 1)
         )
       )

Commit message: big reorg
Parts:
- added C39, C60: 100uf, symbol Device:C
- added C40, C61: 1uf, symbol Device:C
- renumbered PS1 to PS6
Connections:
- net +12V: now also C39.1, C40.1
- net 48V: now also C60.1, C61.1
- net GND: now also C39.2, C40.2, C60.2, C61.2

Commit message: big changes
Parts:
- removed C39, C60: 100uf, symbol Device:C
- removed C40, C61: 1uf, symbol Device:C
- removed PS6: EHHD010A0B41-HZ, BCRL_power_supply:CONV_EHHD010A0B41-HZ, symbol BCRL_power_supply:EHHD010A0B41-HZ
- added C67, C69: 100uf, Capacitor_SMD:C_0603_1608Metric, symbol Device:C
- added C68, C70: 1uf, Capacitor_SMD:C_0603_1608Metric, symbol Device:C
- added PS11: EHHD010A0B41-HZ, BCRL_power_supply:CONV_EHHD010A0B41-HZ, symbol BCRL_power_supply:EHHD010A0B41-HZ
Connections:
- net +12V: now also C69.1, C70.1, PS11.8 (VO+)
- net 48V: now also C67.1, C68.1, PS11.1 (VI+)
- net GND: now also C67.2, C68.2, C69.2, C70.2, PS11.3 (VI-), PS11.4 (VO-)
- net ON/OFF: now also PS11.2 (ON/OFF)
