File: kicad_files/bcrl_power_supply/EHHD010A0B41-HZ.kicad_sch (KiCad schematic)
At the start: 5 parts

Commit message: almost done schematic
Parts:
- C31: renamed from C67; value 100uf -> 100u
- C32: renamed from C68; value 1uf -> 1u
- C33: renamed from C69; value 100uf -> 100u
- C34: renamed from C70; value 1uf -> 1u
- renumbered PS11 to PS5
Connections:
- net 48V renamed +48V

Commit message: board review
Other:
- note added: "Positive logic is to leave ON/OFF open https://www.mouser.ca/datasheet/2/167/ehhd010_ds-3395666.pdf"
Changed lines of the file:
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@@
+		)
+	)
+	(text "Positive logic is to leave ON/OFF open\nhttps://www.mouser.ca/datasheet/2/167/ehhd010_ds-3395666.pdf\n"
+		(exclude_from_sim no)
+		(at 115.57 73.66 0)
+		(effects
+			(font
+				(size 1.27 1.27)
+			)
 		)
 	)
@@
 					(unit 1)
 				)
-				(path "/77f0f57c-9586-4625-9281-fa8cbd8015db/8821cb9d-826b-46ea-a4b0-096cc3dd800f/cf656899-5e10-4d7d-a034-78bbc07a41e7"
-					(reference "#PWR0181")
-					(unit 1)
-				)
 				(path "/77f0f57c-9586-4625-9281-fa8cbd8015db/94fee228-5462-46f6-ad6c-1e47c0f1b343/f872ad55-a9da-44cf-ae79-afc2db1e1edb"
 					(reference "#PWR0212")
@@
 				(path "/77f0f57c-9586-4625-9281-fa8cbd8015db/86d69f20-72a8-480c-899a-1cc522974f16/044ed215-894f-4fc1-8dec-169dde83377a"
 					(reference "#PWR0187")
+					(unit 1)
+				)
+				(path "/77f0f57c-9586-4625-9281-fa8cbd8015db/8821cb9d-826b-46ea-a4b0-096cc3dd800f/4ae7f17d-3ea4-4f06-8b49-de2d8b431673"
+					(reference "#PWR0163")
 					(unit 1)
 				)
@@
 					(unit 1)
 				)
-				(path "/77f0f57c-9586-4625-9281-fa8cbd8015db/8821cb9d-826b-46ea-a4b0-096cc3dd800f/cf656899-5e10-4d7d-a034-78bbc07a41e7"
-					(reference "C70")
-					(unit 1)
-				)
 				(path "/77f0f57c-9586-4625-9281-fa8cbd8015db/94fee228-5462-46f6-ad6c-1e47c0f1b343/f872ad55-a9da-44cf-ae79-afc2db1e1edb"
 					(reference "C102")
@@
 				(path "/77f0f57c-9586-4625-9281-fa8cbd8015db/86d69f20-72a8-480c-899a-1cc522974f16/044ed215-894f-4fc1-8dec-169dde83377a"
 					(reference "C78")
+					(unit 1)
+				)
+				(path "/77f0f57c-9586-4625-9281-fa8cbd8015db/8821cb9d-826b-46ea-a4b0-096cc3dd800f/4ae7f17d-3ea4-4f06-8b49-de2d8b431673"
+					(reference "C43")
 					(unit 1)
 				)
@@
 					(unit 1)
 				)
-				(path "/77f0f57c-9586-4625-9281-fa8cbd8015db/8821cb9d-826b-46ea-a4b0-096cc3dd800f/cf656899-5e10-4d7d-a034-78bbc07a41e7"
-					(reference "#PWR0182")
-					(unit 1)
-				)
 				(path "/77f0f57c-9586-4625-9281-fa8cbd8015db/94fee228-5462-46f6-ad6c-1e47c0f1b343/f872ad55-a9da-44cf-ae79-afc2db1e1edb"
 					(reference "#PWR0213")
@@
 				(path "/77f0f57c-9586-4625-9281-fa8cbd8015db/86d69f20-72a8-480c-899a-1cc522974f16/044ed215-894f-4fc1-8dec-169dde83377a"
 					(reference "#PWR0188")
+					(unit 1)
+				)
+				(path "/77f0f57c-9586-4625-9281-fa8cbd8015db/8821cb9d-826b-46ea-a4b0-096cc3dd800f/4ae7f17d-3ea4-4f06-8b49-de2d8b431673"
+					(reference "#PWR0165")
 					(unit 1)
 				)
@@
 					(unit 1)
 				)
-				(path "/77f0f57c-9586-4625-9281-fa8cbd8015db/8821cb9d-826b-46ea-a4b0-096cc3dd800f/cf656899-5e10-4d7d-a034-78bbc07a41e7"
-					(reference "C71")
-					(unit 1)
-				)
 				(path "/77f0f57c-9586-4625-9281-fa8cbd8015db/94fee228-5462-46f6-ad6c-1e47c0f1b343/f872ad55-a9da-44cf-ae79-afc2db1e1edb"
 					(reference "C103")
@@
 				(path "/77f0f57c-9586-4625-9281-fa8cbd8015db/86d69f20-72a8-480c-899a-1cc522974f16/044ed215-894f-4fc1-8dec-169dde83377a"
 					(reference "C79")
+					(unit 1)
+				)
+				(path "/77f0f57c-9586-4625-9281-fa8cbd8015db/8821cb9d-826b-46ea-a4b0-096cc3dd800f/4ae7f17d-3ea4-4f06-8b49-de2d8b431673"
+					(reference "C44")
 					(unit 1)
 				)
@@
 					(unit 1)
 				)
-				(path "/77f0f57c-9586-4625-9281-fa8cbd8015db/8821cb9d-826b-46ea-a4b0-096cc3dd800f/cf656899-5e10-4d7d-a034-78bbc07a41e7"
-					(reference "#PWR0321")
-					(unit 1)
-				)
 				(path "/77f0f57c-9586-4625-9281-fa8cbd8015db/86d69f20-72a8-480c-899a-1cc522974f16/044ed215-894f-4fc1-8dec-169dde83377a"
 					(reference "#PWR0322")
@@
 				(path "/77f0f57c-9586-4625-9281-fa8cbd8015db/94fee228-5462-46f6-ad6c-1e47c0f1b343/f872ad55-a9da-44cf-ae79-afc2db1e1edb"
 					(reference "#PWR0323")
+					(unit 1)
+				)
+				(path "/77f0f57c-9586-4625-9281-fa8cbd8015db/8821cb9d-826b-46ea-a4b0-096cc3dd800f/4ae7f17d-3ea4-4f06-8b49-de2d8b431673"
+					(reference "#PWR0164")
 					(unit 1)
 				)
@@
 					(unit 1)
 				)
-				(path "/77f0f57c-9586-4625-9281-fa8cbd8015db/8821cb9d-826b-46ea-a4b0-096cc3dd800f/cf656899-5e10-4d7d-a034-78bbc07a41e7"
-					(reference "PS9")
-					(unit 1)
-				)
 				(path "/77f0f57c-9586-4625-9281-fa8cbd8015db/94fee228-5462-46f6-ad6c-1e47c0f1b343/f872ad55-a9da-44cf-ae79-afc2db1e1edb"
 					(reference "PS14")
@@
 				(path "/77f0f57c-9586-4625-9281-fa8cbd8015db/86d69f20-72a8-480c-899a-1cc522974f16/044ed215-894f-4fc1-8dec-169dde83377a"
 					(reference "PS10")
+					(unit 1)
+				)
+				(path "/77f0f57c-9586-4625-9281-fa8cbd8015db/8821cb9d-826b-46ea-a4b0-096cc3dd800f/4ae7f17d-3ea4-4f06-8b49-de2d8b431673"
+					(reference "PS6")
 					(unit 1)
 				)
@@
 					(unit 1)
 				)
-				(path "/77f0f57c-9586-4625-9281-fa8cbd8015db/8821cb9d-826b-46ea-a4b0-096cc3dd800f/cf656899-5e10-4d7d-a034-78bbc07a41e7"
-					(reference "C69")
-					(unit 1)
-				)
 				(path "/77f0f57c-9586-4625-9281-fa8cbd8015db/94fee228-5462-46f6-ad6c-1e47c0f1b343/f872ad55-a9da-44cf-ae79-afc2db1e1edb"
 					(reference "C101")
@@
 				(path "/77f0f57c-9586-4625-9281-fa8cbd8015db/86d69f20-72a8-480c-899a-1cc522974f16/044ed215-894f-4fc1-8dec-169dde83377a"
 					(reference "C77")
+					(unit 1)
+				)
+				(path "/77f0f57c-9586-4625-9281-fa8cbd8015db/8821cb9d-826b-46ea-a4b0-096cc3dd800f/4ae7f17d-3ea4-4f06-8b49-de2d8b431673"
+					(reference "C42")
 					(unit 1)
 				)
@@
 					(unit 1)
 				)
-				(path "/77f0f57c-9586-4625-9281-fa8cbd8015db/8821cb9d-826b-46ea-a4b0-096cc3dd800f/cf656899-5e10-4d7d-a034-78bbc07a41e7"
-					(reference "C72")
-					(unit 1)
-				)
 				(path "/77f0f57c-9586-4625-9281-fa8cbd8015db/94fee228-5462-46f6-ad6c-1e47c0f1b343/f872ad55-a9da-44cf-ae79-afc2db1e1edb"
 					(reference "C104")
@@
 					(unit 1)
 				)
+				(path "/77f0f57c-9586-4625-9281-fa8cbd8015db/8821cb9d-826b-46ea-a4b0-096cc3dd800f/4ae7f17d-3ea4-4f06-8b49-de2d8b431673"
+					(reference "C45")
+					(unit 1)
+				)

Commit message: digikey BOM
Parts:
- C31, C33: value 100u -> 47u; footprint Capacitor_SMD:C_0603_1608Metric -> Capacitor_THT:CP_Radial_D12.5mm_P5.00mm; DigiKey_Part_Number (none) -> UCS2E470MHD1TO; rating (none) -> 100v
- C32, C34: DigiKey_Part_Number (none) -> C1608X5R1H105K080DB; rating (none) -> 50v
- PS5: DigiKey_Part_Number (none) -> EHHD010A0B41-HZ
Changed lines of the file:
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@@
 			)
 		)
-		(property "rating" ""
+		(property "rating" "50v"
+			(at 100.33 96.52 0)
+			(effects
+				(font
+					(size 1.27 1.27)
+				)
+				(hide yes)
+			)
+		)
+		(property "DigiKey_Part_Number" "C1608X5R1H105K080DB "
 			(at 100.33 96.52 0)
 			(effects
@@
 			)
 		)
-		(property "Value" "100u"
+		(property "Value" "47u"
 			(at 158.75 97.7899 0)
 			(effects
@@
 			)
 		)
-		(property "Footprint" "Capacitor_SMD:C_0603_1608Metric"
+		(property "Footprint" "Capacitor_THT:CP_Radial_D12.5mm_P5.00mm"
 			(at 155.9052 100.33 0)
 			(effects
@@
 			)
 		)
-		(property "rating" ""
+		(property "rating" "100v"
+			(at 154.94 96.52 0)
+			(effects
+				(font
+					(size 1.27 1.27)
+				)
+				(hide yes)
+			)
+		)
+		(property "DigiKey_Part_Number" "UCS2E470MHD1TO "
 			(at 154.94 96.52 0)
 			(effects
@@
 			)
 		)
-		(property "DigiKey_Part_Number" ""
+		(property "DigiKey_Part_Number" "EHHD010A0B41-HZ"
 			(at 132.08 101.6 0)
 			(effects
@@
 			)
 		)
-		(property "Value" "100u"
+		(property "Value" "47u"
 			(at 92.71 97.7899 0)
 			(effects
@@
 			)
 		)
-		(property "Footprint" "Capacitor_SMD:C_0603_1608Metric"
+		(property "Footprint" "Capacitor_THT:CP_Radial_D12.5mm_P5.00mm"
 			(at 89.8652 100.33 0)
 			(effects
@@
 			)
 		)
-		(property "rating" ""
+		(property "rating" "100v"
+			(at 88.9 96.52 0)
+			(effects
+				(font
+					(size 1.27 1.27)
+				)
+				(hide yes)
+			)
+		)
+		(property "DigiKey_Part_Number" "UCS2E470MHD1TO "
 			(at 88.9 96.52 0)
 			(effects
@@
 			)
 		)
-		(property "rating" ""
+		(property "rating" "50v"
 			(at 166.37 96.52 0)
 			(effects
+				(font
+					(size 1.27 1.27)
+				)
+				(hide yes)
+			)
+		)
+		(property "DigiKey_Part_Number" "C1608X5R1H105K080DB "
+			(at 166.37 96.52 0)
+			(effects
