File: kicad_files/bcrl_power_supply/Eth_Switch.kicad_sch (KiCad schematic)
At the start: 4 parts, among them J43 OSTVN02A150, J44 Conn_01x02

Commit message: almost done schematic
Parts:
- renumbered D31 to D35, J43 to J44, J44 to J45, R61 to R59
Changed lines of the file:
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@@
 		(dnp no)
 		(fields_autoplaced yes)
-		(property "Reference" "J43"
+		(property "Reference" "J44"
 			(at 82.55 116.84 0)
 			(effects
@@
 			)
 		)
+		(property "rating" ""
+			(at 68.58 116.84 0)
+			(effects
+				(font
+					(size 1.27 1.27)
+				)
+				(hide yes)
+			)
+		)
 		(pin "2"
 		)
@@
 			(project "bcrl_power_supply"
 				(path "/77f0f57c-9586-4625-9281-fa8cbd8015db/66481d9d-6957-47e9-a2b4-eda0119b346e"
-					(reference "J43")
-					(unit 1)
-				)
-				(path "/77f0f57c-9586-4625-9281-fa8cbd8015db/396cd466-5b94-4a70-b29a-66669aea6a97"
-					(reference "J41")
+					(reference "J44")
+					(unit 1)
+				)
+				(path "/77f0f57c-9586-4625-9281-fa8cbd8015db/396cd466-5b94-4a70-b29a-66669aea6a97"
+					(reference "J42")
 					(unit 1)
 				)
@@
 		(dnp no)
 		(fields_autoplaced yes)
-		(property "Reference" "D31"
+		(property "Reference" "D35"
 			(at 90.4875 92.71 0)
 			(effects
@@
 			)
 		)
+		(property "rating" ""
+			(at 88.9 99.06 0)
+			(effects
+				(font
+					(size 1.27 1.27)
+				)
+				(hide yes)
+			)
+		)
 		(pin "2"
 		)
@@
 			(project "bcrl_power_supply"
 				(path "/77f0f57c-9586-4625-9281-fa8cbd8015db/396cd466-5b94-4a70-b29a-66669aea6a97"
-					(reference "D31")
-					(unit 1)
-				)
-				(path "/77f0f57c-9586-4625-9281-fa8cbd8015db/66481d9d-6957-47e9-a2b4-eda0119b346e"
-					(reference "D32")
+					(reference "D35")
+					(unit 1)
+				)
+				(path "/77f0f57c-9586-4625-9281-fa8cbd8015db/66481d9d-6957-47e9-a2b4-eda0119b346e"
+					(reference "D36")
 					(unit 1)
 				)
@@
 		(dnp no)
 		(fields_autoplaced yes)
-		(property "Reference" "#PWR0213"
+		(property "Reference" "#PWR0245"
 			(at 62.23 119.38 0)
 			(effects
@@
 			(project "bcrl_power_supply"
 				(path "/77f0f57c-9586-4625-9281-fa8cbd8015db/66481d9d-6957-47e9-a2b4-eda0119b346e"
-					(reference "#PWR0213")
-					(unit 1)
-				)
-				(path "/77f0f57c-9586-4625-9281-fa8cbd8015db/396cd466-5b94-4a70-b29a-66669aea6a97"
-					(reference "#PWR0210")
+					(reference "#PWR0245")
+					(unit 1)
+				)
+				(path "/77f0f57c-9586-4625-9281-fa8cbd8015db/396cd466-5b94-4a70-b29a-66669aea6a97"
+					(reference "#PWR0242")
 					(unit 1)
 				)
@@
 		(dnp no)
 		(fields_autoplaced yes)
-		(property "Reference" "J44"
+		(property "Reference" "J45"
 			(at 78.74 130.175 0)
 			(effects
@@
 			)
 		)
+		(property "rating" ""
+			(at 76.2 130.175 0)
+			(effects
+				(font
+					(size 1.27 1.27)
+				)
+				(hide yes)
+			)
+		)
 		(pin "1"
 		)
@@
 			(project "bcrl_power_supply"
 				(path "/77f0f57c-9586-4625-9281-fa8cbd8015db/66481d9d-6957-47e9-a2b4-eda0119b346e"
-					(reference "J44")
-					(unit 1)
-				)
-				(path "/77f0f57c-9586-4625-9281-fa8cbd8015db/396cd466-5b94-4a70-b29a-66669aea6a97"
-					(reference "J42")
+					(reference "J45")
+					(unit 1)
+				)
+				(path "/77f0f57c-9586-4625-9281-fa8cbd8015db/396cd466-5b94-4a70-b29a-66669aea6a97"
+					(reference "J43")
 					(unit 1)
 				)
@@
 		(dnp no)
 		(fields_autoplaced yes)
-		(property "Reference" "#PWR0212"
+		(property "Reference" "#PWR0244"
 			(at 106.68 99.06 0)
 			(effects
@@
 			(project "bcrl_power_supply"
 				(path "/77f0f57c-9586-4625-9281-fa8cbd8015db/396cd466-5b94-4a70-b29a-66669aea6a97"
-					(reference "#PWR0212")
-					(unit 1)
-				)
-				(path "/77f0f57c-9586-4625-9281-fa8cbd8015db/66481d9d-6957-47e9-a2b4-eda0119b346e"
-					(reference "#PWR0215")
+					(reference "#PWR0244")
+					(unit 1)
+				)
+				(path "/77f0f57c-9586-4625-9281-fa8cbd8015db/66481d9d-6957-47e9-a2b4-eda0119b346e"
+					(reference "#PWR0247")
 					(unit 1)
 				)
@@
 		(dnp no)
 		(fields_autoplaced yes)
-		(property "Reference" "#PWR0214"
+		(property "Reference" "#PWR0246"
 			(at 64.77 132.715 0)
 			(effects
@@
 			(project "bcrl_power_supply"
 				(path "/77f0f57c-9586-4625-9281-fa8cbd8015db/66481d9d-6957-47e9-a2b4-eda0119b346e"
-					(reference "#PWR0214")
-					(unit 1)
-				)
-				(path "/77f0f57c-9586-4625-9281-fa8cbd8015db/396cd466-5b94-4a70-b29a-66669aea6a97"
-					(reference "#PWR0211")
+					(reference "#PWR0246")
+					(unit 1)
+				)
+				(path "/77f0f57c-9586-4625-9281-fa8cbd8015db/396cd466-5b94-4a70-b29a-66669aea6a97"
+					(reference "#PWR0243")
 					(unit 1)
 				)
@@
 		(dnp no)
 		(fields_autoplaced yes)
-		(property "Reference" "R61"
+		(property "Reference" "R59"
 			(at 96.52 92.71 90)
 			(effects
@@
 			)
 		)
+		(property "rating" ""
+			(at 96.52 99.06 0)
+			(effects
+				(font
+					(size 1.27 1.27)
+				)
+				(hide yes)
+			)
+		)
 		(pin "1"
 		)
@@
 			(project "bcrl_power_supply"
 				(path "/77f0f57c-9586-4625-9281-fa8cbd8015db/396cd466-5b94-4a70-b29a-66669aea6a97"
-					(reference "R61")
-					(unit 1)
-				)
-				(path "/77f0f57c-9586-4625-9281-fa8cbd8015db/66481d9d-6957-47e9-a2b4-eda0119b346e"
-					(reference "R62")
-					(unit 1)
-				)
+					(reference "R59")
+					(unit 1)
+				)
+				(path "/77f0f57c-9586-4625-9281-fa8cbd8015db/66481d9d-6957-47e9-a2b4-eda0119b346e"
+					(reference "R60")
+					(unit 1)
+				)

Commit message: board review
Parts:
- added D10: LED 0603, LED_SMD:LED_0603_1608Metric, symbol Device:LED
- added J78: OSTVN02A150, BCRL_power_supply:CONN_OSTVN02A150_OST, symbol 2024-02-14_22-22-09:OSTVN02A150
- added J79: Conn_01x02, Connector_PinHeader_2.54mm:PinHeader_1x02_P2.54mm_Vertical, symbol Connector_Generic:Conn_01x02
- added R13: 1k, Resistor_SMD:R_0603_1608Metric, symbol Device:R
- D35: value LED -> LED 0603
- renumbered J44 to J42, J45 to J43
Connections:
- net GND: now also J78.2, J79.2 (Pin_2), R13.1
- net +5V renamed +5V_Tx
- net CTRL renamed CTRL_Tx
- new net: D10.1 (K), R13.2
- new net +5V_Rx: D10.2 (A), J78.1
- new net CTRL_Rx: J79.1 (Pin_1)
Other:
- added sheet PDQ10-Q48-S5-D_EMC_18 (PDQ10-Q48-S5-D_EMC.kicad_sch)
- moved on the sheet: D35, J42, J43, R59

Commit message: digikey BOM
Parts:
- D10, D35: DigiKey_Part_Number (none) -> 150060GS75000
- J42, J78: DigiKey_Part_Number (none) -> OSTVN02A150
- R13, R59: DigiKey_Part_Number (none) -> ESR03EZPF1001
Changed lines of the file:
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@@
+			)
+		)
+		(property "DigiKey_Part_Number" "OSTVN02A150"
+			(at 123.19 118.11 0)
+			(effects
+				(font
+					(size 1.27 1.27)
+				)
+				(hide yes)
 			)
 		)
@@
 			)
 		)
-		(property "Description" ""
+		(property "Description" "LED diode"
 			(at 153.67 96.52 0)
 			(effects
@@
 		)
 		(property "rating" ""
+			(at 153.67 96.52 0)
+			(effects
+				(font
+					(size 1.27 1.27)
+				)
+				(hide yes)
+			)
+		)
+		(property "DigiKey_Part_Number" "150060GS75000 "
 			(at 153.67 96.52 0)
 			(effects
@@
 			)
 		)
-		(property "Description" ""
+		(property "Description" "Resistor"
 			(at 82.55 88.9 0)
 			(effects
@@
 			)
 		)
+		(property "DigiKey_Part_Number" "ESR03EZPF1001 "
+			(at 82.55 88.9 0)
+			(effects
+				(font
+					(size 1.27 1.27)
+				)
+				(hide yes)
+			)
+		)
 		(pin "1"
 		)
@@
 		)
 		(property "rating" ""
+			(at 50.8 118.11 0)
+			(effects
+				(font
+					(size 1.27 1.27)
+				)
+				(hide yes)
+			)
+		)
+		(property "DigiKey_Part_Number" "OSTVN02A150"
 			(at 50.8 118.11 0)
 			(effects
@@
 			)
 		)
-		(property "Description" ""
+		(property "Description" "Resistor"
 			(at 153.67 88.9 0)
 			(effects
@@
 		)
 		(property "rating" ""
+			(at 153.67 88.9 0)
+			(effects
+				(font
+					(size 1.27 1.27)
+				)
+				(hide yes)
+			)
+		)
+		(property "DigiKey_Part_Number" "ESR03EZPF1001 "
 			(at 153.67 88.9 0)
 			(effects
@@
 			)
 		)
-		(property "Description" ""
+		(property "Description" "LED diode"
 			(at 82.55 96.52 0)
 			(effects
@@
 			(at 82.55 96.52 0)
 			(effects
+				(font
+					(size 1.27 1.27)
+				)
+				(hide yes)
+			)
+		)
+		(property "DigiKey_Part_Number" "150060GS75000 "
+			(at 82.55 96.52 0)
+			(effects
