File: kicad_files/bcrl_power_supply/PDQ10-Q48-S3-D_EMC.kicad_sch (KiCad schematic)
At the start: 3 parts, among them U1 PDQ10-Q48-S3-D

Commit message: WIP
Parts:
- renumbered C13 to C79, C14 to C80, U1 to U2
Changed lines of the file:
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@@
   (symbol (lib_id "BCRL_power_supply:PDQ10-Q48-S3-D") (at 125.73 88.9 0) (unit 1)
     (in_bom yes) (on_board yes) (dnp no) (fields_autoplaced)
-    (property "Reference" "U1" (at 125.73 73.66 0)
+    (property "Reference" "U2" (at 125.73 73.66 0)
       (effects (font (size 1.27 1.27)))
     )
@@
     (instances
       (project "bcrl_power_supply"
-        (path "/77f0f57c-9586-4625-9281-fa8cbd8015db/94fee228-5462-46f6-ad6c-1e47c0f1b343/1086eb20-5b82-4ba4-858a-8bee05c23fdd"
-          (reference "U1") (unit 1)
+        (path "/77f0f57c-9586-4625-9281-fa8cbd8015db/86d69f20-72a8-480c-899a-1cc522974f16/304888ea-efce-4e81-86e4-683c64fddcb4"
+          (reference "U2") (unit 1)
         )
-        (path "/77f0f57c-9586-4625-9281-fa8cbd8015db/86d69f20-72a8-480c-899a-1cc522974f16/304888ea-efce-4e81-86e4-683c64fddcb4"
+        (path "/77f0f57c-9586-4625-9281-fa8cbd8015db/6ef64b97-f9dc-450f-b711-7d52ab21fa20"
           (reference "U2") (unit 1)
         )
@@
   (symbol (lib_id "Device:C_Polarized") (at 81.28 92.71 0) (unit 1)
     (in_bom yes) (on_board yes) (dnp no) (fields_autoplaced)
-    (property "Reference" "C14" (at 85.09 90.551 0)
+    (property "Reference" "C80" (at 85.09 90.551 0)
       (effects (font (size 1.27 1.27)) (justify left))
     )
@@
     (instances
       (project "bcrl_power_supply"
-        (path "/77f0f57c-9586-4625-9281-fa8cbd8015db/94fee228-5462-46f6-ad6c-1e47c0f1b343/1086eb20-5b82-4ba4-858a-8bee05c23fdd"
-          (reference "C14") (unit 1)
+        (path "/77f0f57c-9586-4625-9281-fa8cbd8015db/86d69f20-72a8-480c-899a-1cc522974f16/304888ea-efce-4e81-86e4-683c64fddcb4"
+          (reference "C80") (unit 1)
         )
-        (path "/77f0f57c-9586-4625-9281-fa8cbd8015db/86d69f20-72a8-480c-899a-1cc522974f16/304888ea-efce-4e81-86e4-683c64fddcb4"
+        (path "/77f0f57c-9586-4625-9281-fa8cbd8015db/6ef64b97-f9dc-450f-b711-7d52ab21fa20"
           (reference "C80") (unit 1)
         )
@@
   (symbol (lib_id "Device:C_Polarized") (at 60.96 92.71 0) (unit 1)
     (in_bom yes) (on_board yes) (dnp no)
-    (property "Reference" "C13" (at 64.77 90.551 0)
+    (property "Reference" "C79" (at 64.77 90.551 0)
       (effects (font (size 1.27 1.27)) (justify left))
     )
@@
     (instances
       (project "bcrl_power_supply"
-        (path "/77f0f57c-9586-4625-9281-fa8cbd8015db/94fee228-5462-46f6-ad6c-1e47c0f1b343/1086eb20-5b82-4ba4-858a-8bee05c23fdd"
-          (reference "C13") (unit 1)
+        (path "/77f0f57c-9586-4625-9281-fa8cbd8015db/86d69f20-72a8-480c-899a-1cc522974f16/304888ea-efce-4e81-86e4-683c64fddcb4"
+          (reference "C79") (unit 1)
         )
-        (path "/77f0f57c-9586-4625-9281-fa8cbd8015db/86d69f20-72a8-480c-899a-1cc522974f16/304888ea-efce-4e81-86e4-683c64fddcb4"
+        (path "/77f0f57c-9586-4625-9281-fa8cbd8015db/6ef64b97-f9dc-450f-b711-7d52ab21fa20"
           (reference "C79") (unit 1)
         )
@@
   (symbol (lib_id "power:GND") (at 143.51 86.36 0) (unit 1)
     (in_bom yes) (on_board yes) (dnp no) (fields_autoplaced)
-    (property "Reference" "#PWR062" (at 143.51 92.71 0)
+    (property "Reference" "#PWR0208" (at 143.51 92.71 0)
       (effects (font (size 1.27 1.27)) hide)
     )
@@
     (instances
       (project "bcrl_power_supply"
-        (path "/77f0f57c-9586-4625-9281-fa8cbd8015db/94fee228-5462-46f6-ad6c-1e47c0f1b343/1086eb20-5b82-4ba4-858a-8bee05c23fdd"
-          (reference "#PWR062") (unit 1)
+        (path "/77f0f57c-9586-4625-9281-fa8cbd8015db/86d69f20-72a8-480c-899a-1cc522974f16/304888ea-efce-4e81-86e4-683c64fddcb4"
+          (reference "#PWR0208") (unit 1)
         )
-        (path "/77f0f57c-9586-4625-9281-fa8cbd8015db/86d69f20-72a8-480c-899a-1cc522974f16/304888ea-efce-4e81-86e4-683c64fddcb4"
+        (path "/77f0f57c-9586-4625-9281-fa8cbd8015db/6ef64b97-f9dc-450f-b711-7d52ab21fa20"
           (reference "#PWR0141") (unit 1)
         )
@@
   (symbol (lib_id "power:GND") (at 49.53 101.6 0) (unit 1)
     (in_bom yes) (on_board yes) (dnp no)
-    (property "Reference" "#PWR061" (at 49.53 107.95 0)
+    (property "Reference" "#PWR0207" (at 49.53 107.95 0)
       (effects (font (size 1.27 1.27)) hide)
     )
@@
     (instances
       (project "bcrl_power_supply"
-        (path "/77f0f57c-9586-4625-9281-fa8cbd8015db/94fee228-5462-46f6-ad6c-1e47c0f1b343/1086eb20-5b82-4ba4-858a-8bee05c23fdd"
-          (reference "#PWR061") (unit 1)
+        (path "/77f0f57c-9586-4625-9281-fa8cbd8015db/86d69f20-72a8-480c-899a-1cc522974f16/304888ea-efce-4e81-86e4-683c64fddcb4"
+          (reference "#PWR0207") (unit 1)
         )
-        (path "/77f0f57c-9586-4625-9281-fa8cbd8015db/86d69f20-72a8-480c-899a-1cc522974f16/304888ea-efce-4e81-86e4-683c64fddcb4"
+        (path "/77f0f57c-9586-4625-9281-fa8cbd8015db/6ef64b97-f9dc-450f-b711-7d52ab21fa20"
           (reference "#PWR0140") (unit 1)
         )

Commit message: cleanup PCB
Parts:
- renumbered C79 to C5, C80 to C6, U2 to U3
Changed lines of the file:
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@@
   (symbol (lib_id "BCRL_power_supply:PDQ10-Q48-S3-D") (at 125.73 88.9 0) (unit 1)
     (in_bom yes) (on_board yes) (dnp no) (fields_autoplaced)
-    (property "Reference" "U2" (at 125.73 73.66 0)
+    (property "Reference" "U3" (at 125.73 73.66 0)
       (effects (font (size 1.27 1.27)))
     )
@@
     (instances
       (project "bcrl_power_supply"
-        (path "/77f0f57c-9586-4625-9281-fa8cbd8015db/86d69f20-72a8-480c-899a-1cc522974f16/304888ea-efce-4e81-86e4-683c64fddcb4"
-          (reference "U2") (unit 1)
-        )
         (path "/77f0f57c-9586-4625-9281-fa8cbd8015db/6ef64b97-f9dc-450f-b711-7d52ab21fa20"
-          (reference "U2") (unit 1)
+          (reference "U3") (unit 1)
         )
       )
@@
   (symbol (lib_id "Device:C_Polarized") (at 81.28 92.71 0) (unit 1)
     (in_bom yes) (on_board yes) (dnp no) (fields_autoplaced)
-    (property "Reference" "C80" (at 85.09 90.551 0)
+    (property "Reference" "C6" (at 85.09 90.551 0)
       (effects (font (size 1.27 1.27)) (justify left))
     )
@@
     (instances
       (project "bcrl_power_supply"
-        (path "/77f0f57c-9586-4625-9281-fa8cbd8015db/86d69f20-72a8-480c-899a-1cc522974f16/304888ea-efce-4e81-86e4-683c64fddcb4"
-          (reference "C80") (unit 1)
-        )
         (path "/77f0f57c-9586-4625-9281-fa8cbd8015db/6ef64b97-f9dc-450f-b711-7d52ab21fa20"
-          (reference "C80") (unit 1)
+          (reference "C6") (unit 1)
         )
       )
@@
   (symbol (lib_id "Device:C_Polarized") (at 60.96 92.71 0) (unit 1)
     (in_bom yes) (on_board yes) (dnp no)
-    (property "Reference" "C79" (at 64.77 90.551 0)
+    (property "Reference" "C5" (at 64.77 90.551 0)
       (effects (font (size 1.27 1.27)) (justify left))
     )
@@
     (instances
       (project "bcrl_power_supply"
-        (path "/77f0f57c-9586-4625-9281-fa8cbd8015db/86d69f20-72a8-480c-899a-1cc522974f16/304888ea-efce-4e81-86e4-683c64fddcb4"
-          (reference "C79") (unit 1)
-        )
         (path "/77f0f57c-9586-4625-9281-fa8cbd8015db/6ef64b97-f9dc-450f-b711-7d52ab21fa20"
-          (reference "C79") (unit 1)
+          (reference "C5") (unit 1)
         )
       )
@@
   (symbol (lib_id "power:GND") (at 143.51 86.36 0) (unit 1)
     (in_bom yes) (on_board yes) (dnp no) (fields_autoplaced)
-    (property "Reference" "#PWR0208" (at 143.51 92.71 0)
+    (property "Reference" "#PWR064" (at 143.51 92.71 0)
       (effects (font (size 1.27 1.27)) hide)
     )
@@
     (instances
       (project "bcrl_power_supply"
-        (path "/77f0f57c-9586-4625-9281-fa8cbd8015db/86d69f20-72a8-480c-899a-1cc522974f16/304888ea-efce-4e81-86e4-683c64fddcb4"
-          (reference "#PWR0208") (unit 1)
-        )
         (path "/77f0f57c-9586-4625-9281-fa8cbd8015db/6ef64b97-f9dc-450f-b711-7d52ab21fa20"
-          (reference "#PWR0141") (unit 1)
+          (reference "#PWR064") (unit 1)
         )
       )
@@
   (symbol (lib_id "power:GND") (at 49.53 101.6 0) (unit 1)
     (in_bom yes) (on_board yes) (dnp no)
-    (property "Reference" "#PWR0207" (at 49.53 107.95 0)
+    (property "Reference" "#PWR063" (at 49.53 107.95 0)
       (effects (font (size 1.27 1.27)) hide)
     )
@@
     (instances
       (project "bcrl_power_supply"
-        (path "/77f0f57c-9586-4625-9281-fa8cbd8015db/86d69f20-72a8-480c-899a-1cc522974f16/304888ea-efce-4e81-86e4-683c64fddcb4"
-          (reference "#PWR0207") (unit 1)
-        )
         (path "/77f0f57c-9586-4625-9281-fa8cbd8015db/6ef64b97-f9dc-450f-b711-7d52ab21fa20"
-          (reference "#PWR0140") (unit 1)
+          (reference "#PWR063") (unit 1)
         )
       )

Commit message: started LCSC, fixing DCDC
Parts:
- C5: LCSC (none) -> C784420
- C6: value 4.7uf/100uf -> 4.7uf/100v; LCSC (none) -> C784420
Changed lines of the file:
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@@
+			)
+		)
+		(property "LCSC" ""
+			(at 125.73 88.9 0)
+			(effects
+				(font
+					(size 1.27 1.27)
+				)
+				(hide yes)
 			)
 		)
@@
 			)
 		)
-		(property "Value" "4.7uf/100uf"
+		(property "Value" "4.7uf/100v"
 			(at 85.09 93.091 0)
 			(effects
@@
 		)
 		(property "Description" ""
+			(at 81.28 92.71 0)
+			(effects
+				(font
+					(size 1.27 1.27)
+				)
+				(hide yes)
+			)
+		)
+		(property "LCSC" "C784420"
 			(at 81.28 92.71 0)
 			(effects
@@
 			(at 60.96 92.71 0)
 			(effects
+				(font
+					(size 1.27 1.27)
+				)
+				(hide yes)
+			)
+		)
+		(property "LCSC" "C784420"
+			(at 60.96 92.71 0)
+			(effects
