File: kicad_files/bcrl_power_supply/PDQ10-Q48-S3-D_EMC.kicad_sch (KiCad schematic)
At the start: 3 parts, among them U3 PDQ10-Q48-S3-D

Commit message: almost done schematic
Parts:
- C5, C6: value 4.7uf/100v -> 4.7u; rating (none) -> 100v
Changed lines of the file:
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@@
+			)
+		)
+		(property "rating" ""
+			(at 125.73 88.9 0)
+			(effects
+				(font
+					(size 1.27 1.27)
+				)
+				(hide yes)
 			)
 		)
@@
 			)
 		)
-		(property "Value" "4.7uf/100v"
+		(property "Value" "4.7u"
 			(at 85.09 93.091 0)
 			(effects
@@
 		)
 		(property "SNAPEDA_PN" ""
+			(at 81.28 92.71 0)
+			(effects
+				(font
+					(size 1.27 1.27)
+				)
+				(hide yes)
+			)
+		)
+		(property "rating" "100v"
 			(at 81.28 92.71 0)
 			(effects
@@
 			)
 		)
-		(property "Value" "4.7uf/100v"
+		(property "Value" "4.7u"
 			(at 64.77 92.71 0)
 			(effects
@@
 		)
 		(property "SNAPEDA_PN" ""
+			(at 60.96 92.71 0)
+			(effects
+				(font
+					(size 1.27 1.27)
+				)
+				(hide yes)
+			)
+		)
+		(property "rating" "100v"
 			(at 60.96 92.71 0)
 			(effects
@@
 		(dnp no)
 		(fields_autoplaced yes)
-		(property "Reference" "#PWR061"
+		(property "Reference" "#PWR063"
 			(at 143.51 92.71 0)
 			(effects
@@
 			(project "bcrl_power_supply"
 				(path "/77f0f57c-9586-4625-9281-fa8cbd8015db/6ef64b97-f9dc-450f-b711-7d52ab21fa20"
-					(reference "#PWR061")
+					(reference "#PWR063")
 					(unit 1)
 				)
@@
 		(on_board yes)
 		(dnp no)
-		(property "Reference" "#PWR060"
+		(property "Reference" "#PWR062"
 			(at 49.53 107.95 0)
 			(effects
@@
 			(project "bcrl_power_supply"
 				(path "/77f0f57c-9586-4625-9281-fa8cbd8015db/6ef64b97-f9dc-450f-b711-7d52ab21fa20"
-					(reference "#PWR060")
-					(unit 1)
-				)
+					(reference "#PWR062")
+					(unit 1)
+				)

Commit message: digikey BOM
Parts:
- C5, C6: value 4.7u -> 4.7u; footprint Capacitor_SMD:C_0603_1608Metric -> Capacitor_SMD:C_1206_3216Metric; DigiKey_Part_Number (none) -> GRM31CC72A475KE11L
- U3: DigiKey_Part_Number (none) -> PDQ10-Q48-S3-D
Changed lines of the file:
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@@
+			)
+		)
+		(property "DigiKey_Part_Number" "PDQ10-Q48-S3-D"
+			(at 125.73 88.9 0)
+			(effects
+				(font
+					(size 1.27 1.27)
+				)
+				(hide yes)
 			)
 		)
@@
 			)
 		)
-		(property "Value" "4.7u"
+		(property "Value" " 4.7u"
 			(at 85.09 93.091 0)
 			(effects
@@
 			)
 		)
-		(property "Footprint" "Capacitor_SMD:C_0603_1608Metric"
+		(property "Footprint" "Capacitor_SMD:C_1206_3216Metric"
 			(at 82.2452 96.52 0)
 			(effects
@@
 		)
 		(property "rating" "100v"
+			(at 81.28 92.71 0)
+			(effects
+				(font
+					(size 1.27 1.27)
+				)
+				(hide yes)
+			)
+		)
+		(property "DigiKey_Part_Number" "GRM31CC72A475KE11L "
 			(at 81.28 92.71 0)
 			(effects
@@
 			)
 		)
-		(property "Value" "4.7u"
+		(property "Value" " 4.7u"
 			(at 64.77 92.71 0)
 			(effects
@@
 			)
 		)
-		(property "Footprint" "Capacitor_SMD:C_0603_1608Metric"
+		(property "Footprint" "Capacitor_SMD:C_1206_3216Metric"
 			(at 61.9252 96.52 0)
 			(effects
@@
 			(at 60.96 92.71 0)
 			(effects
+				(font
+					(size 1.27 1.27)
+				)
+				(hide yes)
+			)
+		)
+		(property "DigiKey_Part_Number" "GRM31CC72A475KE11L "
+			(at 60.96 92.71 0)
+			(effects
