File: kicad_files/bcrl_power_supply/PDQ10-Q48-S5-D_EMC.kicad_sch (KiCad schematic)
At the start: 5 parts, among them U8 PDQ10-Q48-S5-D

Commit message: ...
Parts:
- renumbered C111 to C119, C112 to C120, L31 to L35, R11 to R32, U8 to U12
Connections:
- net VIN: now reaches C120.1, L35.2, U12.1 (+VIN)
Other:
- moved on the sheet: C119, C120, L35, R32, U12

Commit message: almost done schematic
Changed lines of the file:
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@@
+		)
+	)
+	(text_box "Trim up 10%, 3400 ohms\n"
+		(exclude_from_sim no)
+		(at 165.1 123.19 0)
+		(size 24.13 7.62)
+		(stroke
+			(width 0)
+			(type default)
+		)
+		(fill
+			(type none)
+		)
+		(effects
+			(font
+				(size 1.27 1.27)
+			)
+			(justify left top)
 		)
 	)

Commit message: started LCSC, fixing DCDC
Parts:
- C119, C120: LCSC (none) -> C784420
Changed lines of the file:
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@@
+			)
+		)
+		(property "LCSC" "C784420"
+			(at 95.25 105.41 0)
+			(effects
+				(font
+					(size 1.27 1.27)
+				)
+				(hide yes)
 			)
 		)
@@
 			)
 		)
+		(property "LCSC" ""
+			(at 170.18 106.68 0)
+			(effects
+				(font
+					(size 1.27 1.27)
+				)
+				(hide yes)
+			)
+		)
 		(pin "2"
 		)
@@
 			)
 		)
+		(property "LCSC" "C784420"
+			(at 111.76 105.41 0)
+			(effects
+				(font
+					(size 1.27 1.27)
+				)
+				(hide yes)
+			)
+		)
 		(pin "2"
 		)
@@
 			)
 		)
+		(property "LCSC" ""
+			(at 104.14 97.79 0)
+			(effects
+				(font
+					(size 1.27 1.27)
+				)
+				(hide yes)
+			)
+		)
 		(pin "1"
 		)
@@
 				(hide yes)
 			)
+		)
+		(property "LCSC" ""
+			(at 152.4 102.87 0)
+			(effects
+				(font
+					(size 1.27 1.27)
+				)
+				(hide yes)
+			)

Commit message: big reorg
Parts:
- renumbered C119 to C41, C120 to C42, L35 to L8, R32 to R19, U12 to U5

Commit message: big changes
Parts:
- renumbered C41 to C39, C42 to C40, L8 to L7, R19 to R20, U5 to U4
