File: kicad_files/bcrl_power_supply/PDQ10-Q48-S5-D_EMC.kicad_sch (KiCad schematic)
At the start: 5 parts, among them U4 PDQ10-Q48-S5-D

Commit message: almost done schematic
Parts:
- C35: renamed from C39; value 4.7uf/100v -> 4.7u; rating (none) -> 100v
- C36: renamed from C40; value 4.7uf/100v -> 4.7u; rating (none) -> 100v
- L3: renamed from L7; value 4.7uh/3.1a -> 4.7u; rating (none) -> 3.1a
- renumbered R20 to R22

Commit message: board review
Parts:
- renumbered C35 to C37, C36 to C38, L3 to L4, R22 to R32, U4 to U5
Changed lines of the file:
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@@
 		(dnp no)
 		(fields_autoplaced yes)
-		(property "Reference" "C35"
+		(property "Reference" "C37"
 			(at 99.06 104.14 0)
 			(effects
@@
 		(instances
 			(project "bcrl_power_supply"
-				(path "/77f0f57c-9586-4625-9281-fa8cbd8015db/66481d9d-6957-47e9-a2b4-eda0119b346e/13fbb956-887b-499a-a3e4-266e83b0f717"
-					(reference "C35")
-					(unit 1)
-				)
 				(path "/77f0f57c-9586-4625-9281-fa8cbd8015db/396cd466-5b94-4a70-b29a-66669aea6a97/13fbb956-887b-499a-a3e4-266e83b0f717"
 					(reference "C37")
@@
 				(path "/77f0f57c-9586-4625-9281-fa8cbd8015db/d38a281a-ebcf-4be6-8e3c-19a868b0087f/d4052f31-6719-4a3f-8e3d-840c16382ac2"
 					(reference "C129")
+					(unit 1)
+				)
+				(path "/77f0f57c-9586-4625-9281-fa8cbd8015db/396cd466-5b94-4a70-b29a-66669aea6a97/cf0e2c0b-fd3e-4094-bc6a-217321274aee"
+					(reference "C39")
 					(unit 1)
 				)
@@
 		(dnp no)
 		(fields_autoplaced yes)
-		(property "Reference" "R22"
+		(property "Reference" "R32"
 			(at 172.72 105.41 0)
 			(effects
@@
 		(instances
 			(project "bcrl_power_supply"
-				(path "/77f0f57c-9586-4625-9281-fa8cbd8015db/66481d9d-6957-47e9-a2b4-eda0119b346e/13fbb956-887b-499a-a3e4-266e83b0f717"
-					(reference "R22")
-					(unit 1)
-				)
 				(path "/77f0f57c-9586-4625-9281-fa8cbd8015db/396cd466-5b94-4a70-b29a-66669aea6a97/13fbb956-887b-499a-a3e4-266e83b0f717"
 					(reference "R32")
@@
 				(path "/77f0f57c-9586-4625-9281-fa8cbd8015db/d38a281a-ebcf-4be6-8e3c-19a868b0087f/d4052f31-6719-4a3f-8e3d-840c16382ac2"
 					(reference "R61")
+					(unit 1)
+				)
+				(path "/77f0f57c-9586-4625-9281-fa8cbd8015db/396cd466-5b94-4a70-b29a-66669aea6a97/cf0e2c0b-fd3e-4094-bc6a-217321274aee"
+					(reference "R12")
 					(unit 1)
 				)
@@
 		(dnp no)
 		(fields_autoplaced yes)
-		(property "Reference" "C36"
+		(property "Reference" "C38"
 			(at 115.57 104.14 0)
 			(effects
@@
 		(instances
 			(project "bcrl_power_supply"
-				(path "/77f0f57c-9586-4625-9281-fa8cbd8015db/66481d9d-6957-47e9-a2b4-eda0119b346e/13fbb956-887b-499a-a3e4-266e83b0f717"
-					(reference "C36")
-					(unit 1)
-				)
 				(path "/77f0f57c-9586-4625-9281-fa8cbd8015db/396cd466-5b94-4a70-b29a-66669aea6a97/13fbb956-887b-499a-a3e4-266e83b0f717"
 					(reference "C38")
@@
 				(path "/77f0f57c-9586-4625-9281-fa8cbd8015db/d38a281a-ebcf-4be6-8e3c-19a868b0087f/d4052f31-6719-4a3f-8e3d-840c16382ac2"
 					(reference "C130")
+					(unit 1)
+				)
+				(path "/77f0f57c-9586-4625-9281-fa8cbd8015db/396cd466-5b94-4a70-b29a-66669aea6a97/cf0e2c0b-fd3e-4094-bc6a-217321274aee"
+					(reference "C40")
 					(unit 1)
 				)
@@
 		(dnp no)
 		(fields_autoplaced yes)
-		(property "Reference" "L3"
+		(property "Reference" "L4"
 			(at 104.14 92.71 90)
 			(effects
@@
 		(instances
 			(project "bcrl_power_supply"
-				(path "/77f0f57c-9586-4625-9281-fa8cbd8015db/66481d9d-6957-47e9-a2b4-eda0119b346e/13fbb956-887b-499a-a3e4-266e83b0f717"
-					(reference "L3")
-					(unit 1)
-				)
 				(path "/77f0f57c-9586-4625-9281-fa8cbd8015db/396cd466-5b94-4a70-b29a-66669aea6a97/13fbb956-887b-499a-a3e4-266e83b0f717"
 					(reference "L4")
@@
 				(path "/77f0f57c-9586-4625-9281-fa8cbd8015db/d38a281a-ebcf-4be6-8e3c-19a868b0087f/d4052f31-6719-4a3f-8e3d-840c16382ac2"
 					(reference "L15")
+					(unit 1)
+				)
+				(path "/77f0f57c-9586-4625-9281-fa8cbd8015db/396cd466-5b94-4a70-b29a-66669aea6a97/cf0e2c0b-fd3e-4094-bc6a-217321274aee"
+					(reference "L5")
 					(unit 1)
 				)
@@
 		(dnp no)
 		(fields_autoplaced yes)
-		(property "Reference" "U4"
+		(property "Reference" "U5"
 			(at 152.4 87.63 0)
 			(effects
@@
 		(instances
 			(project "bcrl_power_supply"
-				(path "/77f0f57c-9586-4625-9281-fa8cbd8015db/66481d9d-6957-47e9-a2b4-eda0119b346e/13fbb956-887b-499a-a3e4-266e83b0f717"
-					(reference "U4")
-					(unit 1)
-				)
 				(path "/77f0f57c-9586-4625-9281-fa8cbd8015db/396cd466-5b94-4a70-b29a-66669aea6a97/13fbb956-887b-499a-a3e4-266e83b0f717"
 					(reference "U5")
@@
 				(path "/77f0f57c-9586-4625-9281-fa8cbd8015db/d38a281a-ebcf-4be6-8e3c-19a868b0087f/d4052f31-6719-4a3f-8e3d-840c16382ac2"
 					(reference "U14")
+					(unit 1)
+				)
+				(path "/77f0f57c-9586-4625-9281-fa8cbd8015db/396cd466-5b94-4a70-b29a-66669aea6a97/cf0e2c0b-fd3e-4094-bc6a-217321274aee"
+					(reference "U6")
 					(unit 1)
 				)
@@
 		(dnp no)
 		(fields_autoplaced yes)
-		(property "Reference" "#PWR096"
+		(property "Reference" "#PWR0156"
 			(at 80.01 119.38 0)
 			(effects
@@
 		(instances
 			(project "bcrl_power_supply"
-				(path "/77f0f57c-9586-4625-9281-fa8cbd8015db/66481d9d-6957-47e9-a2b4-eda0119b346e/13fbb956-887b-499a-a3e4-266e83b0f717"
-					(reference "#PWR096")
-					(unit 1)
-				)
 				(path "/77f0f57c-9586-4625-9281-fa8cbd8015db/396cd466-5b94-4a70-b29a-66669aea6a97/13fbb956-887b-499a-a3e4-266e83b0f717"
 					(reference "#PWR0156")
@@
 				(path "/77f0f57c-9586-4625-9281-fa8cbd8015db/d38a281a-ebcf-4be6-8e3c-19a868b0087f/d4052f31-6719-4a3f-8e3d-840c16382ac2"
 					(reference "#PWR0324")
+					(unit 1)
+				)
+				(path "/77f0f57c-9586-4625-9281-fa8cbd8015db/396cd466-5b94-4a70-b29a-66669aea6a97/cf0e2c0b-fd3e-4094-bc6a-217321274aee"
+					(reference "#PWR064")
 					(unit 1)
 				)
@@
 		(dnp no)
 		(fields_autoplaced yes)
-		(property "Reference" "#PWR097"
+		(property "Reference" "#PWR0157"
 			(at 198.755 106.68 0)
 			(effects
@@
 		(instances
 			(project "bcrl_power_supply"
-				(path "/77f0f57c-9586-4625-9281-fa8cbd8015db/66481d9d-6957-47e9-a2b4-eda0119b346e/13fbb956-887b-499a-a3e4-266e83b0f717"
-					(reference "#PWR097")
-					(unit 1)
-				)
 				(path "/77f0f57c-9586-4625-9281-fa8cbd8015db/396cd466-5b94-4a70-b29a-66669aea6a97/13fbb956-887b-499a-a3e4-266e83b0f717"
 					(reference "#PWR0157")
@@
 					(unit 1)
 				)
+				(path "/77f0f57c-9586-4625-9281-fa8cbd8015db/396cd466-5b94-4a70-b29a-66669aea6a97/cf0e2c0b-fd3e-4094-bc6a-217321274aee"
+					(reference "#PWR065")
+					(unit 1)
+				)

Commit message: digikey BOM
Parts:
- C37, C38: value 4.7u -> 4.7u; footprint Capacitor_SMD:C_0603_1608Metric -> Capacitor_SMD:C_1206_3216Metric; DigiKey_Part_Number (none) -> GRM31CC72A475KE11L
- L4: DigiKey_Part_Number (none) -> MGAH06034R7M-10
- R32: DigiKey_Part_Number (none) -> TNPW06033K40BEEA
- U5: DigiKey_Part_Number (none) -> PDQ10-Q48-S5-D
Changed lines of the file:
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@@
 			)
 		)
-		(property "Value" "4.7u"
+		(property "Value" " 4.7u"
 			(at 99.06 106.68 0)
 			(effects
@@
 			)
 		)
-		(property "Footprint" "Capacitor_SMD:C_0603_1608Metric"
+		(property "Footprint" "Capacitor_SMD:C_1206_3216Metric"
 			(at 96.2152 109.22 0)
 			(effects
@@
 		)
 		(property "rating" "100v"
+			(at 95.25 105.41 0)
+			(effects
+				(font
+					(size 1.27 1.27)
+				)
+				(hide yes)
+			)
+		)
+		(property "DigiKey_Part_Number" "GRM31CC72A475KE11L "
 			(at 95.25 105.41 0)
 			(effects
@@
 			)
 		)
-		(property "Description" ""
+		(property "Description" "Resistor"
 			(at 170.18 106.68 0)
 			(effects
@@
 		)
 		(property "rating" ""
+			(at 170.18 106.68 0)
+			(effects
+				(font
+					(size 1.27 1.27)
+				)
+				(hide yes)
+			)
+		)
+		(property "DigiKey_Part_Number" "TNPW06033K40BEEA "
 			(at 170.18 106.68 0)
 			(effects
@@
 			)
 		)
-		(property "Value" "4.7u"
+		(property "Value" " 4.7u"
 			(at 115.57 106.68 0)
 			(effects
@@
 			)
 		)
-		(property "Footprint" "Capacitor_SMD:C_0603_1608Metric"
+		(property "Footprint" "Capacitor_SMD:C_1206_3216Metric"
 			(at 112.7252 109.22 0)
 			(effects
@@
 		)
 		(property "rating" "100v"
+			(at 111.76 105.41 0)
+			(effects
+				(font
+					(size 1.27 1.27)
+				)
+				(hide yes)
+			)
+		)
+		(property "DigiKey_Part_Number" "GRM31CC72A475KE11L "
 			(at 111.76 105.41 0)
 			(effects
@@
 			)
 		)
-		(property "Description" ""
+		(property "Description" "Inductor"
 			(at 104.14 97.79 0)
 			(effects
@@
 		)
 		(property "rating" "3.1a"
+			(at 104.14 97.79 0)
+			(effects
+				(font
+					(size 1.27 1.27)
+				)
+				(hide yes)
+			)
+		)
+		(property "DigiKey_Part_Number" "MGAH06034R7M-10 "
 			(at 104.14 97.79 0)
 			(effects
@@
 			(at 152.4 102.87 0)
 			(effects
+				(font
+					(size 1.27 1.27)
+				)
+				(hide yes)
+			)
+		)
+		(property "DigiKey_Part_Number" "PDQ10-Q48-S5-D"
+			(at 152.4 102.87 0)
+			(effects
