File: kicad_files/bcrl_power_supply/RPi4_HAT_board.kicad_sch (KiCad schematic)
At the start: 1 part, among them J77 Conn_01x06_Pin

Commit message: WIP
Parts:
- added J43, J44, J45: Conn_01x06_Pin, symbol Connector:Conn_01x06_Pin
Connections:
- net +24V: now also J43.3 (Pin_3), J44.3 (Pin_3), J45.3 (Pin_3)
- net +3.3V: now also J43.6 (Pin_6), J44.6 (Pin_6), J45.6 (Pin_6)
- net +5V: now also J43.2 (Pin_2), J44.2 (Pin_2), J45.2 (Pin_2)
- net GND: now also J43.1 (Pin_1), J43.4 (Pin_4), J43.5 (Pin_5), J44.1 (Pin_1), J44.4 (Pin_4), J44.5 (Pin_5), J45.1 (Pin_1), J45.4 (Pin_4), J45.5 (Pin_5)

Commit message: cleanup PCB
Parts:
- J65: renamed from J43; footprint (none) -> Connector_PinHeader_2.54mm:PinHeader_1x06_P2.54mm_Vertical
- J66: renamed from J44; footprint (none) -> Connector_PinHeader_2.54mm:PinHeader_1x06_P2.54mm_Vertical
- J67: renamed from J45; footprint (none) -> Connector_PinHeader_2.54mm:PinHeader_1x06_P2.54mm_Vertical
- J68: renamed from J77; footprint (none) -> Connector_PinHeader_2.54mm:PinHeader_1x06_P2.54mm_Vertical
Connections:
- net +5V renamed +5V_1
- net +5V_1: no longer J66.2 (Pin_2), J67.2 (Pin_2)
- new net +5V_2: J66.2 (Pin_2), J67.2 (Pin_2)
Other:
- added sheet PDQ10-Q48-S5-D_EMC_7 (PDQ10-Q48-S5-D_EMC.kicad_sch)
- added sheet PDQ10-Q48-S5-D_EMC_8 (PDQ10-Q48-S5-D_EMC.kicad_sch)
- added sheet PDQE15-Q48-D24-D_EMC_1 (PDQE15-Q48-D24-D_EMC.kicad_sch)

Commit message: ...
Parts:
- renumbered J65 to J61, J66 to J62, J67 to J63, J68 to J64

Commit message: schematic done
Parts:
- added D27, D29, D31: LED, LED_SMD:LED_0603_1608Metric, symbol Device:LED
- added R54, R57, R59: 1k, Resistor_SMD:R_0603_1608Metric, symbol Device:R
Connections:
- net +24V: now also D29.2 (A)
- net +5V_1: now also D27.2 (A)
- net +5V_2: now also D31.2 (A)
- net GND: now also R54.1, R57.1, R59.1
- new net: D29.1 (K), R57.2
- new net: D27.1 (K), R54.2
- new net: D31.1 (K), R59.2
Other:
- moved on the sheet: J64

Commit message: big reorg
Parts:
- removed D31: LED, LED_SMD:LED_0603_1608Metric, symbol Device:LED
- removed J61, J62, J63, J64: Conn_01x06_Pin, Connector_PinHeader_2.54mm:PinHeader_1x06_P2.54mm_Vertical, symbol Connector:Conn_01x06_Pin
- removed R59: 1k, Resistor_SMD:R_0603_1608Metric, symbol Device:R
- added D10: LED, LED_SMD:LED_0603_1608Metric, symbol Device:LED
- added R12: 1k, Resistor_SMD:R_0603_1608Metric, symbol Device:R
- renumbered D29 to D11, D27 to D9, R54 to R11, R57 to R13
Connections:
- net +5V_2: now also D10.2 (A)
- net GND: now also R12.1
- new net: D10.1 (K), R12.2
Other:
- moved on the sheet: D11, R13

Commit message: big changes
Parts:
- removed D10: LED, LED_SMD:LED_0603_1608Metric, symbol Device:LED
- removed R12: 1k, Resistor_SMD:R_0603_1608Metric, symbol Device:R
Connections:
- net +5V_1 renamed +5V
Other:
- removed sheet PDQ10-Q48-S5-D_EMC_7
- moved on the sheet: D11, D9, R11, R13
