File: kicad_files/bcrl_power_supply/bcrl_power_supply.kicad_sch (KiCad schematic)
At the start: 9 parts, among them J1 OSTVN02A150, J2 OSTVN02A150, J3 Conn_01x02

Commit message: board review
Connections:
- net +48V: no longer J1.1, J2.1
- new net +48V_unfiltered: J1.1, J2.1
Other:
- sheet Tx_Eth_Switch renamed Eth_Switch
- removed sheet Rx_Eth_Switch
- added sheet FLT007A0Z_EMC (FLT007A0Z_EMC.kicad_sch)
- moved on the sheet: J1, J2

Commit message: digikey BOM
Parts:
- J1, J2: DigiKey_Part_Number (none) -> OSTVN02A150
Changed lines of the file:
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@@
+			)
+		)
+		(property "DigiKey_Part_Number" "OSTVN02A150"
+			(at 66.04 34.29 0)
+			(effects
+				(font
+					(size 1.27 1.27)
+				)
+				(hide yes)
 			)
 		)
@@
 			(at 66.04 24.13 0)
 			(effects
+				(font
+					(size 1.27 1.27)
+				)
+				(hide yes)
+			)
+		)
+		(property "DigiKey_Part_Number" "OSTVN02A150"
+			(at 66.04 24.13 0)
+			(effects
