File: kicad_files/bcrl_power_supply/fan_20x.kicad_sch (KiCad schematic)
At the start: 2 parts, among them J23 OSTVN02A150, J69 Conn_01x02

Commit message: almost done schematic
Parts:
- removed J23: OSTVN02A150, BCRL_power_supply:CONN_OSTVN02A150_OST, symbol 2024-02-14_22-22-09:OSTVN02A150
- removed J69: Conn_01x02, Connector_PinHeader_2.54mm:PinHeader_1x02_P2.54mm_Vertical, symbol Connector_Generic:Conn_01x02
- added J71, J72, J73, J74: OSTVN02A150, BCRL_power_supply:CONN_OSTVN02A150_OST, symbol 2024-02-14_22-22-09:OSTVN02A150
Connections:
- net GND: now also J71.2, J72.2, J73.2, J74.2
- new net V_FAN: J71.1, J72.1, J73.1, J74.1
Other:
- removed sheet PDQ10-Q48-S5-D_EMC_13
- added sheet PQC50-48-S5-O_EMC_trimmed_15 (PQC50-48-S5-O_EMC_trimmed.kicad_sch)

Commit message: schematic done
Other:
- moved on the sheet: J71, J72, J73, J74

Commit message: big changes
Parts:
- removed J72, J73, J74: OSTVN02A150, BCRL_power_supply:CONN_OSTVN02A150_OST, symbol 2024-02-14_22-22-09:OSTVN02A150
- added J46, J47, J48: OSTVN02A150, BCRL_power_supply:CONN_OSTVN02A150_OST, symbol 2024-02-14_22-22-09:OSTVN02A150
- renumbered J71 to J45
Connections:
- net GND: now also J46.2, J47.2, J48.2
- net V_FAN renamed +12V_1
- net +12V_1: now also J46.1
- new net +12V_2: J47.1, J48.1
Other:
- removed sheet PQC50-48-S5-O_EMC_trimmed_15
