File: kicad_files/bcrl_power_supply/fan_20x.kicad_sch (KiCad schematic)
At the start: 4 parts, among them J45 OSTVN02A150, J46 OSTVN02A150, J47 OSTVN02A150, J48 OSTVN02A150

Commit message: almost done schematic
Parts:
- renumbered J45 to J46, J46 to J47, J47 to J48, J48 to J49
Changed lines of the file:
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@@
 		(dnp no)
 		(fields_autoplaced yes)
-		(property "Reference" "#PWR0183"
+		(property "Reference" "#PWR0251"
 			(at 71.12 140.97 0)
 			(effects
@@
 			(project "bcrl_power_supply"
 				(path "/77f0f57c-9586-4625-9281-fa8cbd8015db/33e29609-c49f-40d6-8d19-845b9c0d1d83"
-					(reference "#PWR0183")
+					(reference "#PWR0251")
 					(unit 1)
 				)
@@
 		(dnp no)
 		(fields_autoplaced yes)
-		(property "Reference" "J47"
+		(property "Reference" "J48"
 			(at 91.44 118.11 0)
 			(effects
@@
 			)
 		)
+		(property "rating" ""
+			(at 77.47 118.11 0)
+			(effects
+				(font
+					(size 1.27 1.27)
+				)
+				(hide yes)
+			)
+		)
 		(pin "2"
 		)
@@
 			(project "bcrl_power_supply"
 				(path "/77f0f57c-9586-4625-9281-fa8cbd8015db/33e29609-c49f-40d6-8d19-845b9c0d1d83"
-					(reference "J47")
+					(reference "J48")
 					(unit 1)
 				)
@@
 		(dnp no)
 		(fields_autoplaced yes)
-		(property "Reference" "J48"
+		(property "Reference" "J49"
 			(at 91.44 138.43 0)
 			(effects
@@
 			)
 		)
+		(property "rating" ""
+			(at 77.47 138.43 0)
+			(effects
+				(font
+					(size 1.27 1.27)
+				)
+				(hide yes)
+			)
+		)
 		(pin "2"
 		)
@@
 			(project "bcrl_power_supply"
 				(path "/77f0f57c-9586-4625-9281-fa8cbd8015db/33e29609-c49f-40d6-8d19-845b9c0d1d83"
-					(reference "J48")
+					(reference "J49")
 					(unit 1)
 				)
@@
 		(dnp no)
 		(fields_autoplaced yes)
-		(property "Reference" "#PWR0182"
+		(property "Reference" "#PWR0250"
 			(at 71.12 120.65 0)
 			(effects
@@
 			(project "bcrl_power_supply"
 				(path "/77f0f57c-9586-4625-9281-fa8cbd8015db/33e29609-c49f-40d6-8d19-845b9c0d1d83"
-					(reference "#PWR0182")
+					(reference "#PWR0250")
 					(unit 1)
 				)
@@
 		(dnp no)
 		(fields_autoplaced yes)
-		(property "Reference" "#PWR0181"
+		(property "Reference" "#PWR0249"
 			(at 71.12 102.87 0)
 			(effects
@@
 			(project "bcrl_power_supply"
 				(path "/77f0f57c-9586-4625-9281-fa8cbd8015db/33e29609-c49f-40d6-8d19-845b9c0d1d83"
-					(reference "#PWR0181")
+					(reference "#PWR0249")
 					(unit 1)
 				)
@@
 		(dnp no)
 		(fields_autoplaced yes)
-		(property "Reference" "#PWR0221"
+		(property "Reference" "#PWR0248"
 			(at 71.12 83.82 0)
 			(effects
@@
 			(project "bcrl_power_supply"
 				(path "/77f0f57c-9586-4625-9281-fa8cbd8015db/33e29609-c49f-40d6-8d19-845b9c0d1d83"
-					(reference "#PWR0221")
+					(reference "#PWR0248")
 					(unit 1)
 				)
@@
 		(dnp no)
 		(fields_autoplaced yes)
-		(property "Reference" "J45"
+		(property "Reference" "J46"
 			(at 91.44 81.28 0)
 			(effects
@@
 			)
 		)
+		(property "rating" ""
+			(at 77.47 81.28 0)
+			(effects
+				(font
+					(size 1.27 1.27)
+				)
+				(hide yes)
+			)
+		)
 		(pin "2"
 		)
@@
 			(project "bcrl_power_supply"
 				(path "/77f0f57c-9586-4625-9281-fa8cbd8015db/33e29609-c49f-40d6-8d19-845b9c0d1d83"
-					(reference "J45")
+					(reference "J46")
 					(unit 1)
 				)
@@
 		(dnp no)
 		(fields_autoplaced yes)
-		(property "Reference" "J46"
+		(property "Reference" "J47"
 			(at 91.44 100.33 0)
 			(effects
@@
 			)
 		)
+		(property "rating" ""
+			(at 77.47 100.33 0)
+			(effects
+				(font
+					(size 1.27 1.27)
+				)
+				(hide yes)
+			)
+		)
 		(pin "2"
 		)
@@
 			(project "bcrl_power_supply"
 				(path "/77f0f57c-9586-4625-9281-fa8cbd8015db/33e29609-c49f-40d6-8d19-845b9c0d1d83"
-					(reference "J46")
-					(unit 1)
-				)
+					(reference "J47")
+					(unit 1)
+				)

Commit message: digikey BOM
Parts:
- J46, J47, J48, J49: DigiKey_Part_Number (none) -> OSTVN02A150
Changed lines of the file:
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@@
+			)
+		)
+		(property "DigiKey_Part_Number" "OSTVN02A150"
+			(at 77.47 118.11 0)
+			(effects
+				(font
+					(size 1.27 1.27)
+				)
+				(hide yes)
 			)
 		)
@@
 			)
 		)
+		(property "DigiKey_Part_Number" "OSTVN02A150"
+			(at 77.47 138.43 0)
+			(effects
+				(font
+					(size 1.27 1.27)
+				)
+				(hide yes)
+			)
+		)
 		(pin "2"
 		)
@@
 			)
 		)
+		(property "DigiKey_Part_Number" "OSTVN02A150"
+			(at 77.47 81.28 0)
+			(effects
+				(font
+					(size 1.27 1.27)
+				)
+				(hide yes)
+			)
+		)
 		(pin "2"
 		)
@@
 			(at 77.47 100.33 0)
 			(effects
+				(font
+					(size 1.27 1.27)
+				)
+				(hide yes)
+			)
+		)
+		(property "DigiKey_Part_Number" "OSTVN02A150"
+			(at 77.47 100.33 0)
+			(effects
