File: kicad_files/bcrl_power_supply/BFN.kicad_sch (KiCad schematic)
At the start: 18 parts, among them J49 Conn_01x04_Pin, J50 Conn_01x04_Pin, J51 Conn_01x04_Pin, J52 Conn_01x04_Pin, J53 Conn_01x04_Pin, J54 Conn_01x04_Pin, J55 Conn_01x04_Pin, J56 Conn_01x04_Pin, J57 Conn_01x04_Pin, J58 Conn_01x04_Pin, J59 Conn_01x04_Pin, J60 Conn_01x04_Pin, J61 Conn_01x04_Pin, J62 Conn_01x04_Pin, J63 Conn_01x04_Pin, J64 Conn_01x04_Pin, J65 Conn_01x04_Pin, J66 Conn_01x04_Pin

Commit message: almost done schematic
Parts:
- renumbered J49 to J51, J51 to J52, J52 to J53, J53 to J54, J54 to J55, J55 to J56, J56 to J57, J57 to J58, J58 to J59, J59 to J60, J65 to J62, J62 to J63, J63 to J64, J60 to J65, J64 to J66, J66 to J67

Commit message: board review
Parts:
- added D11, D12, D13, D14: LED 0603, LED_SMD:LED_0603_1608Metric, symbol Device:LED
- added J44, J45, J69, J70, J71, J72: Conn_01x02, Connector_PinHeader_2.54mm:PinHeader_1x02_P2.54mm_Vertical, symbol Connector_Generic:Conn_01x02
- added R15, R17, R19, R21: 1k, Resistor_SMD:R_0603_1608Metric, symbol Device:R
Connections:
- net +6.5V_RxBFN_C: now also D11.2 (A)
- net +6.5V_RxBFN_F: now also D12.2 (A)
- net +6.5V_TxBFN_C: now also D13.2 (A)
- net +6.5V_TxBFN_F: now also D14.2 (A)
- net GND: now also J44.2 (Pin_2), J45.2 (Pin_2), J69.2 (Pin_2), J70.2 (Pin_2), J71.2 (Pin_2), J72.2 (Pin_2), R15.1, R17.1, R19.1, R21.1
- new net: D11.1 (K), R15.2
- new net: D12.1 (K), R17.2
- new net: D14.1 (K), R21.2
- new net: D13.1 (K), R19.2
- new net +12V_CTRL_RxBFN: J44.1 (Pin_1)
- new net +12V_CTRL_TxBFN: J70.1 (Pin_1)
- new net +6.5V_CTRL_RxBFN_C: J45.1 (Pin_1)
- new net +6.5V_CTRL_RxBFN_F: J69.1 (Pin_1)
- new net +6.5V_CTRL_TxBFN_C: J71.1 (Pin_1)
- new net +6.5V_CTRL_TxBFN_F: J72.1 (Pin_1)
Other:
- moved on the sheet: J50, J51, J52, J53, J55, J56, J57, J58, J59, J60, J61, J62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

Commit message: digikey BOM
Parts:
- D11, D12, D13, D14: DigiKey_Part_Number (none) -> 150060GS75000
- R15, R17, R19, R21: DigiKey_Part_Number (none) -> ESR03EZPF1001
Changed lines of the file:
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@@
 			)
 		)
-		(property "Description" ""
+		(property "Description" "LED diode"
 			(at 135.89 31.75 0)
 			(effects
@@
 			)
 		)
+		(property "DigiKey_Part_Number" "150060GS75000 "
+			(at 135.89 31.75 0)
+			(effects
+				(font
+					(size 1.27 1.27)
+				)
+				(hide yes)
+			)
+		)
 		(pin "2"
 		)
@@
 			)
 		)
-		(property "Description" ""
+		(property "Description" "Resistor"
 			(at 135.89 66.04 0)
 			(effects
@@
 			)
 		)
+		(property "DigiKey_Part_Number" "ESR03EZPF1001 "
+			(at 135.89 66.04 0)
+			(effects
+				(font
+					(size 1.27 1.27)
+				)
+				(hide yes)
+			)
+		)
 		(pin "1"
 		)
@@
 			)
 		)
-		(property "Description" ""
+		(property "Description" "Resistor"
 			(at 267.97 66.04 0)
 			(effects
@@
 			)
 		)
+		(property "DigiKey_Part_Number" "ESR03EZPF1001 "
+			(at 267.97 66.04 0)
+			(effects
+				(font
+					(size 1.27 1.27)
+				)
+				(hide yes)
+			)
+		)
 		(pin "1"
 		)
@@
 			)
 		)
-		(property "Description" ""
+		(property "Description" "Resistor"
 			(at 135.89 24.13 0)
 			(effects
@@
 			)
 		)
+		(property "DigiKey_Part_Number" "ESR03EZPF1001 "
+			(at 135.89 24.13 0)
+			(effects
+				(font
+					(size 1.27 1.27)
+				)
+				(hide yes)
+			)
+		)
 		(pin "1"
 		)
@@
 			)
 		)
-		(property "Description" ""
+		(property "Description" "LED diode"
 			(at 267.97 31.75 0)
 			(effects
@@
 			)
 		)
+		(property "DigiKey_Part_Number" "150060GS75000 "
+			(at 267.97 31.75 0)
+			(effects
+				(font
+					(size 1.27 1.27)
+				)
+				(hide yes)
+			)
+		)
 		(pin "2"
 		)
@@
 			)
 		)
-		(property "Description" ""
+		(property "Description" "LED diode"
 			(at 135.89 58.42 0)
 			(effects
@@
 			)
 		)
+		(property "DigiKey_Part_Number" "150060GS75000 "
+			(at 135.89 58.42 0)
+			(effects
+				(font
+					(size 1.27 1.27)
+				)
+				(hide yes)
+			)
+		)
 		(pin "2"
 		)
@@
 			)
 		)
-		(property "Description" ""
+		(property "Description" "Resistor"
 			(at 267.97 24.13 0)
 			(effects
@@
 			)
 		)
+		(property "DigiKey_Part_Number" "ESR03EZPF1001 "
+			(at 267.97 24.13 0)
+			(effects
+				(font
+					(size 1.27 1.27)
+				)
+				(hide yes)
+			)
+		)
 		(pin "1"
 		)
@@
 			)
 		)
-		(property "Description" ""
+		(property "Description" "LED diode"
 			(at 267.97 58.42 0)
 			(effects
@@
 			(at 267.97 58.42 0)
 			(effects
+				(font
+					(size 1.27 1.27)
+				)
+				(hide yes)
+			)
+		)
+		(property "DigiKey_Part_Number" "150060GS75000 "
+			(at 267.97 58.42 0)
+			(effects
