File: kicad_files/bcrl_power_supply/FLT007A0Z_EMC.kicad_sch (KiCad schematic)
At the start: 4 parts

Commit message: digikey BOM
Parts:
- C35, C36, C41: footprint Capacitor_SMD:C_0603_1608Metric -> Capacitor_SMD:C_1206_3216Metric; DigiKey_Part_Number (none) -> HMK316AC7225KL-TE
- FL1: DigiKey_Part_Number (none) -> FLT007A0Z
Changed lines of the file:
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@@
+			)
+		)
+		(property "DigiKey_Part_Number" "FLT007A0Z"
+			(at 123.19 85.09 0)
+			(effects
+				(font
+					(size 1.27 1.27)
+				)
+				(hide yes)
 			)
 		)
@@
 			)
 		)
-		(property "Footprint" "Capacitor_SMD:C_0603_1608Metric"
+		(property "Footprint" "Capacitor_SMD:C_1206_3216Metric"
 			(at 72.0852 91.44 0)
 			(effects
@@
 			)
 		)
+		(property "DigiKey_Part_Number" "HMK316AC7225KL-TE "
+			(at 71.12 87.63 0)
+			(effects
+				(font
+					(size 1.27 1.27)
+				)
+				(hide yes)
+			)
+		)
 		(pin "1"
 		)
@@
 			)
 		)
-		(property "Footprint" "Capacitor_SMD:C_0603_1608Metric"
+		(property "Footprint" "Capacitor_SMD:C_1206_3216Metric"
 			(at 86.0552 91.44 0)
 			(effects
@@
 			)
 		)
+		(property "DigiKey_Part_Number" "HMK316AC7225KL-TE "
+			(at 85.09 87.63 0)
+			(effects
+				(font
+					(size 1.27 1.27)
+				)
+				(hide yes)
+			)
+		)
 		(pin "1"
 		)
@@
 			)
 		)
-		(property "Footprint" "Capacitor_SMD:C_0603_1608Metric"
+		(property "Footprint" "Capacitor_SMD:C_1206_3216Metric"
 			(at 100.0252 91.44 0)
 			(effects
@@
 			(at 99.06 87.63 0)
 			(effects
+				(font
+					(size 1.27 1.27)
+				)
+				(hide yes)
+			)
+		)
+		(property "DigiKey_Part_Number" "HMK316AC7225KL-TE "
+			(at 99.06 87.63 0)
+			(effects
