File: kicad_files/bcrl_power_supply/IND108W_EMC_6.5V.kicad_sch (KiCad schematic)
At the start: 10 parts

Commit message: almost done schematic
Parts:
- C87: renamed from C125; value 22uf -> 22u
- C88: renamed from C126; value 22uf -> 22u
- C89: renamed from C127; value 22uf -> 22u
- C90: renamed from C128; value 22uf -> 22u
- C91: renamed from C129; value 22uf -> 22u
- C92: renamed from C130; value 22uf -> 22u
- R46: renamed from R36; value 9.59k -> 12.06k
- renumbered D23 to D29, PS15 to PS12, R39 to R47
Connections:
- net +8V renamed +6.5V
- net +8V_CTRL renamed +6.5V_CTRL
Other:
- note added: "Rtrim = 70/(Vout - 0.7) kiloohms"

Commit message: board review
Parts:
- removed D29: LED, LED_SMD:LED_0603_1608Metric, symbol Device:LED
- removed R47: 1k, Resistor_SMD:R_0603_1608Metric, symbol Device:R
- PS12: footprint IND108W -> BCRL_power_supply:IND108W
Other:
- note added: "Rtrim = 70/(Vout - 0.7) kiloohms https://www.mouser.ca/datasheet/2/167/ind108w_ds-3402027.pdf"
- note removed: "Rtrim = 70/(Vout - 0.7) kiloohms"

Commit message: digikey BOM
Parts:
- C87, C88, C89, C90, C91, C92: footprint Capacitor_SMD:C_0603_1608Metric -> Capacitor_SMD:C_1206_3216Metric; DigiKey_Part_Number (none) -> C3216X5R1V226M160AC
- PS12: DigiKey_Part_Number (none) -> IND108W
- R46: DigiKey_Part_Number (none) -> ESR03EZPJ123
Changed lines of the file:
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@@
 			)
 		)
-		(property "Footprint" "Capacitor_SMD:C_0603_1608Metric"
+		(property "Footprint" "Capacitor_SMD:C_1206_3216Metric"
 			(at 122.8852 111.76 0)
 			(effects
@@
 		)
 		(property "rating" ""
+			(at 121.92 107.95 0)
+			(effects
+				(font
+					(size 1.27 1.27)
+				)
+				(hide yes)
+			)
+		)
+		(property "DigiKey_Part_Number" " C3216X5R1V226M160AC "
 			(at 121.92 107.95 0)
 			(effects
@@
 			)
 		)
-		(property "Footprint" "Capacitor_SMD:C_0603_1608Metric"
+		(property "Footprint" "Capacitor_SMD:C_1206_3216Metric"
 			(at 135.5852 111.76 0)
 			(effects
@@
 		)
 		(property "rating" ""
+			(at 134.62 107.95 0)
+			(effects
+				(font
+					(size 1.27 1.27)
+				)
+				(hide yes)
+			)
+		)
+		(property "DigiKey_Part_Number" " C3216X5R1V226M160AC "
 			(at 134.62 107.95 0)
 			(effects
@@
 			)
 		)
+		(property "DigiKey_Part_Number" "IND108W"
+			(at 128.27 85.09 0)
+			(effects
+				(font
+					(size 1.27 1.27)
+				)
+				(hide yes)
+			)
+		)
 		(pin "5"
 		)
@@
 			)
 		)
-		(property "Footprint" "Capacitor_SMD:C_0603_1608Metric"
+		(property "Footprint" "Capacitor_SMD:C_1206_3216Metric"
 			(at 162.2552 109.22 0)
 			(effects
@@
 		)
 		(property "rating" ""
+			(at 161.29 105.41 0)
+			(effects
+				(font
+					(size 1.27 1.27)
+				)
+				(hide yes)
+			)
+		)
+		(property "DigiKey_Part_Number" " C3216X5R1V226M160AC "
 			(at 161.29 105.41 0)
 			(effects
@@
 			)
 		)
-		(property "Footprint" "Capacitor_SMD:C_0603_1608Metric"
+		(property "Footprint" "Capacitor_SMD:C_1206_3216Metric"
 			(at 174.9552 109.22 0)
 			(effects
@@
 		)
 		(property "rating" ""
+			(at 173.99 105.41 0)
+			(effects
+				(font
+					(size 1.27 1.27)
+				)
+				(hide yes)
+			)
+		)
+		(property "DigiKey_Part_Number" " C3216X5R1V226M160AC "
 			(at 173.99 105.41 0)
 			(effects
@@
 			)
 		)
-		(property "Description" ""
+		(property "Description" "Resistor"
 			(at 102.87 85.09 0)
 			(effects
@@
 		)
 		(property "rating" ""
+			(at 102.87 85.09 0)
+			(effects
+				(font
+					(size 1.27 1.27)
+				)
+				(hide yes)
+			)
+		)
+		(property "DigiKey_Part_Number" "ESR03EZPJ123 "
 			(at 102.87 85.09 0)
 			(effects
@@
 			)
 		)
-		(property "Footprint" "Capacitor_SMD:C_0603_1608Metric"
+		(property "Footprint" "Capacitor_SMD:C_1206_3216Metric"
 			(at 149.5552 109.22 0)
 			(effects
@@
 		)
 		(property "rating" ""
+			(at 148.59 105.41 0)
+			(effects
+				(font
+					(size 1.27 1.27)
+				)
+				(hide yes)
+			)
+		)
+		(property "DigiKey_Part_Number" " C3216X5R1V226M160AC "
 			(at 148.59 105.41 0)
 			(effects
@@
 			)
 		)
-		(property "Footprint" "Capacitor_SMD:C_0603_1608Metric"
+		(property "Footprint" "Capacitor_SMD:C_1206_3216Metric"
 			(at 110.1852 111.76 0)
 			(effects
@@
 			(at 109.22 107.95 0)
 			(effects
+				(font
+					(size 1.27 1.27)
+				)
+				(hide yes)
+			)
+		)
+		(property "DigiKey_Part_Number" " C3216X5R1V226M160AC "
+			(at 109.22 107.95 0)
+			(effects
