File: kicad_files/bcrl_power_supply/IND108W_EMC_8V.kicad_sch (KiCad schematic)
At the start: 10 parts

Commit message: almost done schematic
Parts:
- removed C153, C154, C155, C156, C157, C158: 22uf, Capacitor_SMD:C_0603_1608Metric, symbol Device:C
- removed D27: LED, LED_SMD:LED_0603_1608Metric, symbol Device:LED
- removed PS20: IND108W, IND108W, symbol BCRL_power_supply:IND108W
- removed R53: 9.59k, Resistor_SMD:R_0603_1608Metric, symbol Device:R
- removed R54: 1k, Resistor_SMD:R_0603_1608Metric, symbol Device:R
- added C117, C118, C119, C120, C121, C122: 22u, Capacitor_SMD:C_0603_1608Metric, symbol Device:C
- added D33: LED, LED_SMD:LED_0603_1608Metric, symbol Device:LED
- added PS17: IND108W, IND108W, symbol BCRL_power_supply:IND108W
- added R55: 9.59k, Resistor_SMD:R_0603_1608Metric, symbol Device:R
- added R56: 1k, Resistor_SMD:R_0603_1608Metric, symbol Device:R
Connections:
- net +12V: now also C120.1, C121.1, C122.1, PS17.9 (VIN)
- net +8V: now also C117.1, C118.1, C119.1, D33.2 (A), PS17.3 (VS+), PS17.5 (VOUT)
- net +8V_CTRL: now also PS17.1 (ON/OFF)
- net GND: now also C117.2, C118.2, C119.2, C120.2, C121.2, C122.2, PS17.2 (GND_1), PS17.6 (GND_2), PS17.7 (SYNC), PS17.8 (GND_3), R55.2, R56.1
- new net: PS17.4 (TRIM), R55.1
- new net: D33.1 (K), R56.2
Other:
- note added: "Rtrim = 70/(Vout - 0.7) kiloohms"

Commit message: board review
Parts:
- removed D33: LED, LED_SMD:LED_0603_1608Metric, symbol Device:LED
- removed R56: 1k, Resistor_SMD:R_0603_1608Metric, symbol Device:R
- PS17: footprint IND108W -> BCRL_power_supply:IND108W
Other:
- note added: "Rtrim = 70/(Vout - 0.7) kiloohms https://www.mouser.ca/datasheet/2/167/ind108w_ds-3402027.pdf"
- note removed: "Rtrim = 70/(Vout - 0.7) kiloohms"

Commit message: digikey BOM
Parts:
- C117, C118, C119, C120, C121, C122: footprint Capacitor_SMD:C_0603_1608Metric -> Capacitor_SMD:C_1206_3216Metric; DigiKey_Part_Number (none) -> C3216X5R1V226M160AC
- PS17: DigiKey_Part_Number (none) -> IND108W
- R55: DigiKey_Part_Number (none) -> RCS06039K53FKEA
Changed lines of the file:
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@@
+			)
+		)
+		(property "DigiKey_Part_Number" "IND108W"
+			(at 128.27 85.09 0)
+			(effects
+				(font
+					(size 1.27 1.27)
+				)
+				(hide yes)
 			)
 		)
@@
 			)
 		)
-		(property "Description" ""
+		(property "Description" "Resistor"
 			(at 102.87 85.09 0)
 			(effects
@@
 		)
 		(property "rating" ""
+			(at 102.87 85.09 0)
+			(effects
+				(font
+					(size 1.27 1.27)
+				)
+				(hide yes)
+			)
+		)
+		(property "DigiKey_Part_Number" "RCS06039K53FKEA "
 			(at 102.87 85.09 0)
 			(effects
@@
 			)
 		)
-		(property "Footprint" "Capacitor_SMD:C_0603_1608Metric"
+		(property "Footprint" "Capacitor_SMD:C_1206_3216Metric"
 			(at 122.8852 111.76 0)
 			(effects
@@
 		)
 		(property "rating" ""
+			(at 121.92 107.95 0)
+			(effects
+				(font
+					(size 1.27 1.27)
+				)
+				(hide yes)
+			)
+		)
+		(property "DigiKey_Part_Number" " C3216X5R1V226M160AC "
 			(at 121.92 107.95 0)
 			(effects
@@
 			)
 		)
-		(property "Footprint" "Capacitor_SMD:C_0603_1608Metric"
+		(property "Footprint" "Capacitor_SMD:C_1206_3216Metric"
 			(at 110.1852 111.76 0)
 			(effects
@@
 		)
 		(property "rating" ""
+			(at 109.22 107.95 0)
+			(effects
+				(font
+					(size 1.27 1.27)
+				)
+				(hide yes)
+			)
+		)
+		(property "DigiKey_Part_Number" " C3216X5R1V226M160AC "
 			(at 109.22 107.95 0)
 			(effects
@@
 			)
 		)
-		(property "Footprint" "Capacitor_SMD:C_0603_1608Metric"
+		(property "Footprint" "Capacitor_SMD:C_1206_3216Metric"
 			(at 174.9552 109.22 0)
 			(effects
@@
 		)
 		(property "rating" ""
+			(at 173.99 105.41 0)
+			(effects
+				(font
+					(size 1.27 1.27)
+				)
+				(hide yes)
+			)
+		)
+		(property "DigiKey_Part_Number" " C3216X5R1V226M160AC "
 			(at 173.99 105.41 0)
 			(effects
@@
 			)
 		)
-		(property "Footprint" "Capacitor_SMD:C_0603_1608Metric"
+		(property "Footprint" "Capacitor_SMD:C_1206_3216Metric"
 			(at 149.5552 109.22 0)
 			(effects
@@
 		)
 		(property "rating" ""
+			(at 148.59 105.41 0)
+			(effects
+				(font
+					(size 1.27 1.27)
+				)
+				(hide yes)
+			)
+		)
+		(property "DigiKey_Part_Number" " C3216X5R1V226M160AC "
 			(at 148.59 105.41 0)
 			(effects
@@
 			)
 		)
-		(property "Footprint" "Capacitor_SMD:C_0603_1608Metric"
+		(property "Footprint" "Capacitor_SMD:C_1206_3216Metric"
 			(at 135.5852 111.76 0)
 			(effects
@@
 		)
 		(property "rating" ""
+			(at 134.62 107.95 0)
+			(effects
+				(font
+					(size 1.27 1.27)
+				)
+				(hide yes)
+			)
+		)
+		(property "DigiKey_Part_Number" " C3216X5R1V226M160AC "
 			(at 134.62 107.95 0)
 			(effects
@@
 			)
 		)
-		(property "Footprint" "Capacitor_SMD:C_0603_1608Metric"
+		(property "Footprint" "Capacitor_SMD:C_1206_3216Metric"
 			(at 162.2552 109.22 0)
 			(effects
@@
 			(at 161.29 105.41 0)
 			(effects
+				(font
+					(size 1.27 1.27)
+				)
+				(hide yes)
+			)
+		)
+		(property "DigiKey_Part_Number" " C3216X5R1V226M160AC "
+			(at 161.29 105.41 0)
+			(effects
