File: kicad_files/bcrl_power_supply/RPi_HAT.kicad_sch (KiCad schematic)
At the start: 8 parts, among them J67 Conn_01x06_Pin, J68 Conn_01x06_Pin, J69 Conn_01x06_Pin, J70 Conn_01x06_Pin, J75 Conn_01x06_Pin, J76 Conn_01x06_Pin, J77 Conn_01x06_Pin, J78 Conn_01x06_Pin

Commit message: almost done schematic
Parts:
- added D37, D38: LED, LED_SMD:LED_0603_1608Metric, symbol Device:LED
- added J76, J77: Conn_01x02, Connector_PinHeader_2.54mm:PinHeader_1x02_P2.54mm_Vertical, symbol Connector_Generic:Conn_01x02
- added R62, R63: 1k, Resistor_SMD:R_0603_1608Metric, symbol Device:R
- renumbered J75 to J68, J76 to J69, J77 to J70, J78 to J71, J67 to J72, J68 to J73, J69 to J74, J70 to J75
Connections:
- net GND: now also R62.1, R63.1
- new net: D38.1 (K), R63.2
- new net: D37.1 (K), R62.2
- new net +24V: D38.2 (A)
- new net +5V: D37.2 (A)
- new net +5V_CTRL: J76.1 (Pin_1)
Other:
- removed sheet Rx_RPi4_HAT_board1
- removed sheet Tx_RPi4_HAT_board1
- added sheet PDQ10-Q48-S5-D_EMC_9 (PDQ10-Q48-S5-D_EMC.kicad_sch)
- added sheet PDQE15-Q48-D24-D_EMC_2 (PDQE15-Q48-D24-D_EMC.kicad_sch)
- moved on the sheet: J68, J69, J70, J71, J72, J73, J74, J75

Commit message: board review
Parts:
- removed J69, J70, J71, J72: Conn_01x06_Pin, Connector_PinHeader_2.54mm:PinHeader_1x06_P2.54mm_Vertical, symbol Connector:Conn_01x06_Pin
- added J80, J81, J82, J83: Conn_01x06_Pin, Connector_PinHeader_2.54mm:PinHeader_1x06_P2.54mm_Vertical, symbol Connector:Conn_01x06_Pin
- D37, D38: value LED -> LED 0603
Connections:
- net +24V_Rx_RPi4_HAT is gone; now on net +24V: J68.3 (Pin_3)
- net +24V_Tx_RPi4_HAT is gone; now on net +24V: J73.3 (Pin_3), J74.3 (Pin_3), J75.3 (Pin_3)
- net +5V_Rx_RPi4_HAT is gone; now on net +5V: J68.2 (Pin_2)
- net +5V_Tx_RPi4_HAT is gone; now on net +5V: J73.2 (Pin_2), J74.2 (Pin_2), J75.2 (Pin_2)
- net +24V: now also J80.3 (Pin_3), J81.3 (Pin_3), J82.3 (Pin_3), J83.3 (Pin_3)
- net +24V_CTRL: now also J77.1 (Pin_1)
- net +3.3V: now also J80.6 (Pin_6), J81.6 (Pin_6), J82.6 (Pin_6), J83.6 (Pin_6)
- net +5V: now also J80.2 (Pin_2), J81.2 (Pin_2), J82.2 (Pin_2), J83.2 (Pin_2)
- net GND: now also J76.2 (Pin_2), J77.2 (Pin_2), J80.1 (Pin_1), J80.4 (Pin_4), J80.5 (Pin_5), J81.1 (Pin_1), J81.4 (Pin_4), J81.5 (Pin_5), J82.1 (Pin_1), J82.4 (Pin_4), J82.5 (Pin_5), J83.1 (Pin_1), J83.4 (Pin_4), J83.5 (Pin_5)
Other:
- moved on the sheet: J68, J76, J77

Commit message: digikey BOM
Parts:
- D37, D38: DigiKey_Part_Number (none) -> 150060GS75000
- R62, R63: DigiKey_Part_Number (none) -> ESR03EZPF1001
Changed lines of the file:
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@@
 			)
 		)
-		(property "Description" ""
+		(property "Description" "LED diode"
 			(at 91.44 60.96 0)
 			(effects
@@
 		)
 		(property "rating" ""
+			(at 91.44 60.96 0)
+			(effects
+				(font
+					(size 1.27 1.27)
+				)
+				(hide yes)
+			)
+		)
+		(property "DigiKey_Part_Number" "150060GS75000 "
 			(at 91.44 60.96 0)
 			(effects
@@
 			)
 		)
-		(property "Description" ""
+		(property "Description" "Resistor"
 			(at 91.44 33.02 0)
 			(effects
@@
 		)
 		(property "rating" ""
+			(at 91.44 33.02 0)
+			(effects
+				(font
+					(size 1.27 1.27)
+				)
+				(hide yes)
+			)
+		)
+		(property "DigiKey_Part_Number" "ESR03EZPF1001 "
 			(at 91.44 33.02 0)
 			(effects
@@
 			)
 		)
-		(property "Description" ""
+		(property "Description" "LED diode"
 			(at 83.82 33.02 0)
 			(effects
@@
 		)
 		(property "rating" ""
+			(at 83.82 33.02 0)
+			(effects
+				(font
+					(size 1.27 1.27)
+				)
+				(hide yes)
+			)
+		)
+		(property "DigiKey_Part_Number" "150060GS75000 "
 			(at 83.82 33.02 0)
 			(effects
@@
 			)
 		)
-		(property "Description" ""
+		(property "Description" "Resistor"
 			(at 99.06 60.96 0)
 			(effects
@@
 			(at 99.06 60.96 0)
 			(effects
+				(font
+					(size 1.27 1.27)
+				)
+				(hide yes)
+			)
+		)
+		(property "DigiKey_Part_Number" "ESR03EZPF1001 "
+			(at 99.06 60.96 0)
+			(effects
